File: 100Base-TX-PHY7.kicad_sch (KiCad schematic)
At the start: 52 parts, among them J9 JK0654219, U12 KSZ9131RNX, U13 SC4626C, U2 SJA1105Q

Commit message: Minor corrections
Parts:
- renumbered R194 to R201, R195 to R202, R196 to R203, R197 to R204, R198 to R205, R199 to R206, R200 to R207, R201 to R208, R202 to R209, R203 to R210, R204 to R211, R205 to R212, R206 to R213, R207 to R214, R208 to R215, R209 to R216, R210 to R217, R211 to R218, R212 to R219, R213 to R220, R214 to R221, R215 to R222, R216 to R223
Other:
- note added: "Mode: 0b1110 --------- 1000BaseT FDX 10/100BaseTX FDX 10BaseT HDX (NOT SUPPORTED BY MAC!!!)"
- note added: "PHY ADDRESS: 0b111"
- note removed: "Mode: 0b1110 1000BT FD / 10/100BT FD / 10BT HD"
- note removed: "PHY-ADDR 7: 0b111"

Commit message: Assigning Footprints
Parts:
- added R321, R322: 470, Resistor_SMD:R_0603_1608Metric, symbol Device:R
- FB16, FB17, FB18: value FerriteBead -> 782763301; footprint (none) -> Inductor_SMD:L_1206_3216Metric
- H8: footprint (none) -> MountingHole:MountingHole_3.2mm_M3_Pad_Via
Connections:
- net at R205.2, U12.17 (LED1/PME_N1/PHYAD0): now also R321.1; no longer J9.15 (LED1-)
- net at R206.2, U12.15 (LED2/PHYAD1): now also R322.1; no longer J9.13 (LED2-)
- new net: J9.15 (LED1-), R321.2
- new net: J9.13 (LED2-), R322.2
Changed lines of the file:
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@@
   (junction (at 171.45 132.08) (diameter 0) (color 0 0 0 0)
   )
+  (junction (at 238.76 100.33) (diameter 0) (color 0 0 0 0)
+  )
+  (junction (at 171.45 160.02) (diameter 0) (color 0 0 0 0)
+  )
+  (junction (at 90.17 48.26) (diameter 0) (color 0 0 0 0)
+  )
+  (junction (at 163.83 139.7) (diameter 0) (color 0 0 0 0)
+  )
+  (junction (at 179.07 132.08) (diameter 0) (color 0 0 0 0)
+  )
   (junction (at 172.72 88.9) (diameter 0) (color 0 0 0 0)
   )
-  (junction (at 238.76 100.33) (diameter 0) (color 0 0 0 0)
-  )
-  (junction (at 171.45 160.02) (diameter 0) (color 0 0 0 0)
-  )
-  (junction (at 90.17 48.26) (diameter 0) (color 0 0 0 0)
-  )
-  (junction (at 163.83 139.7) (diameter 0) (color 0 0 0 0)
-  )
-  (junction (at 179.07 132.08) (diameter 0) (color 0 0 0 0)
-  )
   (junction (at 186.69 58.42) (diameter 0) (color 0 0 0 0)
   )
@@
   (junction (at 237.49 152.4) (diameter 0) (color 0 0 0 0)
   )
+  (junction (at 186.69 160.02) (diameter 0) (color 0 0 0 0)
+  )
+  (junction (at 179.07 104.14) (diameter 0) (color 0 0 0 0)
+  )
+  (junction (at 163.83 124.46) (diameter 0) (color 0 0 0 0)
+  )
+  (junction (at 186.69 147.32) (diameter 0) (color 0 0 0 0)
+  )
   (junction (at 167.64 40.64) (diameter 0) (color 0 0 0 0)
   )
-  (junction (at 186.69 160.02) (diameter 0) (color 0 0 0 0)
-  )
-  (junction (at 179.07 104.14) (diameter 0) (color 0 0 0 0)
-  )
-  (junction (at 163.83 124.46) (diameter 0) (color 0 0 0 0)
-  )
-  (junction (at 186.69 147.32) (diameter 0) (color 0 0 0 0)
-  )
   (junction (at 201.93 104.14) (diameter 0) (color 0 0 0 0)
   )
@@
     (stroke (width 0) (type default) (color 0 0 0 0))
   )
+  (wire (pts (xy 200.66 40.64) (xy 220.98 40.64))
+    (stroke (width 0) (type default) (color 0 0 0 0))
+  )
   (wire (pts (xy 194.31 132.08) (xy 201.93 132.08))
     (stroke (width 0) (type default) (color 0 0 0 0))
@@
     (stroke (width 0) (type default) (color 0 0 0 0))
   )
+  (wire (pts (xy 167.64 40.64) (xy 193.04 40.64))
+    (stroke (width 0) (type default) (color 0 0 0 0))
+  )
   (wire (pts (xy 161.29 160.02) (xy 163.83 160.02))
     (stroke (width 0) (type default) (color 0 0 0 0))
@@
     (stroke (width 0) (type default) (color 0 0 0 0))
   )
-  (wire (pts (xy 220.98 40.64) (xy 167.64 40.64))
-    (stroke (width 0) (type default) (color 0 0 0 0))
-  )
   (wire (pts (xy 67.31 40.64) (xy 100.33 40.64))
     (stroke (width 0) (type default) (color 0 0 0 0))
@@
     (stroke (width 0) (type default) (color 0 0 0 0))
   )
+  (wire (pts (xy 172.72 88.9) (xy 193.04 88.9))
+    (stroke (width 0) (type default) (color 0 0 0 0))
+  )
   (wire (pts (xy 238.76 100.33) (xy 238.76 102.87))
     (stroke (width 0) (type default) (color 0 0 0 0))
@@
     (stroke (width 0) (type default) (color 0 0 0 0))
   )
-  (wire (pts (xy 220.98 88.9) (xy 172.72 88.9))
-    (stroke (width 0) (type default) (color 0 0 0 0))
-  )
   (wire (pts (xy 194.31 147.32) (xy 201.93 147.32))
     (stroke (width 0) (type default) (color 0 0 0 0))
@@
   )
   (wire (pts (xy 67.31 53.34) (xy 81.28 53.34))
+    (stroke (width 0) (type default) (color 0 0 0 0))
+  )
+  (wire (pts (xy 200.66 88.9) (xy 220.98 88.9))
     (stroke (width 0) (type default) (color 0 0 0 0))
   )
@@
     (in_bom yes) (on_board yes)
     (property "Reference" "FB17" (id 0) (at 210.185 107.95 90))
-    (property "Value" "FerriteBead" (id 1) (at 210.82 100.33 90))
-    (property "Footprint" "" (id 2) (at 210.82 105.918 90)
+    (property "Value" "782763301" (id 1) (at 210.82 100.33 90))
+    (property "Footprint" "Inductor_SMD:L_1206_3216Metric" (id 2) (at 210.82 105.918 90)
       (effects (font (size 1.27 1.27)) hide)
     )
@@
       (effects (font (size 1.27 1.27)) hide)
     )
-    (property "Datasheet" "https://www.mouser.com/datasheet/2/761/sc4626-1277391.pdf" (id 3) (at 246.38 130.81 0)
+    (property "Datasheet" "~" (id 3) (at 246.38 130.81 0)
       (effects (font (size 1.27 1.27)) hide)
     )
@@
     (pin "5")
   )
+  (symbol (lib_id "Device:R") (at 196.85 40.64 90) (unit 1)
+    (in_bom yes) (on_board yes)
+    (property "Reference" "R321" (id 0) (at 196.85 38.608 90))
+    (property "Value" "470" (id 1) (at 196.85 40.64 90))
+    (property "Footprint" "Resistor_SMD:R_0603_1608Metric" (id 2) (at 196.85 42.418 90)
+      (effects (font (size 1.27 1.27)) hide)
+    )
+    (property "Datasheet" "~" (id 3) (at 196.85 40.64 0)
+      (effects (font (size 1.27 1.27)) hide)
+    )
+    (pin "1")
+    (pin "2")
+  )
   (symbol (lib_id "Device:R") (at 76.2 34.29 0) (unit 1)
     (in_bom yes) (on_board yes)
@@
     (property "Reference" "H8" (id 0) (at 260.35 100.33 0))
     (property "Value" "CHASSIS_PE" (id 1) (at 258.445 100.33 0))
-    (property "Footprint" "" (id 2) (at 254 100.33 0)
+    (property "Footprint" "MountingHole:MountingHole_3.2mm_M3_Pad_Via" (id 2) (at 254 100.33 0)
       (effects (font (size 1.27 1.27)) hide)
     )
@@
     )
     (property "Datasheet" "~" (id 3) (at 81.28 34.29 0)
+      (effects (font (size 1.27 1.27)) hide)
+    )
+    (pin "1")
+    (pin "2")
+  )
+  (symbol (lib_id "Device:R") (at 196.85 88.9 90) (unit 1)
+    (in_bom yes) (on_board yes)
+    (property "Reference" "R322" (id 0) (at 196.85 86.868 90))
+    (property "Value" "470" (id 1) (at 196.85 88.9 90))
+    (property "Footprint" "Resistor_SMD:R_0603_1608Metric" (id 2) (at 196.85 90.678 90)
+      (effects (font (size 1.27 1.27)) hide)
+    )
+    (property "Datasheet" "~" (id 3) (at 196.85 88.9 0)
       (effects (font (size 1.27 1.27)) hide)
     )
@@
     (in_bom yes) (on_board yes)
     (property "Reference" "FB16" (id 0) (at 187.325 107.95 90))
-    (property "Value" "FerriteBead" (id 1) (at 187.96 100.33 90))
-    (property "Footprint" "" (id 2) (at 187.96 105.918 90)
+    (property "Value" "782763301" (id 1) (at 187.96 100.33 90))
+    (property "Footprint" "Inductor_SMD:L_1206_3216Metric" (id 2) (at 187.96 105.918 90)
       (effects (font (size 1.27 1.27)) hide)
     )
@@
     (in_bom yes) (on_board yes)
     (property "Reference" "FB18" (id 0) (at 210.185 151.13 90))
-    (property "Value" "FerriteBead" (id 1) (at 210.82 143.51 90))
-    (property "Footprint" "" (id 2) (at 210.82 149.098 90)
+    (property "Value" "782763301" (id 1) (at 210.82 143.51 90))
+    (property "Footprint" "Inductor_SMD:L_1206_3216Metric" (id 2) (at 210.82 149.098 90)
       (effects (font (size 1.27 1.27)) hide)
     )
@@
       (effects (font (size 1.27 1.27)) hide)
     )
-    (property "Datasheet" "https://media.digikey.com/pdf/Data%20Sheets/Pulse%20PDFs/JK%20Series.pdf" (id 3) (at 238.633 96.393 0)
-      (effects (font (size 1.27 1.27)) hide)
-    )
+    (property "Datasheet" "~" (id 3) (at 238.633 96.393 0)
+      (effects (font (size 1.27 1.27)) hide)
+    )
