File: 10Base-T1L-PHY4.kicad_sch (KiCad schematic)
At the start: 52 parts, among them J6 PHY5_MDI, U2 SJA1105Q, U9 ADIN1100

Commit message: Minor corrections
Parts:
- added R125: 4K7, Resistor_SMD:R_0603_1608Metric, symbol Device:R
- R126: renamed from R121; value 1K -> 4K7
- renumbered R117 to R121, R118 to R122, R119 to R123, R120 to R124, R122 to R127, R123 to R128, R124 to R129, R125 to R130, R126 to R131, R127 to R132, R128 to R133, R129 to R134, R130 to R135, R131 to R136, R132 to R137, R133 to R138, R134 to R139, R135 to R140, R136 to R141, R137 to R142, R138 to R143, R139 to R144, R140 to R145, R141 to R146
Connections:
- net +3V3: now also R125.2
- net at R129.1, U2.A4 (MII1_RX_DV): now also R125.1
Other:
- note added: "Config: ------ MACIF_SEL: 0b00 => RMII MS_SEL2: 0b0 => Prefer Slave TX2P4: 0b0 => Enable 1.0V and 2.4V TX SWPD_ENB: 0b1 => Do not enter power down"

Commit message: Assigning Footprints
Parts:
- added C265: 8p2, Capacitor_SMD:C_0603_1608Metric, symbol Device:C
- added C266: 10p, Capacitor_SMD:C_0603_1608Metric, symbol Device:C
- D23: footprint (none) -> Diode_SMD:D_SOD-323
- D24, D25: footprint (none) -> UCLAMP3311P:SLP1006P2
- FB13: footprint Inductor_SMD:L_0805_2012Metric -> Inductor_SMD:L_1206_3216Metric
- H5: footprint (none) -> MountingHole:MountingHole_3.2mm_M3_Pad_Via
- J6: footprint (none) -> TerminalBlock_RND:TerminalBlock_RND_205-00288_1x03_P5.08mm_Horizontal
- L15: footprint (none) -> PID75:PID75-251M
- L16, L17: footprint (none) -> ICI70CGI:ICI70CGI
Connections:
- net GND: now also C266.2
- net at R136.2: now also C265.1; no longer U9.8 (XTAL_I/CLK_IN)
- new net: C265.2, C266.1, U9.8 (XTAL_I/CLK_IN)
Other:
- note added: "1Vp-p attenuation"
Changed lines of the file:
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@@
   (junction (at 200.66 80.01) (diameter 0) (color 0 0 0 0)
   )
+  (junction (at 55.88 102.87) (diameter 0) (color 0 0 0 0)
+  )
   (junction (at 147.32 109.22) (diameter 0) (color 0 0 0 0)
   )
@@
     (stroke (width 0) (type default) (color 0 0 0 0))
   )
+  (wire (pts (xy 55.88 83.82) (xy 55.88 95.25))
+    (stroke (width 0) (type default) (color 0 0 0 0))
+  )
   (wire (pts (xy 262.89 72.39) (xy 259.08 72.39))
     (stroke (width 0) (type default) (color 0 0 0 0))
@@
     (stroke (width 0) (type default) (color 0 0 0 0))
   )
-  (wire (pts (xy 68.58 83.82) (xy 68.58 106.68))
-    (stroke (width 0) (type default) (color 0 0 0 0))
-  )
   (wire (pts (xy 49.53 54.61) (xy 49.53 52.07))
     (stroke (width 0) (type default) (color 0 0 0 0))
@@
     (stroke (width 0) (type default) (color 0 0 0 0))
   )
+  (wire (pts (xy 55.88 102.87) (xy 68.58 102.87))
+    (stroke (width 0) (type default) (color 0 0 0 0))
+  )
   (wire (pts (xy 68.58 132.08) (xy 77.47 132.08))
     (stroke (width 0) (type default) (color 0 0 0 0))
@@
     (stroke (width 0) (type default) (color 0 0 0 0))
   )
+  (wire (pts (xy 68.58 102.87) (xy 68.58 106.68))
+    (stroke (width 0) (type default) (color 0 0 0 0))
+  )
   (wire (pts (xy 154.94 109.22) (xy 147.32 109.22))
     (stroke (width 0) (type default) (color 0 0 0 0))
@@
     (stroke (width 0) (type default) (color 0 0 0 0))
   )
-  (wire (pts (xy 49.53 83.82) (xy 68.58 83.82))
+  (wire (pts (xy 49.53 83.82) (xy 55.88 83.82))
     (stroke (width 0) (type default) (color 0 0 0 0))
   )
@@
   )
   (text "DNP" (at 176.53 57.15 0)
+    (effects (font (size 1.27 1.27)) (justify left bottom))
+  )
+  (text "1Vp-p\nattenuation" (at 60.96 101.6 0)
     (effects (font (size 1.27 1.27)) (justify left bottom))
   )
@@
     (property "Reference" "L17" (id 0) (at 224.79 66.675 0))
     (property "Value" "RCM70CGI-471" (id 1) (at 224.79 77.47 0))
-    (property "Footprint" "" (id 2) (at 224.79 71.12 0)
-      (effects (font (size 1.27 1.27)) hide)
-    )
-    (property "Datasheet" "~" (id 3) (at 224.79 71.12 0)
+    (property "Footprint" "ICI70CGI:ICI70CGI" (id 2) (at 224.79 71.12 0)
+      (effects (font (size 1.27 1.27)) hide)
+    )
+    (property "Datasheet" "https://product.tdk.com/system/files/dam/doc/product/transformer/transformer/lan/data_sheet/30/ds/lan_mod/rcm70cgi.pdf" (id 3) (at 224.79 71.12 0)
       (effects (font (size 1.27 1.27)) hide)
     )
@@
     (property "Reference" "D25" (id 0) (at 168.91 93.98 0))
     (property "Value" "UCLAMP3311P" (id 1) (at 180.34 93.98 90))
-    (property "Footprint" "" (id 2) (at 171.45 93.98 0)
+    (property "Footprint" "UCLAMP3311P:SLP1006P2" (id 2) (at 171.45 93.98 0)
       (effects (font (size 1.27 1.27)) hide)
     )
@@
     (pin "2")
   )
+  (symbol (lib_id "Device:C") (at 55.88 99.06 0) (unit 1)
+    (in_bom yes) (on_board yes)
+    (property "Reference" "C265" (id 0) (at 56.515 96.52 0)
+      (effects (font (size 1.27 1.27)) (justify left))
+    )
+    (property "Value" "8p2" (id 1) (at 56.515 101.6 0)
+      (effects (font (size 1.27 1.27)) (justify left))
+    )
+    (property "Footprint" "Capacitor_SMD:C_0603_1608Metric" (id 2) (at 56.8452 102.87 0)
+      (effects (font (size 1.27 1.27)) hide)
+    )
+    (property "Datasheet" "~" (id 3) (at 55.88 99.06 0)
+      (effects (font (size 1.27 1.27)) hide)
+    )
+    (pin "1")
+    (pin "2")
+  )
   (symbol (lib_id "Device:R") (at 73.66 68.58 90) (unit 1)
     (in_bom yes) (on_board yes)
@@
     (property "Reference" "D23" (id 0) (at 248.92 71.12 0))
     (property "Value" "CDSOD323-T36SC" (id 1) (at 251.46 63.5 90))
-    (property "Footprint" "" (id 2) (at 251.46 71.12 0)
+    (property "Footprint" "Diode_SMD:D_SOD-323" (id 2) (at 251.46 71.12 0)
       (effects (font (size 1.27 1.27)) hide)
     )
@@
     (property "Reference" "H5" (id 0) (at 279.4 87.63 0))
     (property "Value" "CHASSIS_PE" (id 1) (at 277.495 87.63 0))
-    (property "Footprint" "" (id 2) (at 273.05 87.63 0)
+    (property "Footprint" "MountingHole:MountingHole_3.2mm_M3_Pad_Via" (id 2) (at 273.05 87.63 0)
       (effects (font (size 1.27 1.27)) hide)
     )
@@
     (property "Reference" "FB13" (id 0) (at 161.925 113.03 90))
     (property "Value" "FerriteBead" (id 1) (at 162.56 105.41 90))
-    (property "Footprint" "Inductor_SMD:L_0805_2012Metric" (id 2) (at 162.56 110.998 90)
+    (property "Footprint" "Inductor_SMD:L_1206_3216Metric" (id 2) (at 162.56 110.998 90)
       (effects (font (size 1.27 1.27)) hide)
     )
@@
     (property "Reference" "L16" (id 0) (at 192.405 71.12 0))
     (property "Value" "ICI70CGI-222" (id 1) (at 179.07 71.12 90))
-    (property "Footprint" "" (id 2) (at 187.96 71.12 0)
-      (effects (font (size 1.27 1.27)) hide)
-    )
-    (property "Datasheet" "~" (id 3) (at 187.96 71.12 0)
+    (property "Footprint" "ICI70CGI:ICI70CGI" (id 2) (at 187.96 71.12 0)
+      (effects (font (size 1.27 1.27)) hide)
+    )
+    (property "Datasheet" "https://product.tdk.com/system/files/dam/doc/product/transformer/transformer/lan/data_sheet/30/ds/lan_mod/ici70cgi.pdf" (id 3) (at 187.96 71.12 0)
       (effects (font (size 1.27 1.27)) hide)
     )
@@
     (property "Reference" "D24" (id 0) (at 163.83 93.98 0))
     (property "Value" "UCLAMP3311P" (id 1) (at 156.21 93.98 90))
-    (property "Footprint" "" (id 2) (at 166.37 93.98 0)
+    (property "Footprint" "UCLAMP3311P:SLP1006P2" (id 2) (at 166.37 93.98 0)
       (effects (font (size 1.27 1.27)) hide)
     )
@@
     (property "Reference" "J6" (id 0) (at 267.97 67.31 0))
     (property "Value" "PHY5_MDI" (id 1) (at 267.97 77.47 0))
-    (property "Footprint" "" (id 2) (at 267.97 72.39 0)
+    (property "Footprint" "TerminalBlock_RND:TerminalBlock_RND_205-00288_1x03_P5.08mm_Horizontal" (id 2) (at 267.97 72.39 0)
       (effects (font (size 1.27 1.27)) hide)
     )
@@
     (property "Reference" "L15" (id 0) (at 230.505 53.34 0))
     (property "Value" "PID75-251M" (id 1) (at 239.395 53.34 0))
-    (property "Footprint" "" (id 2) (at 234.95 53.34 0)
-      (effects (font (size 1.27 1.27)) hide)
-    )
-    (property "Datasheet" "~" (id 3) (at 234.95 53.34 0)
+    (property "Footprint" "PID75:PID75-251M" (id 2) (at 234.95 53.34 0)
+      (effects (font (size 1.27 1.27)) hide)
+    )
+    (property "Datasheet" "https://product.tdk.com/system/files/dam/doc/product/inductor/inductor/smd/data_sheet/30/db/ind_2008/pidx251m.pdf" (id 3) (at 234.95 53.34 0)
       (effects (font (size 1.27 1.27)) hide)
     )
@@
     (pin "2")
   )
+  (symbol (lib_id "power:GND") (at 55.88 110.49 0) (unit 1)
+    (in_bom yes) (on_board yes)
+    (property "Reference" "#PWR0252" (id 0) (at 55.88 116.84 0)
+      (effects (font (size 1.27 1.27)) hide)
+    )
+    (property "Value" "GND" (id 1) (at 55.88 114.3 0))
+    (property "Footprint" "" (id 2) (at 55.88 110.49 0)
+      (effects (font (size 1.27 1.27)) hide)
+    )
+    (property "Datasheet" "" (id 3) (at 55.88 110.49 0)
+      (effects (font (size 1.27 1.27)) hide)
+    )
+    (pin "1")
+  )
   (symbol (lib_id "Device:R") (at 154.94 73.66 90) (unit 1)
     (in_bom yes) (on_board yes)
@@
       (effects (font (size 1.27 1.27)) hide)
     )
+    (pin "1")
+    (pin "2")
+  )
+  (symbol (lib_id "Device:C") (at 55.88 106.68 0) (unit 1)
+    (in_bom yes) (on_board yes)
+    (property "Reference" "C266" (id 0) (at 56.515 104.14 0)
+      (effects (font (size 1.27 1.27)) (justify left))
+    )
+    (property "Value" "10p" (id 1) (at 56.515 109.22 0)
+      (effects (font (size 1.27 1.27)) (justify left))
+    )
+    (property "Footprint" "Capacitor_SMD:C_0603_1608Metric" (id 2) (at 56.8452 110.49 0)
+      (effects (font (size 1.27 1.27)) hide)
+    )
+    (property "Datasheet" "~" (id 3) (at 55.88 106.68 0)
+      (effects (font (size 1.27 1.27)) hide)
+    )
