File: PoDL_PHY0-1.kicad_sch (KiCad schematic)
At the start: 45 parts, among them Q1 DMG3414U, Q10 DMG3414U, Q11 DMG3414U, Q12 MMBT3904, Q2 MMBTA06, Q3 MMBT3904, Q4 DMG3414U, Q5 DMG3414U, Q6 MMBT3904, Q7 DMG3414U, Q8 MMBTA06, Q9 MMBT3904, U14 LTC4296-1

Commit message: Minor corrections
Parts:
- renumbered R217 to R224, R218 to R225, R219 to R226, R220 to R227, R221 to R228, R222 to R229, R223 to R230, R224 to R231, R225 to R232, R226 to R233, R227 to R234, R228 to R235, R229 to R236, R230 to R237, R231 to R238, R232 to R239, R233 to R240, R234 to R241
Changed lines of the file:
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@@
   (symbol (lib_id "Device:R") (at 63.5 143.51 90) (unit 1)
     (in_bom yes) (on_board yes)
-    (property "Reference" "R232" (id 0) (at 63.5 141.478 90))
+    (property "Reference" "R239" (id 0) (at 63.5 141.478 90))
     (property "Value" "10K" (id 1) (at 63.5 143.51 90))
     (property "Footprint" "Resistor_SMD:R_0603_1608Metric" (id 2) (at 63.5 145.288 90)
@@
   (symbol (lib_id "power:+24V") (at 62.23 26.67 0) (unit 1)
     (in_bom yes) (on_board yes)
-    (property "Reference" "#PWR0185" (id 0) (at 62.23 30.48 0)
+    (property "Reference" "#PWR0186" (id 0) (at 62.23 30.48 0)
       (effects (font (size 1.27 1.27)) hide)
     )
@@
   (symbol (lib_id "Device:R") (at 140.97 133.35 180) (unit 1)
     (in_bom yes) (on_board yes)
-    (property "Reference" "R230" (id 0) (at 138.938 133.35 90))
+    (property "Reference" "R237" (id 0) (at 138.938 133.35 90))
     (property "Value" "5K" (id 1) (at 140.97 133.35 90))
     (property "Footprint" "Resistor_SMD:R_0603_1608Metric" (id 2) (at 142.748 133.35 90)
@@
   (symbol (lib_id "Device:R") (at 180.34 123.19 180) (unit 1)
     (in_bom yes) (on_board yes)
-    (property "Reference" "R227" (id 0) (at 178.308 123.19 90))
+    (property "Reference" "R234" (id 0) (at 178.308 123.19 90))
     (property "Value" "50K" (id 1) (at 180.34 123.19 90))
     (property "Footprint" "Resistor_SMD:R_0603_1608Metric" (id 2) (at 182.118 123.19 90)
@@
       (effects (font (size 1.27 1.27)) hide)
     )
-    (property "Datasheet" "" (id 3) (at 29.21 25.4 0)
+    (property "Datasheet" "https://www.analog.com/media/en/technical-documentation/data-sheets/ltc4296-1.pdf" (id 3) (at 29.21 25.4 0)
       (effects (font (size 1.27 1.27)) hide)
     )
@@
   (symbol (lib_id "power:GND") (at 77.47 120.65 0) (unit 1)
     (in_bom yes) (on_board yes)
-    (property "Reference" "#PWR0191" (id 0) (at 77.47 127 0)
+    (property "Reference" "#PWR0192" (id 0) (at 77.47 127 0)
       (effects (font (size 1.27 1.27)) hide)
     )
@@
   (symbol (lib_id "power:GND") (at 156.21 138.43 0) (unit 1)
     (in_bom yes) (on_board yes)
-    (property "Reference" "#PWR0192" (id 0) (at 156.21 144.78 0)
+    (property "Reference" "#PWR0193" (id 0) (at 156.21 144.78 0)
       (effects (font (size 1.27 1.27)) hide)
     )
@@
   (symbol (lib_id "Device:R") (at 140.97 50.8 180) (unit 1)
     (in_bom yes) (on_board yes)
-    (property "Reference" "R221" (id 0) (at 138.938 50.8 90))
+    (property "Reference" "R228" (id 0) (at 138.938 50.8 90))
     (property "Value" "5K" (id 1) (at 140.97 50.8 90))
     (property "Footprint" "Resistor_SMD:R_0603_1608Metric" (id 2) (at 142.748 50.8 90)
@@
   (symbol (lib_id "Device:R") (at 86.36 153.67 0) (unit 1)
     (in_bom yes) (on_board yes)
-    (property "Reference" "R233" (id 0) (at 88.392 153.67 90))
+    (property "Reference" "R240" (id 0) (at 88.392 153.67 90))
     (property "Value" "5" (id 1) (at 86.36 153.67 90))
     (property "Footprint" "Resistor_SMD:R_1206_3216Metric" (id 2) (at 84.582 153.67 90)
@@
       (effects (font (size 1.27 1.27)) hide)
     )
-    (property "Datasheet" "" (id 3) (at 29.21 107.95 0)
+    (property "Datasheet" "https://www.analog.com/media/en/technical-documentation/data-sheets/ltc4296-1.pdf" (id 3) (at 29.21 107.95 0)
       (effects (font (size 1.27 1.27)) hide)
     )
@@
   (symbol (lib_id "Device:R") (at 62.23 116.84 0) (unit 1)
     (in_bom yes) (on_board yes)
-    (property "Reference" "R226" (id 0) (at 64.262 116.84 90))
+    (property "Reference" "R233" (id 0) (at 64.262 116.84 90))
     (property "Value" "0R24" (id 1) (at 62.23 116.84 90))
     (property "Footprint" "Resistor_SMD:R_1206_3216Metric" (id 2) (at 60.452 116.84 90)
@@
   (symbol (lib_id "Device:R") (at 156.21 50.8 0) (unit 1)
     (in_bom yes) (on_board yes)
-    (property "Reference" "R222" (id 0) (at 158.242 50.8 90))
+    (property "Reference" "R229" (id 0) (at 158.242 50.8 90))
     (property "Value" "5" (id 1) (at 156.21 50.8 90))
     (property "Footprint" "Resistor_SMD:R_1206_3216Metric" (id 2) (at 154.432 50.8 90)
@@
   (symbol (lib_id "Device:R") (at 58.42 82.55 90) (unit 1)
     (in_bom yes) (on_board yes)
-    (property "Reference" "R225" (id 0) (at 58.42 80.518 90))
+    (property "Reference" "R232" (id 0) (at 58.42 80.518 90))
     (property "Value" "0R062" (id 1) (at 58.42 85.09 90))
     (property "Footprint" "Resistor_SMD:R_1206_3216Metric" (id 2) (at 58.42 84.328 90)
@@
   (symbol (lib_id "Device:R") (at 58.42 165.1 90) (unit 1)
     (in_bom yes) (on_board yes)
-    (property "Reference" "R234" (id 0) (at 58.42 163.068 90))
+    (property "Reference" "R241" (id 0) (at 58.42 163.068 90))
     (property "Value" "0R062" (id 1) (at 58.42 167.64 90))
     (property "Footprint" "Resistor_SMD:R_1206_3216Metric" (id 2) (at 58.42 166.878 90)
@@
   (symbol (lib_id "Device:R") (at 86.36 124.46 0) (unit 1)
     (in_bom yes) (on_board yes)
-    (property "Reference" "R228" (id 0) (at 88.392 124.46 90))
+    (property "Reference" "R235" (id 0) (at 88.392 124.46 90))
     (property "Value" "20" (id 1) (at 86.36 124.46 90))
     (property "Footprint" "Resistor_SMD:R_1206_3216Metric" (id 2) (at 84.582 124.46 90)
@@
   (symbol (lib_id "Device:R") (at 105.41 41.91 0) (unit 1)
     (in_bom yes) (on_board yes)
-    (property "Reference" "R220" (id 0) (at 107.442 41.91 90))
+    (property "Reference" "R227" (id 0) (at 107.442 41.91 90))
     (property "Value" "50" (id 1) (at 105.41 41.91 90))
     (property "Footprint" "Resistor_SMD:R_1206_3216Metric" (id 2) (at 103.632 41.91 90)
@@
   (symbol (lib_id "power:+24V") (at 62.23 109.22 0) (unit 1)
     (in_bom yes) (on_board yes)
-    (property "Reference" "#PWR0189" (id 0) (at 62.23 113.03 0)
+    (property "Reference" "#PWR0190" (id 0) (at 62.23 113.03 0)
       (effects (font (size 1.27 1.27)) hide)
     )
@@
   (symbol (lib_id "power:GND") (at 77.47 38.1 0) (unit 1)
     (in_bom yes) (on_board yes)
-    (property "Reference" "#PWR0187" (id 0) (at 77.47 44.45 0)
+    (property "Reference" "#PWR0188" (id 0) (at 77.47 44.45 0)
       (effects (font (size 1.27 1.27)) hide)
     )
@@
   (symbol (lib_id "Device:R") (at 63.5 60.96 90) (unit 1)
     (in_bom yes) (on_board yes)
-    (property "Reference" "R223" (id 0) (at 63.5 58.928 90))
+    (property "Reference" "R230" (id 0) (at 63.5 58.928 90))
     (property "Value" "10K" (id 1) (at 63.5 60.96 90))
     (property "Footprint" "Resistor_SMD:R_0603_1608Metric" (id 2) (at 63.5 62.738 90)
@@
   (symbol (lib_id "power:+3V3") (at 173.99 116.84 0) (unit 1)
     (in_bom yes) (on_board yes)
-    (property "Reference" "#PWR0190" (id 0) (at 173.99 120.65 0)
+    (property "Reference" "#PWR0191" (id 0) (at 173.99 120.65 0)
       (effects (font (size 1.27 1.27)) hide)
     )
@@
   (symbol (lib_id "Device:R") (at 156.21 133.35 0) (unit 1)
     (in_bom yes) (on_board yes)
-    (property "Reference" "R231" (id 0) (at 158.242 133.35 90))
+    (property "Reference" "R238" (id 0) (at 158.242 133.35 90))
     (property "Value" "5" (id 1) (at 156.21 133.35 90))
     (property "Footprint" "Resistor_SMD:R_1206_3216Metric" (id 2) (at 154.432 133.35 90)
@@
   (symbol (lib_id "power:GND") (at 156.21 55.88 0) (unit 1)
     (in_bom yes) (on_board yes)
-    (property "Reference" "#PWR0188" (id 0) (at 156.21 62.23 0)
+    (property "Reference" "#PWR0189" (id 0) (at 156.21 62.23 0)
       (effects (font (size 1.27 1.27)) hide)
     )
@@
   (symbol (lib_id "Device:R") (at 180.34 40.64 180) (unit 1)
     (in_bom yes) (on_board yes)
-    (property "Reference" "R218" (id 0) (at 178.308 40.64 90))
+    (property "Reference" "R225" (id 0) (at 178.308 40.64 90))
     (property "Value" "50K" (id 1) (at 180.34 40.64 90))
     (property "Footprint" "Resistor_SMD:R_0603_1608Metric" (id 2) (at 182.118 40.64 90)
@@
   (symbol (lib_id "Device:R") (at 86.36 41.91 0) (unit 1)
     (in_bom yes) (on_board yes)
-    (property "Reference" "R219" (id 0) (at 88.392 41.91 90))
+    (property "Reference" "R226" (id 0) (at 88.392 41.91 90))
     (property "Value" "20" (id 1) (at 86.36 41.91 90))
     (property "Footprint" "Resistor_SMD:R_1206_3216Metric" (id 2) (at 84.582 41.91 90)
@@
   (symbol (lib_id "Device:R") (at 62.23 34.29 0) (unit 1)
     (in_bom yes) (on_board yes)
-    (property "Reference" "R217" (id 0) (at 64.262 34.29 90))
+    (property "Reference" "R224" (id 0) (at 64.262 34.29 90))
     (property "Value" "0R24" (id 1) (at 62.23 34.29 90))
     (property "Footprint" "Resistor_SMD:R_1206_3216Metric" (id 2) (at 60.452 34.29 90)
@@
   (symbol (lib_id "Device:R") (at 105.41 124.46 0) (unit 1)
     (in_bom yes) (on_board yes)
-    (property "Reference" "R229" (id 0) (at 107.442 124.46 90))
+    (property "Reference" "R236" (id 0) (at 107.442 124.46 90))
     (property "Value" "50" (id 1) (at 105.41 124.46 90))
     (property "Footprint" "Resistor_SMD:R_1206_3216Metric" (id 2) (at 103.632 124.46 90)
@@
   (symbol (lib_id "Device:R") (at 86.36 71.12 0) (unit 1)
     (in_bom yes) (on_board yes)
-    (property "Reference" "R224" (id 0) (at 88.392 71.12 90))
+    (property "Reference" "R231" (id 0) (at 88.392 71.12 90))
     (property "Value" "5" (id 1) (at 86.36 71.12 90))
     (property "Footprint" "Resistor_SMD:R_1206_3216Metric" (id 2) (at 84.582 71.12 90)
@@
   (symbol (lib_id "power:+3V3") (at 173.99 34.29 0) (unit 1)
     (in_bom yes) (on_board yes)
-    (property "Reference" "#PWR0186" (id 0) (at 173.99 38.1 0)
-      (effects (font (size 1.27 1.27)) hide)
-    )
+    (property "Reference" "#PWR0187" (id 0) (at 173.99 38.1 0)
+      (effects (font (size 1.27 1.27)) hide)
+    )

Commit message: Assigning Footprints
Parts:
- C192, C193, C196, C197: footprint (none) -> Capacitor_SMD:C_0603_1608Metric
- Q1, Q10, Q11, Q12, Q2, Q3, Q4, Q5, Q6, Q7, Q8, Q9: footprint (none) -> Package_TO_SOT_SMD:SOT-23
- U14: footprint (none) -> Package_DFN_QFN:QFN-48-1EP_7x7mm_P0.5mm_EP5.3x5.3mm_ThermalVias
Changed lines of the file:
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@@
       (effects (font (size 1.27 1.27)) (justify left))
     )
-    (property "Footprint" "" (id 2) (at 106.3752 38.1 0)
+    (property "Footprint" "Capacitor_SMD:C_0603_1608Metric" (id 2) (at 106.3752 38.1 0)
       (effects (font (size 1.27 1.27)) hide)
     )
@@
       (effects (font (size 1.27 1.27)) (justify left))
     )
-    (property "Footprint" "" (id 2) (at 29.21 25.4 0)
+    (property "Footprint" "Package_DFN_QFN:QFN-48-1EP_7x7mm_P0.5mm_EP5.3x5.3mm_ThermalVias" (id 2) (at 29.21 25.4 0)
       (effects (font (size 1.27 1.27)) hide)
     )
@@
       (effects (font (size 1.27 1.27)) (justify left))
     )
-    (property "Footprint" "" (id 2) (at 76.2 147.32 0)
+    (property "Footprint" "Package_TO_SOT_SMD:SOT-23" (id 2) (at 76.2 147.32 0)
       (effects (font (size 1.27 1.27)) hide)
     )
@@
       (effects (font (size 1.27 1.27)) (justify left))
     )
-    (property "Footprint" "" (id 2) (at 146.05 44.45 0)
+    (property "Footprint" "Package_TO_SOT_SMD:SOT-23" (id 2) (at 146.05 44.45 0)
       (effects (font (size 1.27 1.27)) hide)
     )
@@
       (effects (font (size 1.27 1.27)) (justify left))
     )
-    (property "Footprint" "" (id 2) (at 29.21 107.95 0)
+    (property "Footprint" "Package_DFN_QFN:QFN-48-1EP_7x7mm_P0.5mm_EP5.3x5.3mm_ThermalVias" (id 2) (at 29.21 107.95 0)
       (effects (font (size 1.27 1.27)) hide)
     )
@@
       (effects (font (size 1.27 1.27)) (justify left))
     )
-    (property "Footprint" "" (id 2) (at 87.3252 120.65 0)
+    (property "Footprint" "Capacitor_SMD:C_0603_1608Metric" (id 2) (at 87.3252 120.65 0)
       (effects (font (size 1.27 1.27)) hide)
     )
@@
       (effects (font (size 1.27 1.27)) (justify left))
     )
-    (property "Footprint" "" (id 2) (at 87.3252 38.1 0)
+    (property "Footprint" "Capacitor_SMD:C_0603_1608Metric" (id 2) (at 87.3252 38.1 0)
       (effects (font (size 1.27 1.27)) hide)
     )
@@
       (effects (font (size 1.27 1.27)) (justify left))
     )
-    (property "Footprint" "" (id 2) (at 88.9 140.97 0)
+    (property "Footprint" "Package_TO_SOT_SMD:SOT-23" (id 2) (at 88.9 140.97 0)
       (effects (font (size 1.27 1.27)) hide)
     )
@@
       (effects (font (size 1.27 1.27)) (justify left))
     )
-    (property "Footprint" "" (id 2) (at 76.2 64.77 0)
+    (property "Footprint" "Package_TO_SOT_SMD:SOT-23" (id 2) (at 76.2 64.77 0)
       (effects (font (size 1.27 1.27)) hide)
     )
@@
       (effects (font (size 1.27 1.27)) (justify left))
     )
-    (property "Footprint" "" (id 2) (at 88.9 58.42 0)
+    (property "Footprint" "Package_TO_SOT_SMD:SOT-23" (id 2) (at 88.9 58.42 0)
       (effects (font (size 1.27 1.27)) hide)
     )
@@
       (effects (font (size 1.27 1.27)) (justify left))
     )
-    (property "Footprint" "" (id 2) (at 146.05 127 0)
+    (property "Footprint" "Package_TO_SOT_SMD:SOT-23" (id 2) (at 146.05 127 0)
       (effects (font (size 1.27 1.27)) hide)
     )
@@
       (effects (font (size 1.27 1.27)) (justify left))
     )
-    (property "Footprint" "" (id 2) (at 106.3752 120.65 0)
+    (property "Footprint" "Capacitor_SMD:C_0603_1608Metric" (id 2) (at 106.3752 120.65 0)
       (effects (font (size 1.27 1.27)) hide)
     )
@@
       (effects (font (size 1.27 1.27)) (justify left))
     )
-    (property "Footprint" "" (id 2) (at 158.75 38.1 0)
+    (property "Footprint" "Package_TO_SOT_SMD:SOT-23" (id 2) (at 158.75 38.1 0)
       (effects (font (size 1.27 1.27)) hide)
     )
@@
       (effects (font (size 1.27 1.27)) (justify left))
     )
-    (property "Footprint" "" (id 2) (at 64.77 45.72 0)
+    (property "Footprint" "Package_TO_SOT_SMD:SOT-23" (id 2) (at 64.77 45.72 0)
       (effects (font (size 1.27 1.27)) hide)
     )
@@
       (effects (font (size 1.27 1.27)) (justify left))
     )
-    (property "Footprint" "" (id 2) (at 64.77 128.27 0)
+    (property "Footprint" "Package_TO_SOT_SMD:SOT-23" (id 2) (at 64.77 128.27 0)
       (effects (font (size 1.27 1.27)) hide)
     )
@@
       (effects (font (size 1.27 1.27)) (justify left))
     )
-    (property "Footprint" "" (id 2) (at 158.75 120.65 0)
+    (property "Footprint" "Package_TO_SOT_SMD:SOT-23" (id 2) (at 158.75 120.65 0)
       (effects (font (size 1.27 1.27)) hide)
     )
@@
       (effects (font (size 1.27 1.27)) (justify left))
     )
-    (property "Footprint" "" (id 2) (at 191.77 43.18 0)
+    (property "Footprint" "Package_TO_SOT_SMD:SOT-23" (id 2) (at 191.77 43.18 0)
       (effects (font (size 1.27 1.27)) hide)
     )
@@
       (effects (font (size 1.27 1.27)) (justify left))
     )
-    (property "Footprint" "" (id 2) (at 191.77 125.73 0)
-      (effects (font (size 1.27 1.27)) hide)
-    )
+    (property "Footprint" "Package_TO_SOT_SMD:SOT-23" (id 2) (at 191.77 125.73 0)
+      (effects (font (size 1.27 1.27)) hide)
+    )
