File: PoDL_PHY2-3.kicad_sch (KiCad schematic)
At the start: 45 parts, among them Q13 DMG3414U, Q14 MMBTA06, Q15 MMBT3904, Q16 DMG3414U, Q17 DMG3414U, Q18 MMBT3904, Q19 DMG3414U, Q20 MMBTA06, Q21 MMBT3904, Q22 DMG3414U, Q23 DMG3414U, Q24 MMBT3904, U14 LTC4296-1

Commit message: Minor corrections
Parts:
- renumbered R235 to R242, R236 to R243, R237 to R244, R238 to R245, R239 to R246, R240 to R247, R241 to R248, R242 to R249, R243 to R250, R244 to R251, R245 to R252, R246 to R253, R247 to R254, R248 to R255, R249 to R256, R250 to R257, R251 to R258, R252 to R259
Connections:
- net REG0_LSNS23 renamed REG0_LSNS34

Commit message: Assigning Footprints
Parts:
- C200, C201, C204, C205: footprint (none) -> Capacitor_SMD:C_0603_1608Metric
- Q13, Q14, Q15, Q16, Q17, Q18, Q19, Q20, Q21, Q22, Q23, Q24: footprint (none) -> Package_TO_SOT_SMD:SOT-23
- U14: footprint (none) -> Package_DFN_QFN:QFN-48-1EP_7x7mm_P0.5mm_EP5.3x5.3mm_ThermalVias
Changed lines of the file:
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@@
       (effects (font (size 1.27 1.27)) (justify left))
     )
-    (property "Footprint" "" (id 2) (at 158.75 38.1 0)
+    (property "Footprint" "Package_TO_SOT_SMD:SOT-23" (id 2) (at 158.75 38.1 0)
       (effects (font (size 1.27 1.27)) hide)
     )
@@
       (effects (font (size 1.27 1.27)) (justify left))
     )
-    (property "Footprint" "" (id 2) (at 87.3252 38.1 0)
+    (property "Footprint" "Capacitor_SMD:C_0603_1608Metric" (id 2) (at 87.3252 38.1 0)
       (effects (font (size 1.27 1.27)) hide)
     )
@@
       (effects (font (size 1.27 1.27)) (justify left))
     )
-    (property "Footprint" "" (id 2) (at 76.2 64.77 0)
+    (property "Footprint" "Package_TO_SOT_SMD:SOT-23" (id 2) (at 76.2 64.77 0)
       (effects (font (size 1.27 1.27)) hide)
     )
@@
       (effects (font (size 1.27 1.27)) (justify left))
     )
-    (property "Footprint" "" (id 2) (at 87.3252 120.65 0)
+    (property "Footprint" "Capacitor_SMD:C_0603_1608Metric" (id 2) (at 87.3252 120.65 0)
       (effects (font (size 1.27 1.27)) hide)
     )
@@
       (effects (font (size 1.27 1.27)) (justify left))
     )
-    (property "Footprint" "" (id 2) (at 191.77 43.18 0)
+    (property "Footprint" "Package_TO_SOT_SMD:SOT-23" (id 2) (at 191.77 43.18 0)
       (effects (font (size 1.27 1.27)) hide)
     )
@@
       (effects (font (size 1.27 1.27)) (justify left))
     )
-    (property "Footprint" "" (id 2) (at 106.3752 120.65 0)
+    (property "Footprint" "Capacitor_SMD:C_0603_1608Metric" (id 2) (at 106.3752 120.65 0)
       (effects (font (size 1.27 1.27)) hide)
     )
@@
       (effects (font (size 1.27 1.27)) (justify left))
     )
-    (property "Footprint" "" (id 2) (at 146.05 44.45 0)
+    (property "Footprint" "Package_TO_SOT_SMD:SOT-23" (id 2) (at 146.05 44.45 0)
       (effects (font (size 1.27 1.27)) hide)
     )
@@
       (effects (font (size 1.27 1.27)) (justify left))
     )
-    (property "Footprint" "" (id 2) (at 88.9 58.42 0)
+    (property "Footprint" "Package_TO_SOT_SMD:SOT-23" (id 2) (at 88.9 58.42 0)
       (effects (font (size 1.27 1.27)) hide)
     )
@@
       (effects (font (size 1.27 1.27)) (justify left))
     )
-    (property "Footprint" "" (id 2) (at 29.21 25.4 0)
+    (property "Footprint" "Package_DFN_QFN:QFN-48-1EP_7x7mm_P0.5mm_EP5.3x5.3mm_ThermalVias" (id 2) (at 29.21 25.4 0)
       (effects (font (size 1.27 1.27)) hide)
     )
@@
       (effects (font (size 1.27 1.27)) (justify left))
     )
-    (property "Footprint" "" (id 2) (at 191.77 125.73 0)
+    (property "Footprint" "Package_TO_SOT_SMD:SOT-23" (id 2) (at 191.77 125.73 0)
       (effects (font (size 1.27 1.27)) hide)
     )
@@
       (effects (font (size 1.27 1.27)) (justify left))
     )
-    (property "Footprint" "" (id 2) (at 88.9 140.97 0)
+    (property "Footprint" "Package_TO_SOT_SMD:SOT-23" (id 2) (at 88.9 140.97 0)
       (effects (font (size 1.27 1.27)) hide)
     )
@@
       (effects (font (size 1.27 1.27)) (justify left))
     )
-    (property "Footprint" "" (id 2) (at 76.2 147.32 0)
+    (property "Footprint" "Package_TO_SOT_SMD:SOT-23" (id 2) (at 76.2 147.32 0)
       (effects (font (size 1.27 1.27)) hide)
     )
@@
       (effects (font (size 1.27 1.27)) (justify left))
     )
-    (property "Footprint" "" (id 2) (at 64.77 45.72 0)
+    (property "Footprint" "Package_TO_SOT_SMD:SOT-23" (id 2) (at 64.77 45.72 0)
       (effects (font (size 1.27 1.27)) hide)
     )
@@
       (effects (font (size 1.27 1.27)) (justify left))
     )
-    (property "Footprint" "" (id 2) (at 64.77 128.27 0)
+    (property "Footprint" "Package_TO_SOT_SMD:SOT-23" (id 2) (at 64.77 128.27 0)
       (effects (font (size 1.27 1.27)) hide)
     )
@@
       (effects (font (size 1.27 1.27)) (justify left))
     )
-    (property "Footprint" "" (id 2) (at 106.3752 38.1 0)
+    (property "Footprint" "Capacitor_SMD:C_0603_1608Metric" (id 2) (at 106.3752 38.1 0)
       (effects (font (size 1.27 1.27)) hide)
     )
@@
       (effects (font (size 1.27 1.27)) (justify left))
     )
-    (property "Footprint" "" (id 2) (at 29.21 107.95 0)
+    (property "Footprint" "Package_DFN_QFN:QFN-48-1EP_7x7mm_P0.5mm_EP5.3x5.3mm_ThermalVias" (id 2) (at 29.21 107.95 0)
       (effects (font (size 1.27 1.27)) hide)
     )
@@
       (effects (font (size 1.27 1.27)) (justify left))
     )
-    (property "Footprint" "" (id 2) (at 146.05 127 0)
+    (property "Footprint" "Package_TO_SOT_SMD:SOT-23" (id 2) (at 146.05 127 0)
       (effects (font (size 1.27 1.27)) hide)
     )
@@
       (effects (font (size 1.27 1.27)) (justify left))
     )
-    (property "Footprint" "" (id 2) (at 158.75 120.65 0)
-      (effects (font (size 1.27 1.27)) hide)
-    )
+    (property "Footprint" "Package_TO_SOT_SMD:SOT-23" (id 2) (at 158.75 120.65 0)
+      (effects (font (size 1.27 1.27)) hide)
+    )
