File: PoDL_PHY4_REG0.kicad_sch (KiCad schematic)
At the start: 29 parts, among them Q25 DMG3414U, Q26 MMBTA06, Q27 MMBT3904, Q28 DMG3414U, Q29 DMG3414U, Q30 MMBT3904, Q31 SIS412DN, U14 LTC4296-1

Commit message: Minor corrections
Parts:
- removed Q31: SIS412DN, Package_SO:Vishay_PowerPAK_1212-8_Single, symbol Transistor_FET:SiS415DNT
- added Q31: SiS412DN, Package_SO:Vishay_PowerPAK_1212-8_Single, symbol Transistor_FET:SiS454DN
- renumbered R253 to R260, R254 to R261, R255 to R262, R256 to R263, R257 to R264, R258 to R265, R259 to R266, R260 to R267, R261 to R268, R262 to R269, R263 to R270
Connections:
- net GND: now also Q31.1 (S), Q31.2 (S), Q31.3 (S)
- net REG0_LSNS0: now also Q31.5 (D)
- net at U14.23 (LGATE): now also Q31.4 (G)

Commit message: Assigning Footprints
Parts:
- C208, C209: footprint (none) -> Capacitor_SMD:C_0603_1608Metric
- Q25, Q26, Q27, Q28, Q29, Q30: footprint (none) -> Package_TO_SOT_SMD:SOT-23
- U14: footprint (none) -> Package_DFN_QFN:QFN-48-1EP_7x7mm_P0.5mm_EP5.3x5.3mm_ThermalVias
Changed lines of the file:
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@@
       (effects (font (size 1.27 1.27)) (justify left))
     )
-    (property "Footprint" "" (id 2) (at 87.3252 38.1 0)
+    (property "Footprint" "Capacitor_SMD:C_0603_1608Metric" (id 2) (at 87.3252 38.1 0)
       (effects (font (size 1.27 1.27)) hide)
     )
@@
       (effects (font (size 1.27 1.27)) (justify left))
     )
-    (property "Footprint" "" (id 2) (at 76.2 64.77 0)
+    (property "Footprint" "Package_TO_SOT_SMD:SOT-23" (id 2) (at 76.2 64.77 0)
       (effects (font (size 1.27 1.27)) hide)
     )
@@
       (effects (font (size 1.27 1.27)) (justify left))
     )
-    (property "Footprint" "" (id 2) (at 193.04 77.47 0)
+    (property "Footprint" "Package_DFN_QFN:QFN-48-1EP_7x7mm_P0.5mm_EP5.3x5.3mm_ThermalVias" (id 2) (at 193.04 77.47 0)
       (effects (font (size 1.27 1.27)) hide)
     )
@@
       (effects (font (size 1.27 1.27)) (justify left))
     )
-    (property "Footprint" "" (id 2) (at 158.75 38.1 0)
+    (property "Footprint" "Package_TO_SOT_SMD:SOT-23" (id 2) (at 158.75 38.1 0)
       (effects (font (size 1.27 1.27)) hide)
     )
@@
       (effects (font (size 1.27 1.27)) (justify left))
     )
-    (property "Footprint" "" (id 2) (at 106.3752 38.1 0)
+    (property "Footprint" "Capacitor_SMD:C_0603_1608Metric" (id 2) (at 106.3752 38.1 0)
       (effects (font (size 1.27 1.27)) hide)
     )
@@
       (effects (font (size 1.27 1.27) italic) (justify left) hide)
     )
-    (property "Datasheet" "https://www.vishay.com/docs/66707/sis454dn.pdf" (id 3) (at 187.96 138.43 0)
+    (property "Datasheet" "~" (id 3) (at 187.96 138.43 0)
       (effects (font (size 1.27 1.27)) (justify left) hide)
     )
@@
       (effects (font (size 1.27 1.27)) (justify left))
     )
-    (property "Footprint" "" (id 2) (at 146.05 44.45 0)
+    (property "Footprint" "Package_TO_SOT_SMD:SOT-23" (id 2) (at 146.05 44.45 0)
       (effects (font (size 1.27 1.27)) hide)
     )
@@
       (effects (font (size 1.27 1.27)) (justify left))
     )
-    (property "Footprint" "" (id 2) (at 64.77 45.72 0)
+    (property "Footprint" "Package_TO_SOT_SMD:SOT-23" (id 2) (at 64.77 45.72 0)
       (effects (font (size 1.27 1.27)) hide)
     )
@@
       (effects (font (size 1.27 1.27)) (justify left))
     )
-    (property "Footprint" "" (id 2) (at 191.77 43.18 0)
+    (property "Footprint" "Package_TO_SOT_SMD:SOT-23" (id 2) (at 191.77 43.18 0)
       (effects (font (size 1.27 1.27)) hide)
     )
@@
       (effects (font (size 1.27 1.27)) (justify left))
     )
-    (property "Footprint" "" (id 2) (at 29.21 25.4 0)
+    (property "Footprint" "Package_DFN_QFN:QFN-48-1EP_7x7mm_P0.5mm_EP5.3x5.3mm_ThermalVias" (id 2) (at 29.21 25.4 0)
       (effects (font (size 1.27 1.27)) hide)
     )
@@
       (effects (font (size 1.27 1.27)) (justify left))
     )
-    (property "Footprint" "" (id 2) (at 88.9 58.42 0)
-      (effects (font (size 1.27 1.27)) hide)
-    )
+    (property "Footprint" "Package_TO_SOT_SMD:SOT-23" (id 2) (at 88.9 58.42 0)
+      (effects (font (size 1.27 1.27)) hide)
+    )
