File: PoDL_PHY5-6.kicad_sch (KiCad schematic)
At the start: 45 parts, among them Q32 DMG3414U, Q33 MMBTA06, Q34 MMBT3904, Q35 DMG3414U, Q36 DMG3414U, Q37 MMBT3904, Q38 DMG3414U, Q39 MMBTA06, Q40 MMBT3904, Q41 DMG3414U, Q42 DMG3414U, Q43 MMBT3904, U15 LTC4296-1

Commit message: Minor corrections
Parts:
- renumbered R264 to R271, R265 to R272, R266 to R273, R267 to R274, R268 to R275, R269 to R276, R270 to R277, R271 to R278, R272 to R279, R273 to R280, R274 to R281, R275 to R282, R276 to R283, R277 to R284, R278 to R285, R279 to R286, R280 to R287, R281 to R288

Commit message: Assigning Footprints
Parts:
- C215, C216, C219, C220: footprint (none) -> Capacitor_SMD:C_0603_1608Metric
- Q32, Q33, Q34, Q35, Q36, Q37, Q38, Q39, Q40, Q41, Q42, Q43: footprint (none) -> Package_TO_SOT_SMD:SOT-23
- U15: footprint (none) -> Package_DFN_QFN:QFN-48-1EP_7x7mm_P0.5mm_EP5.3x5.3mm_ThermalVias
Changed lines of the file:
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@@
       (effects (font (size 1.27 1.27)) (justify left))
     )
-    (property "Footprint" "" (id 2) (at 106.3752 38.1 0)
+    (property "Footprint" "Capacitor_SMD:C_0603_1608Metric" (id 2) (at 106.3752 38.1 0)
       (effects (font (size 1.27 1.27)) hide)
     )
@@
       (effects (font (size 1.27 1.27)) (justify left))
     )
-    (property "Footprint" "" (id 2) (at 88.9 140.97 0)
+    (property "Footprint" "Package_TO_SOT_SMD:SOT-23" (id 2) (at 88.9 140.97 0)
       (effects (font (size 1.27 1.27)) hide)
     )
@@
       (effects (font (size 1.27 1.27)) (justify left))
     )
-    (property "Footprint" "" (id 2) (at 158.75 120.65 0)
+    (property "Footprint" "Package_TO_SOT_SMD:SOT-23" (id 2) (at 158.75 120.65 0)
       (effects (font (size 1.27 1.27)) hide)
     )
@@
       (effects (font (size 1.27 1.27)) (justify left))
     )
-    (property "Footprint" "" (id 2) (at 158.75 38.1 0)
+    (property "Footprint" "Package_TO_SOT_SMD:SOT-23" (id 2) (at 158.75 38.1 0)
       (effects (font (size 1.27 1.27)) hide)
     )
@@
       (effects (font (size 1.27 1.27)) (justify left))
     )
-    (property "Footprint" "" (id 2) (at 87.3252 38.1 0)
+    (property "Footprint" "Capacitor_SMD:C_0603_1608Metric" (id 2) (at 87.3252 38.1 0)
       (effects (font (size 1.27 1.27)) hide)
     )
@@
       (effects (font (size 1.27 1.27)) (justify left))
     )
-    (property "Footprint" "" (id 2) (at 146.05 44.45 0)
+    (property "Footprint" "Package_TO_SOT_SMD:SOT-23" (id 2) (at 146.05 44.45 0)
       (effects (font (size 1.27 1.27)) hide)
     )
@@
       (effects (font (size 1.27 1.27)) (justify left))
     )
-    (property "Footprint" "" (id 2) (at 146.05 127 0)
+    (property "Footprint" "Package_TO_SOT_SMD:SOT-23" (id 2) (at 146.05 127 0)
       (effects (font (size 1.27 1.27)) hide)
     )
@@
       (effects (font (size 1.27 1.27)) (justify left))
     )
-    (property "Footprint" "" (id 2) (at 29.21 25.4 0)
+    (property "Footprint" "Package_DFN_QFN:QFN-48-1EP_7x7mm_P0.5mm_EP5.3x5.3mm_ThermalVias" (id 2) (at 29.21 25.4 0)
       (effects (font (size 1.27 1.27)) hide)
     )
@@
       (effects (font (size 1.27 1.27)) (justify left))
     )
-    (property "Footprint" "" (id 2) (at 87.3252 120.65 0)
+    (property "Footprint" "Capacitor_SMD:C_0603_1608Metric" (id 2) (at 87.3252 120.65 0)
       (effects (font (size 1.27 1.27)) hide)
     )
@@
       (effects (font (size 1.27 1.27)) (justify left))
     )
-    (property "Footprint" "" (id 2) (at 64.77 45.72 0)
+    (property "Footprint" "Package_TO_SOT_SMD:SOT-23" (id 2) (at 64.77 45.72 0)
       (effects (font (size 1.27 1.27)) hide)
     )
@@
       (effects (font (size 1.27 1.27)) (justify left))
     )
-    (property "Footprint" "" (id 2) (at 106.3752 120.65 0)
+    (property "Footprint" "Capacitor_SMD:C_0603_1608Metric" (id 2) (at 106.3752 120.65 0)
       (effects (font (size 1.27 1.27)) hide)
     )
@@
       (effects (font (size 1.27 1.27)) (justify left))
     )
-    (property "Footprint" "" (id 2) (at 191.77 125.73 0)
+    (property "Footprint" "Package_TO_SOT_SMD:SOT-23" (id 2) (at 191.77 125.73 0)
       (effects (font (size 1.27 1.27)) hide)
     )
@@
       (effects (font (size 1.27 1.27)) (justify left))
     )
-    (property "Footprint" "" (id 2) (at 29.21 107.95 0)
+    (property "Footprint" "Package_DFN_QFN:QFN-48-1EP_7x7mm_P0.5mm_EP5.3x5.3mm_ThermalVias" (id 2) (at 29.21 107.95 0)
       (effects (font (size 1.27 1.27)) hide)
     )
@@
       (effects (font (size 1.27 1.27)) (justify left))
     )
-    (property "Footprint" "" (id 2) (at 191.77 43.18 0)
+    (property "Footprint" "Package_TO_SOT_SMD:SOT-23" (id 2) (at 191.77 43.18 0)
       (effects (font (size 1.27 1.27)) hide)
     )
@@
       (effects (font (size 1.27 1.27)) (justify left))
     )
-    (property "Footprint" "" (id 2) (at 64.77 128.27 0)
+    (property "Footprint" "Package_TO_SOT_SMD:SOT-23" (id 2) (at 64.77 128.27 0)
       (effects (font (size 1.27 1.27)) hide)
     )
@@
       (effects (font (size 1.27 1.27)) (justify left))
     )
-    (property "Footprint" "" (id 2) (at 88.9 58.42 0)
+    (property "Footprint" "Package_TO_SOT_SMD:SOT-23" (id 2) (at 88.9 58.42 0)
       (effects (font (size 1.27 1.27)) hide)
     )
@@
       (effects (font (size 1.27 1.27)) (justify left))
     )
-    (property "Footprint" "" (id 2) (at 76.2 64.77 0)
+    (property "Footprint" "Package_TO_SOT_SMD:SOT-23" (id 2) (at 76.2 64.77 0)
       (effects (font (size 1.27 1.27)) hide)
     )
@@
       (effects (font (size 1.27 1.27)) (justify left))
     )
-    (property "Footprint" "" (id 2) (at 76.2 147.32 0)
-      (effects (font (size 1.27 1.27)) hide)
-    )
+    (property "Footprint" "Package_TO_SOT_SMD:SOT-23" (id 2) (at 76.2 147.32 0)
+      (effects (font (size 1.27 1.27)) hide)
+    )
