File: PoDL_REG1.kicad_sch (KiCad schematic)
At the start: 7 parts, among them Q44 SIS412DN, U15 LTC4296-1

Commit message: Minor corrections
Parts:
- removed Q44: SIS412DN, Package_SO:Vishay_PowerPAK_1212-8_Single, symbol Transistor_FET:SiS415DNT
- added Q44: SiS412DN, Package_SO:Vishay_PowerPAK_1212-8_Single, symbol Transistor_FET:SiS454DN
- renumbered R282 to R289, R283 to R290
Connections:
- net GND: now also Q44.1 (S), Q44.2 (S), Q44.3 (S)
- net REG1_LSNS0: now also Q44.5 (D)
- net at U15.23 (LGATE): now also Q44.4 (G)
Changed lines of the file:
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@@
   (symbol (lib_id "power:+24V") (at 177.8 77.47 0) (unit 1)
     (in_bom yes) (on_board yes)
-    (property "Reference" "#PWR0216" (id 0) (at 177.8 81.28 0)
+    (property "Reference" "#PWR0217" (id 0) (at 177.8 81.28 0)
       (effects (font (size 1.27 1.27)) hide)
     )
@@
   (symbol (lib_id "power:GND") (at 228.6 99.06 0) (unit 1)
     (in_bom yes) (on_board yes)
-    (property "Reference" "#PWR0217" (id 0) (at 228.6 105.41 0)
+    (property "Reference" "#PWR0218" (id 0) (at 228.6 105.41 0)
       (effects (font (size 1.27 1.27)) hide)
     )
@@
   (symbol (lib_id "power:GND") (at 177.8 160.02 0) (unit 1)
     (in_bom yes) (on_board yes)
-    (property "Reference" "#PWR0218" (id 0) (at 177.8 166.37 0)
+    (property "Reference" "#PWR0219" (id 0) (at 177.8 166.37 0)
       (effects (font (size 1.27 1.27)) hide)
     )
@@
   (symbol (lib_id "Device:R") (at 187.96 151.13 90) (unit 1)
     (in_bom yes) (on_board yes)
-    (property "Reference" "R283" (id 0) (at 187.96 149.098 90))
+    (property "Reference" "R290" (id 0) (at 187.96 149.098 90))
     (property "Value" "49K9" (id 1) (at 187.96 151.13 90))
     (property "Footprint" "Resistor_SMD:R_0805_2012Metric" (id 2) (at 187.96 152.908 90)
@@
       (effects (font (size 1.27 1.27)) hide)
     )
-    (property "Datasheet" "" (id 3) (at 29.21 25.4 0)
+    (property "Datasheet" "https://www.analog.com/media/en/technical-documentation/data-sheets/ltc4296-1.pdf" (id 3) (at 29.21 25.4 0)
       (effects (font (size 1.27 1.27)) hide)
     )
@@
       (effects (font (size 1.27 1.27)) hide)
     )
-    (property "Datasheet" "" (id 3) (at 193.04 77.47 0)
+    (property "Datasheet" "https://www.analog.com/media/en/technical-documentation/data-sheets/ltc4296-1.pdf" (id 3) (at 193.04 77.47 0)
       (effects (font (size 1.27 1.27)) hide)
     )
@@
       (effects (font (size 1.27 1.27)) hide)
     )
-    (property "Datasheet" "" (id 3) (at 60.96 25.4 0)
+    (property "Datasheet" "https://www.analog.com/media/en/technical-documentation/data-sheets/ltc4296-1.pdf" (id 3) (at 60.96 25.4 0)
       (effects (font (size 1.27 1.27)) hide)
     )
@@
     (pin "9")
   )
+  (symbol (lib_id "Transistor_FET:SiS454DN") (at 187.96 138.43 270) (unit 1)
+    (in_bom yes) (on_board yes)
+    (property "Reference" "Q44" (id 0) (at 189.865 143.51 0)
+      (effects (font (size 1.27 1.27)) (justify left))
+    )
+    (property "Value" "SiS412DN" (id 1) (at 179.07 144.78 90)
+      (effects (font (size 1.27 1.27)) (justify left))
+    )
+    (property "Footprint" "Package_SO:Vishay_PowerPAK_1212-8_Single" (id 2) (at 186.055 143.51 0)
+      (effects (font (size 1.27 1.27) italic) (justify left) hide)
+    )
+    (property "Datasheet" "https://www.vishay.com/docs/66707/sis454dn.pdf" (id 3) (at 187.96 138.43 0)
+      (effects (font (size 1.27 1.27)) (justify left) hide)
+    )
+    (pin "1")
+    (pin "2")
+    (pin "3")
+    (pin "4")
+    (pin "5")
+  )
   (symbol (lib_id "Device:R") (at 177.8 109.22 0) (unit 1)
     (in_bom yes) (on_board yes)
-    (property "Reference" "R282" (id 0) (at 179.832 109.22 90))
+    (property "Reference" "R289" (id 0) (at 179.832 109.22 90))
     (property "Value" "24K3" (id 1) (at 177.8 109.22 90))
     (property "Footprint" "Resistor_SMD:R_0603_1608Metric" (id 2) (at 176.022 109.22 90)
@@
       (effects (font (size 1.27 1.27)) hide)
     )
-    (property "Datasheet" "" (id 3) (at 29.21 86.36 0)
+    (property "Datasheet" "https://www.analog.com/media/en/technical-documentation/data-sheets/ltc4296-1.pdf" (id 3) (at 29.21 86.36 0)
       (effects (font (size 1.27 1.27)) hide)
     )
@@
     (pin "9")
   )
-  (symbol (lib_id "Transistor_FET:SiS415DNT") (at 187.96 138.43 90) (mirror x) (unit 1)
-    (in_bom yes) (on_board yes)
-    (property "Reference" "Q44" (id 0) (at 186.055 143.51 0)
-      (effects (font (size 1.27 1.27)) (justify left))
-    )
-    (property "Value" "SIS412DN" (id 1) (at 200.66 137.16 90)
-      (effects (font (size 1.27 1.27)) (justify left))
-    )
-    (property "Footprint" "Package_SO:Vishay_PowerPAK_1212-8_Single" (id 2) (at 189.865 143.51 0)
-      (effects (font (size 1.27 1.27) italic) (justify left) hide)
-    )
-    (property "Datasheet" "https://www.vishay.com/docs/63684/sis415dnt.pdf" (id 3) (at 187.96 138.43 90)
-      (effects (font (size 1.27 1.27)) (justify left) hide)
-    )
-    (pin "1")
-    (pin "2")
-    (pin "3")
-    (pin "4")
-    (pin "5")
-  )
   (symbol (lib_id "Device:C") (at 187.96 157.48 90) (unit 1)

Commit message: Assigning Footprints
Parts:
- U15: footprint (none) -> Package_DFN_QFN:QFN-48-1EP_7x7mm_P0.5mm_EP5.3x5.3mm_ThermalVias
Changed lines of the file:
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@@
       (effects (font (size 1.27 1.27)) (justify left))
     )
-    (property "Footprint" "" (id 2) (at 29.21 25.4 0)
+    (property "Footprint" "Package_DFN_QFN:QFN-48-1EP_7x7mm_P0.5mm_EP5.3x5.3mm_ThermalVias" (id 2) (at 29.21 25.4 0)
       (effects (font (size 1.27 1.27)) hide)
     )
@@
       (effects (font (size 1.27 1.27)) (justify left))
     )
-    (property "Footprint" "" (id 2) (at 193.04 77.47 0)
+    (property "Footprint" "Package_DFN_QFN:QFN-48-1EP_7x7mm_P0.5mm_EP5.3x5.3mm_ThermalVias" (id 2) (at 193.04 77.47 0)
       (effects (font (size 1.27 1.27)) hide)
     )
@@
       (effects (font (size 1.27 1.27)) (justify left))
     )
-    (property "Footprint" "" (id 2) (at 60.96 25.4 0)
+    (property "Footprint" "Package_DFN_QFN:QFN-48-1EP_7x7mm_P0.5mm_EP5.3x5.3mm_ThermalVias" (id 2) (at 60.96 25.4 0)
       (effects (font (size 1.27 1.27)) hide)
     )
@@
       (effects (font (size 1.27 1.27) italic) (justify left) hide)
     )
-    (property "Datasheet" "https://www.vishay.com/docs/66707/sis454dn.pdf" (id 3) (at 187.96 138.43 0)
+    (property "Datasheet" "~" (id 3) (at 187.96 138.43 0)
       (effects (font (size 1.27 1.27)) (justify left) hide)
     )
@@
       (effects (font (size 1.27 1.27)) (justify left))
     )
-    (property "Footprint" "" (id 2) (at 29.21 86.36 0)
-      (effects (font (size 1.27 1.27)) hide)
-    )
+    (property "Footprint" "Package_DFN_QFN:QFN-48-1EP_7x7mm_P0.5mm_EP5.3x5.3mm_ThermalVias" (id 2) (at 29.21 86.36 0)
+      (effects (font (size 1.27 1.27)) hide)
+    )
