File: SJA1105Q_Power.kicad_sch (KiCad schematic)
At the start: 84 parts, among them U1 SJA1105Q, U2 SJA1105Q, U3 SC4626C, U4 SC4626C

Commit message: Assigning Footprints
Parts:
- FB1, FB2, FB3, FB4, FB5, FB6, FB7, FB8: value FerriteBead -> 782763301; footprint (none) -> Inductor_SMD:L_1206_3216Metric
Changed lines of the file:
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@@
     (in_bom yes) (on_board yes)
     (property "Reference" "FB1" (id 0) (at 26.035 31.75 90))
-    (property "Value" "FerriteBead" (id 1) (at 26.67 24.13 90))
-    (property "Footprint" "" (id 2) (at 26.67 29.718 90)
+    (property "Value" "782763301" (id 1) (at 26.67 24.13 90))
+    (property "Footprint" "Inductor_SMD:L_1206_3216Metric" (id 2) (at 26.67 29.718 90)
       (effects (font (size 1.27 1.27)) hide)
     )
@@
     (in_bom yes) (on_board yes)
     (property "Reference" "FB4" (id 0) (at 259.08 73.025 90))
-    (property "Value" "FerriteBead" (id 1) (at 251.46 72.39 90))
-    (property "Footprint" "" (id 2) (at 257.048 72.39 90)
+    (property "Value" "782763301" (id 1) (at 251.46 72.39 90))
+    (property "Footprint" "Inductor_SMD:L_1206_3216Metric" (id 2) (at 257.048 72.39 90)
       (effects (font (size 1.27 1.27)) hide)
     )
@@
     (in_bom yes) (on_board yes)
     (property "Reference" "FB2" (id 0) (at 167.005 31.75 90))
-    (property "Value" "FerriteBead" (id 1) (at 167.64 24.13 90))
-    (property "Footprint" "" (id 2) (at 167.64 29.718 90)
+    (property "Value" "782763301" (id 1) (at 167.64 24.13 90))
+    (property "Footprint" "Inductor_SMD:L_1206_3216Metric" (id 2) (at 167.64 29.718 90)
       (effects (font (size 1.27 1.27)) hide)
     )
@@
     (in_bom yes) (on_board yes)
     (property "Reference" "FB5" (id 0) (at 33.655 83.82 90))
-    (property "Value" "FerriteBead" (id 1) (at 34.29 76.2 90))
-    (property "Footprint" "" (id 2) (at 34.29 81.788 90)
+    (property "Value" "782763301" (id 1) (at 34.29 76.2 90))
+    (property "Footprint" "Inductor_SMD:L_1206_3216Metric" (id 2) (at 34.29 81.788 90)
       (effects (font (size 1.27 1.27)) hide)
     )
@@
     (in_bom yes) (on_board yes)
     (property "Reference" "FB3" (id 0) (at 118.11 73.025 90))
-    (property "Value" "FerriteBead" (id 1) (at 110.49 72.39 90))
-    (property "Footprint" "" (id 2) (at 116.078 72.39 90)
+    (property "Value" "782763301" (id 1) (at 110.49 72.39 90))
+    (property "Footprint" "Inductor_SMD:L_1206_3216Metric" (id 2) (at 116.078 72.39 90)
       (effects (font (size 1.27 1.27)) hide)
     )
@@
     (in_bom yes) (on_board yes)
     (property "Reference" "FB7" (id 0) (at 33.655 104.14 90))
-    (property "Value" "FerriteBead" (id 1) (at 34.29 96.52 90))
-    (property "Footprint" "" (id 2) (at 34.29 102.108 90)
+    (property "Value" "782763301" (id 1) (at 34.29 96.52 90))
+    (property "Footprint" "Inductor_SMD:L_1206_3216Metric" (id 2) (at 34.29 102.108 90)
       (effects (font (size 1.27 1.27)) hide)
     )
@@
     (in_bom yes) (on_board yes)
     (property "Reference" "FB6" (id 0) (at 174.625 83.82 90))
-    (property "Value" "FerriteBead" (id 1) (at 175.26 76.2 90))
-    (property "Footprint" "" (id 2) (at 175.26 81.788 90)
+    (property "Value" "782763301" (id 1) (at 175.26 76.2 90))
+    (property "Footprint" "Inductor_SMD:L_1206_3216Metric" (id 2) (at 175.26 81.788 90)
       (effects (font (size 1.27 1.27)) hide)
     )
@@
     (in_bom yes) (on_board yes)
     (property "Reference" "FB8" (id 0) (at 174.625 104.14 90))
-    (property "Value" "FerriteBead" (id 1) (at 175.26 96.52 90))
-    (property "Footprint" "" (id 2) (at 175.26 102.108 90)
+    (property "Value" "782763301" (id 1) (at 175.26 96.52 90))
+    (property "Footprint" "Inductor_SMD:L_1206_3216Metric" (id 2) (at 175.26 102.108 90)
       (effects (font (size 1.27 1.27)) hide)
     )
@@
       (effects (font (size 1.27 1.27)) hide)
     )
-    (property "Datasheet" "https://www.mouser.com/datasheet/2/761/sc4626-1277391.pdf" (id 3) (at 184.15 19.05 0)
+    (property "Datasheet" "~" (id 3) (at 184.15 19.05 0)
       (effects (font (size 1.27 1.27)) hide)
     )
@@
       (effects (font (size 1.27 1.27)) hide)
     )
-    (property "Datasheet" "https://www.mouser.com/datasheet/2/761/sc4626-1277391.pdf" (id 3) (at 43.18 19.05 0)
-      (effects (font (size 1.27 1.27)) hide)
-    )
+    (property "Datasheet" "~" (id 3) (at 43.18 19.05 0)
+      (effects (font (size 1.27 1.27)) hide)
+    )
