File: System_Controller.kicad_sch (KiCad schematic)
At the start: 49 parts, among them J10 CONSOLE, J11 USB_B_Micro, J12 Conn_ARM_JTAG_SWD_10, SW1 USB_PGM, SW2 USB_PGM, U16 RP2040, U17 IS25LP128F-JBLE, Y1 12MHz

Commit message: Minor corrections
Parts:
- renumbered R284 to R291, R285 to R292, R286 to R293, R287 to R294, R288 to R295, R289 to R296, R290 to R297, R291 to R298, R292 to R299, R293 to R300, R294 to R301, R295 to R302, R296 to R303, R297 to R304, R298 to R305, R299 to R306, R300 to R307, R301 to R308, R302 to R309, R303 to R310, R304 to R311, R305 to R312, R306 to R313
Connections:
- net MDI_SSCPI_0: no longer U16.17 (GPIO14), U16.27 (GPIO16), U16.29 (GPIO18), U16.31 (GPIO20), U16.34 (GPIO22), U16.36 (GPIO24)
- net MDI_SSCPO_0: no longer R303.2, R304.2, R306.2, R307.2, R309.2, R310.2
- new net MDI_SSCPI_1: U16.17 (GPIO14)
- new net MDI_SSCPI_2: U16.27 (GPIO16)
- new net MDI_SSCPI_3: U16.29 (GPIO18)
- new net MDI_SSCPI_4: U16.31 (GPIO20)
- new net MDI_SSCPI_5: U16.34 (GPIO22)
- new net MDI_SSCPI_6: U16.36 (GPIO24)
- new net MDI_SSCPO_1: R303.2
- new net MDI_SSCPO_2: R304.2
- new net MDI_SSCPO_3: R306.2
- new net MDI_SSCPO_4: R307.2
- new net MDI_SSCPO_5: R309.2
- new net MDI_SSCPO_6: R310.2
Other:
- note added: "330R for rise time control"
- note removed: "330R to soften the edge slope"
- moved on the sheet: C237, R291, SW1

Commit message: Assigning Footprints
Parts:
- H9: footprint (none) -> MountingHole:MountingHole_3.2mm_M3_Pad_Via
- J12: footprint (none) -> Connector_PinHeader_2.54mm:PinHeader_2x05_P2.54mm_Vertical
- R292, R293, R294, R295, R296, R297, R298, R299, R300, R301, R302, R303, R304, R306, R307, R309, R310, R311: footprint (none) -> Resistor_SMD:R_0603_1608Metric
