File: 10Base-T1L-PHY0.kicad_sch (KiCad schematic)
At the start: 51 parts, among them J2 PHY0_MDI, U1 SJA1105Q, U5 ADIN1100

Commit message: Minor corrections
Parts:
- added R21: 4K7, Resistor_SMD:R_0603_1608Metric, symbol Device:R
- renumbered R21 to R22, R22 to R23, R23 to R24, R24 to R25, R25 to R26, R26 to R27, R27 to R28, R28 to R29, R29 to R30, R30 to R31, R31 to R32, R32 to R33, R33 to R34, R34 to R35, R35 to R36, R36 to R37, R37 to R38, R38 to R39, R39 to R40, R40 to R41
Connections:
- net +3V3: now also R21.2
- net at R24.1, U1.G1 (MII0_RX_DV): now also R21.1
Other:
- note added: "Config: ------ MACIF_SEL: 0b00 => RMII MS_SEL2: 0b0 => Prefer Slave TX2P4: 0b0 => Enable 1.0V and 2.4V TX SWPD_ENB: 0b1 => Do not enter power down"

Commit message: Assigning Footprints
Parts:
- added C257: 8p2, Capacitor_SMD:C_0603_1608Metric, symbol Device:C
- added C258: 10p, Capacitor_SMD:C_0603_1608Metric, symbol Device:C
- D3: footprint (none) -> Diode_SMD:D_SOD-323
- D4, D5: footprint (none) -> UCLAMP3311P:SLP1006P2
- FB9: footprint Inductor_SMD:L_0805_2012Metric -> Inductor_SMD:L_1206_3216Metric
- H1: footprint (none) -> MountingHole:MountingHole_3.2mm_M3_Pad_Via
- J2: footprint (none) -> TerminalBlock_RND:TerminalBlock_RND_205-00288_1x03_P5.08mm_Horizontal
- L3: footprint (none) -> PID75:PID75-251M
- L4, L5: footprint (none) -> ICI70CGI:ICI70CGI
Connections:
- net GND: now also C258.2
- net at R31.2: now also C257.1; no longer U5.8 (XTAL_I/CLK_IN)
- new net: C257.2, C258.1, U5.8 (XTAL_I/CLK_IN)
Other:
- note added: "1Vp-p attenuation"
Changed lines of the file:
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@@
   (junction (at 251.46 76.2) (diameter 0) (color 0 0 0 0)
   )
+  (junction (at 55.88 102.87) (diameter 0) (color 0 0 0 0)
+  )
   (junction (at 261.62 87.63) (diameter 0) (color 0 0 0 0)
   )
@@
     (stroke (width 0) (type default) (color 0 0 0 0))
   )
+  (wire (pts (xy 55.88 83.82) (xy 55.88 95.25))
+    (stroke (width 0) (type default) (color 0 0 0 0))
+  )
   (wire (pts (xy 53.34 49.53) (xy 53.34 52.07))
     (stroke (width 0) (type default) (color 0 0 0 0))
@@
     (stroke (width 0) (type default) (color 0 0 0 0))
   )
-  (wire (pts (xy 68.58 83.82) (xy 68.58 106.68))
-    (stroke (width 0) (type default) (color 0 0 0 0))
-  )
   (wire (pts (xy 115.57 132.08) (xy 118.11 132.08))
     (stroke (width 0) (type default) (color 0 0 0 0))
@@
     (stroke (width 0) (type default) (color 0 0 0 0))
   )
-  (wire (pts (xy 49.53 83.82) (xy 68.58 83.82))
+  (wire (pts (xy 49.53 83.82) (xy 55.88 83.82))
     (stroke (width 0) (type default) (color 0 0 0 0))
   )
@@
     (stroke (width 0) (type default) (color 0 0 0 0))
   )
+  (wire (pts (xy 68.58 102.87) (xy 68.58 106.68))
+    (stroke (width 0) (type default) (color 0 0 0 0))
+  )
   (wire (pts (xy 41.91 68.58) (xy 69.85 68.58))
     (stroke (width 0) (type default) (color 0 0 0 0))
@@
     (stroke (width 0) (type default) (color 0 0 0 0))
   )
+  (wire (pts (xy 55.88 102.87) (xy 68.58 102.87))
+    (stroke (width 0) (type default) (color 0 0 0 0))
+  )
   (wire (pts (xy 219.71 73.66) (xy 213.36 73.66))
     (stroke (width 0) (type default) (color 0 0 0 0))
@@
   (wire (pts (xy 49.53 93.98) (xy 77.47 93.98))
     (stroke (width 0) (type default) (color 0 0 0 0))
+  )
+  (text "1Vp-p\nattenuation" (at 60.96 101.6 0)
+    (effects (font (size 1.27 1.27)) (justify left bottom))
   )
   (text "Config:\n------\nMACIF_SEL: 	0b00 	=> RMII\nMS_SEL2: 	0b0 	=> Prefer Slave\nTX2P4: 		0b0 	=> Enable 1.0V and 2.4V TX\nSWPD_ENB: 	0b1 	=> Do not enter power down"
@@
     (property "Reference" "L5" (id 0) (at 224.79 66.675 0))
     (property "Value" "RCM70CGI-471" (id 1) (at 224.79 77.47 0))
-    (property "Footprint" "" (id 2) (at 224.79 71.12 0)
-      (effects (font (size 1.27 1.27)) hide)
-    )
-    (property "Datasheet" "~" (id 3) (at 224.79 71.12 0)
+    (property "Footprint" "ICI70CGI:ICI70CGI" (id 2) (at 224.79 71.12 0)
+      (effects (font (size 1.27 1.27)) hide)
+    )
+    (property "Datasheet" "https://product.tdk.com/system/files/dam/doc/product/transformer/transformer/lan/data_sheet/30/ds/lan_mod/rcm70cgi.pdf" (id 3) (at 224.79 71.12 0)
       (effects (font (size 1.27 1.27)) hide)
     )
@@
     (property "Reference" "D5" (id 0) (at 168.91 93.98 0))
     (property "Value" "UCLAMP3311P" (id 1) (at 180.34 93.98 90))
-    (property "Footprint" "" (id 2) (at 171.45 93.98 0)
+    (property "Footprint" "UCLAMP3311P:SLP1006P2" (id 2) (at 171.45 93.98 0)
       (effects (font (size 1.27 1.27)) hide)
     )
@@
     (property "Reference" "H1" (id 0) (at 279.4 87.63 0))
     (property "Value" "CHASSIS_PE" (id 1) (at 277.495 87.63 0))
-    (property "Footprint" "" (id 2) (at 273.05 87.63 0)
+    (property "Footprint" "MountingHole:MountingHole_3.2mm_M3_Pad_Via" (id 2) (at 273.05 87.63 0)
       (effects (font (size 1.27 1.27)) hide)
     )
@@
     (property "Reference" "FB9" (id 0) (at 161.925 113.03 90))
     (property "Value" "FerriteBead" (id 1) (at 162.56 105.41 90))
-    (property "Footprint" "Inductor_SMD:L_0805_2012Metric" (id 2) (at 162.56 110.998 90)
+    (property "Footprint" "Inductor_SMD:L_1206_3216Metric" (id 2) (at 162.56 110.998 90)
       (effects (font (size 1.27 1.27)) hide)
     )
@@
     (property "Reference" "D3" (id 0) (at 248.92 71.12 0))
     (property "Value" "CDSOD323-T36SC" (id 1) (at 251.46 63.5 90))
-    (property "Footprint" "" (id 2) (at 251.46 71.12 0)
+    (property "Footprint" "Diode_SMD:D_SOD-323" (id 2) (at 251.46 71.12 0)
       (effects (font (size 1.27 1.27)) hide)
     )
@@
     (property "Reference" "L4" (id 0) (at 192.405 71.12 0))
     (property "Value" "ICI70CGI-222" (id 1) (at 179.07 71.12 90))
-    (property "Footprint" "" (id 2) (at 187.96 71.12 0)
-      (effects (font (size 1.27 1.27)) hide)
-    )
-    (property "Datasheet" "~" (id 3) (at 187.96 71.12 0)
+    (property "Footprint" "ICI70CGI:ICI70CGI" (id 2) (at 187.96 71.12 0)
+      (effects (font (size 1.27 1.27)) hide)
+    )
+    (property "Datasheet" "https://product.tdk.com/system/files/dam/doc/product/transformer/transformer/lan/data_sheet/30/ds/lan_mod/ici70cgi.pdf" (id 3) (at 187.96 71.12 0)
       (effects (font (size 1.27 1.27)) hide)
     )
@@
     (pin "1")
   )
+  (symbol (lib_id "Device:C") (at 55.88 106.68 0) (unit 1)
+    (in_bom yes) (on_board yes)
+    (property "Reference" "C258" (id 0) (at 56.515 104.14 0)
+      (effects (font (size 1.27 1.27)) (justify left))
+    )
+    (property "Value" "10p" (id 1) (at 56.515 109.22 0)
+      (effects (font (size 1.27 1.27)) (justify left))
+    )
+    (property "Footprint" "Capacitor_SMD:C_0603_1608Metric" (id 2) (at 56.8452 110.49 0)
+      (effects (font (size 1.27 1.27)) hide)
+    )
+    (property "Datasheet" "~" (id 3) (at 55.88 106.68 0)
+      (effects (font (size 1.27 1.27)) hide)
+    )
+    (pin "1")
+    (pin "2")
+  )
   (symbol (lib_id "Device:LED") (at 127 43.18 90) (unit 1)
     (in_bom yes) (on_board yes)
@@
     )
     (property "Datasheet" "~" (id 3) (at 119.38 43.18 0)
+      (effects (font (size 1.27 1.27)) hide)
+    )
+    (pin "1")
+    (pin "2")
+  )
+  (symbol (lib_id "Device:C") (at 55.88 99.06 0) (unit 1)
+    (in_bom yes) (on_board yes)
+    (property "Reference" "C257" (id 0) (at 56.515 96.52 0)
+      (effects (font (size 1.27 1.27)) (justify left))
+    )
+    (property "Value" "8p2" (id 1) (at 56.515 101.6 0)
+      (effects (font (size 1.27 1.27)) (justify left))
+    )
+    (property "Footprint" "Capacitor_SMD:C_0603_1608Metric" (id 2) (at 56.8452 102.87 0)
+      (effects (font (size 1.27 1.27)) hide)
+    )
+    (property "Datasheet" "~" (id 3) (at 55.88 99.06 0)
       (effects (font (size 1.27 1.27)) hide)
     )
@@
     (property "Reference" "D4" (id 0) (at 163.83 93.98 0))
     (property "Value" "UCLAMP3311P" (id 1) (at 156.21 93.98 90))
-    (property "Footprint" "" (id 2) (at 166.37 93.98 0)
+    (property "Footprint" "UCLAMP3311P:SLP1006P2" (id 2) (at 166.37 93.98 0)
       (effects (font (size 1.27 1.27)) hide)
     )
@@
     (property "Reference" "J2" (id 0) (at 267.97 67.31 0))
     (property "Value" "PHY0_MDI" (id 1) (at 267.97 77.47 0))
-    (property "Footprint" "" (id 2) (at 267.97 72.39 0)
+    (property "Footprint" "TerminalBlock_RND:TerminalBlock_RND_205-00288_1x03_P5.08mm_Horizontal" (id 2) (at 267.97 72.39 0)
       (effects (font (size 1.27 1.27)) hide)
     )
@@
     (property "Reference" "L3" (id 0) (at 230.505 53.34 0))
     (property "Value" "PID75-251M" (id 1) (at 239.395 53.34 0))
-    (property "Footprint" "" (id 2) (at 234.95 53.34 0)
-      (effects (font (size 1.27 1.27)) hide)
-    )
-    (property "Datasheet" "~" (id 3) (at 234.95 53.34 0)
+    (property "Footprint" "PID75:PID75-251M" (id 2) (at 234.95 53.34 0)
+      (effects (font (size 1.27 1.27)) hide)
+    )
+    (property "Datasheet" "https://product.tdk.com/system/files/dam/doc/product/inductor/inductor/smd/data_sheet/30/db/ind_2008/pidx251m.pdf" (id 3) (at 234.95 53.34 0)
       (effects (font (size 1.27 1.27)) hide)
     )
@@
     (pin "2")
   )
+  (symbol (lib_id "power:GND") (at 55.88 110.49 0) (unit 1)
+    (in_bom yes) (on_board yes)
+    (property "Reference" "#PWR0248" (id 0) (at 55.88 116.84 0)
+      (effects (font (size 1.27 1.27)) hide)
+    )
+    (property "Value" "GND" (id 1) (at 55.88 114.3 0))
+    (property "Footprint" "" (id 2) (at 55.88 110.49 0)
+      (effects (font (size 1.27 1.27)) hide)
+    )
+    (property "Datasheet" "" (id 3) (at 55.88 110.49 0)
+      (effects (font (size 1.27 1.27)) hide)
+    )
+    (pin "1")
+  )
   (symbol (lib_id "Device:C") (at 115.57 124.46 0) (unit 1)

Commit message: Fixing termination for T1L PHYs
Parts:
- removed R40, R41: 100, Resistor_SMD:R_0805_2012Metric, symbol Device:R
- C78, C79: value 10n -> 100p
- FB9: value FerriteBead -> 782763301
Connections:
- net GND: now also C78.2, C79.2
Changed lines of the file:
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@@
     (stroke (width 0) (type default) (color 0 0 0 0))
   )
-  (wire (pts (xy 237.49 99.06) (xy 237.49 100.33))
+  (wire (pts (xy 237.49 87.63) (xy 237.49 88.9))
     (stroke (width 0) (type default) (color 0 0 0 0))
   )
@@
     (stroke (width 0) (type default) (color 0 0 0 0))
   )
-  (wire (pts (xy 246.38 87.63) (xy 246.38 91.44))
-    (stroke (width 0) (type default) (color 0 0 0 0))
-  )
   (wire (pts (xy 48.26 66.04) (xy 69.85 66.04))
     (stroke (width 0) (type default) (color 0 0 0 0))
@@
     (stroke (width 0) (type default) (color 0 0 0 0))
   )
-  (wire (pts (xy 246.38 99.06) (xy 246.38 100.33))
+  (wire (pts (xy 246.38 87.63) (xy 246.38 88.9))
     (stroke (width 0) (type default) (color 0 0 0 0))
   )
@@
   )
   (wire (pts (xy 251.46 66.04) (xy 251.46 67.31))
-    (stroke (width 0) (type default) (color 0 0 0 0))
-  )
-  (wire (pts (xy 237.49 87.63) (xy 237.49 91.44))
     (stroke (width 0) (type default) (color 0 0 0 0))
   )
@@
       (effects (font (size 1.27 1.27)) (justify left))
     )
-    (property "Value" "10n" (id 1) (at 238.125 86.36 0)
+    (property "Value" "100p" (id 1) (at 238.125 86.36 0)
       (effects (font (size 1.27 1.27)) (justify left))
     )
@@
     (pin "2")
   )
-  (symbol (lib_id "Device:R") (at 246.38 95.25 180) (unit 1)
-    (in_bom yes) (on_board yes)
-    (property "Reference" "R41" (id 0) (at 244.348 95.25 90))
-    (property "Value" "100" (id 1) (at 246.38 95.25 90))
-    (property "Footprint" "Resistor_SMD:R_0805_2012Metric" (id 2) (at 248.158 95.25 90)
-      (effects (font (size 1.27 1.27)) hide)
-    )
-    (property "Datasheet" "~" (id 3) (at 246.38 95.25 0)
-      (effects (font (size 1.27 1.27)) hide)
-    )
-    (pin "1")
-    (pin "2")
-  )
   (symbol (lib_id "Mechanical:MountingHole_Pad") (at 273.05 87.63 270) (unit 1)
     (in_bom yes) (on_board yes)
@@
     (in_bom yes) (on_board yes)
     (property "Reference" "FB9" (id 0) (at 161.925 113.03 90))
-    (property "Value" "FerriteBead" (id 1) (at 162.56 105.41 90))
+    (property "Value" "782763301" (id 1) (at 162.56 105.41 90))
     (property "Footprint" "Inductor_SMD:L_1206_3216Metric" (id 2) (at 162.56 110.998 90)
       (effects (font (size 1.27 1.27)) hide)
@@
     (pin "2")
   )
-  (symbol (lib_id "Device:R") (at 237.49 95.25 180) (unit 1)
-    (in_bom yes) (on_board yes)
-    (property "Reference" "R40" (id 0) (at 235.458 95.25 90))
-    (property "Value" "100" (id 1) (at 237.49 95.25 90))
-    (property "Footprint" "Resistor_SMD:R_0805_2012Metric" (id 2) (at 239.268 95.25 90)
-      (effects (font (size 1.27 1.27)) hide)
-    )
-    (property "Datasheet" "~" (id 3) (at 237.49 95.25 0)
-      (effects (font (size 1.27 1.27)) hide)
-    )
-    (pin "1")
-    (pin "2")
-  )
   (symbol (lib_id "Device:C") (at 207.01 62.23 90) (unit 1)
     (in_bom yes) (on_board yes)
@@
     (pin "2")
   )
-  (symbol (lib_id "power:GND") (at 246.38 100.33 0) (unit 1)
-    (in_bom yes) (on_board yes)
-    (property "Reference" "#PWR090" (id 0) (at 246.38 106.68 0)
-      (effects (font (size 1.27 1.27)) hide)
-    )
-    (property "Value" "GND" (id 1) (at 246.38 104.14 0))
-    (property "Footprint" "" (id 2) (at 246.38 100.33 0)
-      (effects (font (size 1.27 1.27)) hide)
-    )
-    (property "Datasheet" "" (id 3) (at 246.38 100.33 0)
+  (symbol (lib_id "power:GND") (at 246.38 88.9 0) (unit 1)
+    (in_bom yes) (on_board yes)
+    (property "Reference" "#PWR090" (id 0) (at 246.38 95.25 0)
+      (effects (font (size 1.27 1.27)) hide)
+    )
+    (property "Value" "GND" (id 1) (at 246.38 92.71 0))
+    (property "Footprint" "" (id 2) (at 246.38 88.9 0)
+      (effects (font (size 1.27 1.27)) hide)
+    )
+    (property "Datasheet" "" (id 3) (at 246.38 88.9 0)
       (effects (font (size 1.27 1.27)) hide)
     )
@@
       (effects (font (size 1.27 1.27)) (justify left))
     )
-    (property "Value" "10n" (id 1) (at 247.015 86.36 0)
+    (property "Value" "100p" (id 1) (at 247.015 86.36 0)
       (effects (font (size 1.27 1.27)) (justify left))
     )
@@
     (pin "2")
   )
-  (symbol (lib_id "power:GND") (at 237.49 100.33 0) (unit 1)
-    (in_bom yes) (on_board yes)
-    (property "Reference" "#PWR089" (id 0) (at 237.49 106.68 0)
-      (effects (font (size 1.27 1.27)) hide)
-    )
-    (property "Value" "GND" (id 1) (at 237.49 104.14 0))
-    (property "Footprint" "" (id 2) (at 237.49 100.33 0)
-      (effects (font (size 1.27 1.27)) hide)
-    )
-    (property "Datasheet" "" (id 3) (at 237.49 100.33 0)
-      (effects (font (size 1.27 1.27)) hide)
-    )
+  (symbol (lib_id "power:GND") (at 237.49 88.9 0) (unit 1)
+    (in_bom yes) (on_board yes)
+    (property "Reference" "#PWR089" (id 0) (at 237.49 95.25 0)
+      (effects (font (size 1.27 1.27)) hide)
+    )
+    (property "Value" "GND" (id 1) (at 237.49 92.71 0))
+    (property "Footprint" "" (id 2) (at 237.49 88.9 0)
+      (effects (font (size 1.27 1.27)) hide)
+    )
+    (property "Datasheet" "" (id 3) (at 237.49 88.9 0)
+      (effects (font (size 1.27 1.27)) hide)
+    )
