File: 10Base-T1L-PHY1.kicad_sch (KiCad schematic)
At the start: 52 parts, among them J3 PHY1_MDI, U1 SJA1105Q, U6 ADIN1100

Commit message: Minor corrections
Parts:
- added R46: 4K7, Resistor_SMD:R_0603_1608Metric, symbol Device:R
- R47: renamed from R45; value 1K -> 4K7
- renumbered R41 to R42, R42 to R43, R43 to R44, R44 to R45, R46 to R48, R47 to R49, R48 to R50, R49 to R51, R50 to R52, R51 to R53, R52 to R54, R53 to R55, R54 to R56, R55 to R57, R56 to R58, R57 to R59, R58 to R60, R59 to R61, R60 to R62, R61 to R63, R62 to R64, R63 to R65, R64 to R66, R65 to R67
Connections:
- net +3V3: now also R46.2
- net at R50.1, U1.A4 (MII1_RX_DV): now also R46.1
Other:
- note added: "Config: ------ MACIF_SEL: 0b00 => RMII MS_SEL2: 0b0 => Prefer Slave TX2P4: 0b0 => Enable 1.0V and 2.4V TX SWPD_ENB: 0b1 => Do not enter power down"

Commit message: Assigning Footprints
Parts:
- added C259: 8p2, Capacitor_SMD:C_0603_1608Metric, symbol Device:C
- added C260: 10p, Capacitor_SMD:C_0603_1608Metric, symbol Device:C
- D10, D9: footprint (none) -> UCLAMP3311P:SLP1006P2
- D8: footprint (none) -> Diode_SMD:D_SOD-323
- FB10: footprint Inductor_SMD:L_0805_2012Metric -> Inductor_SMD:L_1206_3216Metric
- H2: footprint (none) -> MountingHole:MountingHole_3.2mm_M3_Pad_Via
- J3: footprint (none) -> TerminalBlock_RND:TerminalBlock_RND_205-00288_1x03_P5.08mm_Horizontal
- L6: footprint (none) -> PID75:PID75-251M
- L7, L8: footprint (none) -> ICI70CGI:ICI70CGI
Connections:
- net GND: now also C260.2
- net at R57.2: now also C259.1; no longer U6.8 (XTAL_I/CLK_IN)
- new net: C259.2, C260.1, U6.8 (XTAL_I/CLK_IN)
Other:
- note added: "1Vp-p attenuation"
Changed lines of the file:
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@@
   (junction (at 173.99 62.23) (diameter 0) (color 0 0 0 0)
   )
+  (junction (at 55.88 102.87) (diameter 0) (color 0 0 0 0)
+  )
   (junction (at 185.42 80.01) (diameter 0) (color 0 0 0 0)
   )
@@
     (stroke (width 0) (type default) (color 0 0 0 0))
   )
+  (wire (pts (xy 55.88 83.82) (xy 55.88 95.25))
+    (stroke (width 0) (type default) (color 0 0 0 0))
+  )
   (wire (pts (xy 170.18 132.08) (xy 170.18 128.27))
     (stroke (width 0) (type default) (color 0 0 0 0))
@@
     (stroke (width 0) (type default) (color 0 0 0 0))
   )
+  (wire (pts (xy 68.58 102.87) (xy 68.58 106.68))
+    (stroke (width 0) (type default) (color 0 0 0 0))
+  )
   (wire (pts (xy 261.62 87.63) (xy 261.62 74.93))
     (stroke (width 0) (type default) (color 0 0 0 0))
@@
     (stroke (width 0) (type default) (color 0 0 0 0))
   )
+  (wire (pts (xy 55.88 102.87) (xy 68.58 102.87))
+    (stroke (width 0) (type default) (color 0 0 0 0))
+  )
   (wire (pts (xy 173.99 80.01) (xy 166.37 80.01))
     (stroke (width 0) (type default) (color 0 0 0 0))
@@
     (stroke (width 0) (type default) (color 0 0 0 0))
   )
-  (wire (pts (xy 68.58 83.82) (xy 68.58 106.68))
-    (stroke (width 0) (type default) (color 0 0 0 0))
-  )
   (wire (pts (xy 149.86 58.42) (xy 149.86 63.5))
     (stroke (width 0) (type default) (color 0 0 0 0))
@@
     (stroke (width 0) (type default) (color 0 0 0 0))
   )
-  (wire (pts (xy 49.53 83.82) (xy 68.58 83.82))
+  (wire (pts (xy 49.53 83.82) (xy 55.88 83.82))
     (stroke (width 0) (type default) (color 0 0 0 0))
   )
@@
   (text "Generic 1206 Footprints.\nPopulate according \nto EMC needs."
     (at 254 113.03 0)
+    (effects (font (size 1.27 1.27)) (justify left bottom))
+  )
+  (text "1Vp-p\nattenuation" (at 60.96 101.6 0)
     (effects (font (size 1.27 1.27)) (justify left bottom))
   )
@@
     (property "Reference" "J3" (id 0) (at 267.97 67.31 0))
     (property "Value" "PHY1_MDI" (id 1) (at 267.97 77.47 0))
-    (property "Footprint" "" (id 2) (at 267.97 72.39 0)
+    (property "Footprint" "TerminalBlock_RND:TerminalBlock_RND_205-00288_1x03_P5.08mm_Horizontal" (id 2) (at 267.97 72.39 0)
       (effects (font (size 1.27 1.27)) hide)
     )
@@
     (pin "2")
   )
+  (symbol (lib_id "Device:C") (at 55.88 99.06 0) (unit 1)
+    (in_bom yes) (on_board yes)
+    (property "Reference" "C259" (id 0) (at 56.515 96.52 0)
+      (effects (font (size 1.27 1.27)) (justify left))
+    )
+    (property "Value" "8p2" (id 1) (at 56.515 101.6 0)
+      (effects (font (size 1.27 1.27)) (justify left))
+    )
+    (property "Footprint" "Capacitor_SMD:C_0603_1608Metric" (id 2) (at 56.8452 102.87 0)
+      (effects (font (size 1.27 1.27)) hide)
+    )
+    (property "Datasheet" "~" (id 3) (at 55.88 99.06 0)
+      (effects (font (size 1.27 1.27)) hide)
+    )
+    (pin "1")
+    (pin "2")
+  )
   (symbol (lib_id "Device:D_TVS") (at 251.46 71.12 90) (unit 1)
     (in_bom yes) (on_board yes)
     (property "Reference" "D8" (id 0) (at 248.92 71.12 0))
     (property "Value" "CDSOD323-T36SC" (id 1) (at 251.46 63.5 90))
-    (property "Footprint" "" (id 2) (at 251.46 71.12 0)
+    (property "Footprint" "Diode_SMD:D_SOD-323" (id 2) (at 251.46 71.12 0)
       (effects (font (size 1.27 1.27)) hide)
     )
@@
     (property "Reference" "D9" (id 0) (at 163.83 93.98 0))
     (property "Value" "UCLAMP3311P" (id 1) (at 156.21 93.98 90))
-    (property "Footprint" "" (id 2) (at 166.37 93.98 0)
+    (property "Footprint" "UCLAMP3311P:SLP1006P2" (id 2) (at 166.37 93.98 0)
       (effects (font (size 1.27 1.27)) hide)
     )
@@
     (property "Reference" "L7" (id 0) (at 192.405 71.12 0))
     (property "Value" "ICI70CGI-222" (id 1) (at 179.07 71.12 90))
-    (property "Footprint" "" (id 2) (at 187.96 71.12 0)
-      (effects (font (size 1.27 1.27)) hide)
-    )
-    (property "Datasheet" "~" (id 3) (at 187.96 71.12 0)
+    (property "Footprint" "ICI70CGI:ICI70CGI" (id 2) (at 187.96 71.12 0)
+      (effects (font (size 1.27 1.27)) hide)
+    )
+    (property "Datasheet" "https://product.tdk.com/system/files/dam/doc/product/transformer/transformer/lan/data_sheet/30/ds/lan_mod/ici70cgi.pdf" (id 3) (at 187.96 71.12 0)
       (effects (font (size 1.27 1.27)) hide)
     )
@@
     (property "Reference" "H2" (id 0) (at 279.4 87.63 0))
     (property "Value" "CHASSIS_PE" (id 1) (at 277.495 87.63 0))
-    (property "Footprint" "" (id 2) (at 273.05 87.63 0)
+    (property "Footprint" "MountingHole:MountingHole_3.2mm_M3_Pad_Via" (id 2) (at 273.05 87.63 0)
       (effects (font (size 1.27 1.27)) hide)
     )
@@
     (pin "2")
   )
+  (symbol (lib_id "Device:C") (at 55.88 106.68 0) (unit 1)
+    (in_bom yes) (on_board yes)
+    (property "Reference" "C260" (id 0) (at 56.515 104.14 0)
+      (effects (font (size 1.27 1.27)) (justify left))
+    )
+    (property "Value" "10p" (id 1) (at 56.515 109.22 0)
+      (effects (font (size 1.27 1.27)) (justify left))
+    )
+    (property "Footprint" "Capacitor_SMD:C_0603_1608Metric" (id 2) (at 56.8452 110.49 0)
+      (effects (font (size 1.27 1.27)) hide)
+    )
+    (property "Datasheet" "~" (id 3) (at 55.88 106.68 0)
+      (effects (font (size 1.27 1.27)) hide)
+    )
+    (pin "1")
+    (pin "2")
+  )
   (symbol (lib_id "Device:R") (at 144.78 58.42 270) (unit 1)
     (in_bom yes) (on_board yes)
@@
     (property "Reference" "FB10" (id 0) (at 161.925 113.03 90))
     (property "Value" "FerriteBead" (id 1) (at 162.56 105.41 90))
-    (property "Footprint" "Inductor_SMD:L_0805_2012Metric" (id 2) (at 162.56 110.998 90)
+    (property "Footprint" "Inductor_SMD:L_1206_3216Metric" (id 2) (at 162.56 110.998 90)
       (effects (font (size 1.27 1.27)) hide)
     )
@@
     (property "Reference" "L8" (id 0) (at 224.79 66.675 0))
     (property "Value" "RCM70CGI-471" (id 1) (at 224.79 77.47 0))
-    (property "Footprint" "" (id 2) (at 224.79 71.12 0)
-      (effects (font (size 1.27 1.27)) hide)
-    )
-    (property "Datasheet" "~" (id 3) (at 224.79 71.12 0)
+    (property "Footprint" "ICI70CGI:ICI70CGI" (id 2) (at 224.79 71.12 0)
+      (effects (font (size 1.27 1.27)) hide)
+    )
+    (property "Datasheet" "https://product.tdk.com/system/files/dam/doc/product/transformer/transformer/lan/data_sheet/30/ds/lan_mod/rcm70cgi.pdf" (id 3) (at 224.79 71.12 0)
       (effects (font (size 1.27 1.27)) hide)
     )
@@
     (pin "2")
   )
+  (symbol (lib_id "power:GND") (at 55.88 110.49 0) (unit 1)
+    (in_bom yes) (on_board yes)
+    (property "Reference" "#PWR0249" (id 0) (at 55.88 116.84 0)
+      (effects (font (size 1.27 1.27)) hide)
+    )
+    (property "Value" "GND" (id 1) (at 55.88 114.3 0))
+    (property "Footprint" "" (id 2) (at 55.88 110.49 0)
+      (effects (font (size 1.27 1.27)) hide)
+    )
+    (property "Datasheet" "" (id 3) (at 55.88 110.49 0)
+      (effects (font (size 1.27 1.27)) hide)
+    )
+    (pin "1")
+  )
   (symbol (lib_id "Device:D_TVS") (at 171.45 93.98 90) (unit 1)
     (in_bom yes) (on_board yes)
     (property "Reference" "D10" (id 0) (at 168.91 93.98 0))
     (property "Value" "UCLAMP3311P" (id 1) (at 180.34 93.98 90))
-    (property "Footprint" "" (id 2) (at 171.45 93.98 0)
+    (property "Footprint" "UCLAMP3311P:SLP1006P2" (id 2) (at 171.45 93.98 0)
       (effects (font (size 1.27 1.27)) hide)
     )
@@
     (property "Reference" "L6" (id 0) (at 230.505 53.34 0))
     (property "Value" "PID75-251M" (id 1) (at 239.395 53.34 0))
-    (property "Footprint" "" (id 2) (at 234.95 53.34 0)
-      (effects (font (size 1.27 1.27)) hide)
-    )
-    (property "Datasheet" "~" (id 3) (at 234.95 53.34 0)
-      (effects (font (size 1.27 1.27)) hide)
-    )
+    (property "Footprint" "PID75:PID75-251M" (id 2) (at 234.95 53.34 0)
+      (effects (font (size 1.27 1.27)) hide)
+    )
+    (property "Datasheet" "https://product.tdk.com/system/files/dam/doc/product/inductor/inductor/smd/data_sheet/30/db/ind_2008/pidx251m.pdf" (id 3) (at 234.95 53.34 0)
+      (effects (font (size 1.27 1.27)) hide)
+    )

Commit message: Fixing termination for T1L PHYs
Parts:
- removed R66, R67: 100, Resistor_SMD:R_0805_2012Metric, symbol Device:R
- C92, C93: value 10n -> 100p
- FB10: value FerriteBead -> 782763301
Connections:
- net GND: now also C92.2, C93.2
Changed lines of the file:
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@@
-    (stroke (width 0) (type default) (color 0 0 0 0))
-  )
-  (wire (pts (xy 237.49 87.63) (xy 237.49 91.44))
     (stroke (width 0) (type default) (color 0 0 0 0))
   )
@@
     (stroke (width 0) (type default) (color 0 0 0 0))
   )
-  (wire (pts (xy 246.38 87.63) (xy 246.38 91.44))
-    (stroke (width 0) (type default) (color 0 0 0 0))
-  )
   (wire (pts (xy 185.42 62.23) (xy 185.42 66.04))
     (stroke (width 0) (type default) (color 0 0 0 0))
@@
     (stroke (width 0) (type default) (color 0 0 0 0))
   )
-  (wire (pts (xy 237.49 99.06) (xy 237.49 100.33))
-    (stroke (width 0) (type default) (color 0 0 0 0))
-  )
   (wire (pts (xy 113.03 88.9) (xy 132.08 88.9))
     (stroke (width 0) (type default) (color 0 0 0 0))
@@
   )
   (wire (pts (xy 261.62 74.93) (xy 262.89 74.93))
-    (stroke (width 0) (type default) (color 0 0 0 0))
-  )
-  (wire (pts (xy 246.38 99.06) (xy 246.38 100.33))
     (stroke (width 0) (type default) (color 0 0 0 0))
   )
@@
       (effects (font (size 1.27 1.27)) (justify left))
     )
-    (property "Value" "10n" (id 1) (at 247.015 86.36 0)
+    (property "Value" "100p" (id 1) (at 247.015 86.36 0)
       (effects (font (size 1.27 1.27)) (justify left))
     )
@@
     (pin "2")
   )
-  (symbol (lib_id "power:GND") (at 237.49 100.33 0) (unit 1)
-    (in_bom yes) (on_board yes)
-    (property "Reference" "#PWR0101" (id 0) (at 237.49 106.68 0)
-      (effects (font (size 1.27 1.27)) hide)
-    )
-    (property "Value" "GND" (id 1) (at 237.49 104.14 0))
-    (property "Footprint" "" (id 2) (at 237.49 100.33 0)
-      (effects (font (size 1.27 1.27)) hide)
-    )
-    (property "Datasheet" "" (id 3) (at 237.49 100.33 0)
+  (symbol (lib_id "power:GND") (at 237.49 87.63 0) (unit 1)
+    (in_bom yes) (on_board yes)
+    (property "Reference" "#PWR0101" (id 0) (at 237.49 93.98 0)
+      (effects (font (size 1.27 1.27)) hide)
+    )
+    (property "Value" "GND" (id 1) (at 237.49 91.44 0))
+    (property "Footprint" "" (id 2) (at 237.49 87.63 0)
+      (effects (font (size 1.27 1.27)) hide)
+    )
+    (property "Datasheet" "" (id 3) (at 237.49 87.63 0)
       (effects (font (size 1.27 1.27)) hide)
     )
@@
     (pin "1")
   )
-  (symbol (lib_id "power:GND") (at 246.38 100.33 0) (unit 1)
-    (in_bom yes) (on_board yes)
-    (property "Reference" "#PWR0102" (id 0) (at 246.38 106.68 0)
-      (effects (font (size 1.27 1.27)) hide)
-    )
-    (property "Value" "GND" (id 1) (at 246.38 104.14 0))
-    (property "Footprint" "" (id 2) (at 246.38 100.33 0)
-      (effects (font (size 1.27 1.27)) hide)
-    )
-    (property "Datasheet" "" (id 3) (at 246.38 100.33 0)
+  (symbol (lib_id "power:GND") (at 246.38 87.63 0) (unit 1)
+    (in_bom yes) (on_board yes)
+    (property "Reference" "#PWR0102" (id 0) (at 246.38 93.98 0)
+      (effects (font (size 1.27 1.27)) hide)
+    )
+    (property "Value" "GND" (id 1) (at 246.38 91.44 0))
+    (property "Footprint" "" (id 2) (at 246.38 87.63 0)
+      (effects (font (size 1.27 1.27)) hide)
+    )
+    (property "Datasheet" "" (id 3) (at 246.38 87.63 0)
       (effects (font (size 1.27 1.27)) hide)
     )
@@
       (effects (font (size 1.27 1.27)) (justify left))
     )
-    (property "Value" "10n" (id 1) (at 238.125 86.36 0)
+    (property "Value" "100p" (id 1) (at 238.125 86.36 0)
       (effects (font (size 1.27 1.27)) (justify left))
     )
@@
     (in_bom yes) (on_board yes)
     (property "Reference" "FB10" (id 0) (at 161.925 113.03 90))
-    (property "Value" "FerriteBead" (id 1) (at 162.56 105.41 90))
+    (property "Value" "782763301" (id 1) (at 162.56 105.41 90))
     (property "Footprint" "Inductor_SMD:L_1206_3216Metric" (id 2) (at 162.56 110.998 90)
       (effects (font (size 1.27 1.27)) hide)
@@
     )
     (property "Datasheet" "~" (id 3) (at 154.94 68.58 0)
-      (effects (font (size 1.27 1.27)) hide)
-    )
-    (pin "1")
-    (pin "2")
-  )
-  (symbol (lib_id "Device:R") (at 237.49 95.25 180) (unit 1)
-    (in_bom yes) (on_board yes)
-    (property "Reference" "R66" (id 0) (at 235.458 95.25 90))
-    (property "Value" "100" (id 1) (at 237.49 95.25 90))
-    (property "Footprint" "Resistor_SMD:R_0805_2012Metric" (id 2) (at 239.268 95.25 90)
-      (effects (font (size 1.27 1.27)) hide)
-    )
-    (property "Datasheet" "~" (id 3) (at 237.49 95.25 0)
       (effects (font (size 1.27 1.27)) hide)
     )
@@
       (effects (font (size 1.27 1.27)) hide)
     )
-    (pin "1")
-    (pin "2")
-  )
-  (symbol (lib_id "Device:R") (at 246.38 95.25 180) (unit 1)
-    (in_bom yes) (on_board yes)
-    (property "Reference" "R67" (id 0) (at 244.348 95.25 90))
-    (property "Value" "100" (id 1) (at 246.38 95.25 90))
-    (property "Footprint" "Resistor_SMD:R_0805_2012Metric" (id 2) (at 248.158 95.25 90)
-      (effects (font (size 1.27 1.27)) hide)
-    )
-    (property "Datasheet" "~" (id 3) (at 246.38 95.25 0)
-      (effects (font (size 1.27 1.27)) hide)
-    )
