File: 10Base-T1L-PHY2.kicad_sch (KiCad schematic)
At the start: 52 parts, among them J4 PHY2_MDI, U1 SJA1105Q, U7 ADIN1100

Commit message: Minor corrections
Parts:
- added R72: 4K7, Resistor_SMD:R_0603_1608Metric, symbol Device:R
- R73: renamed from R70; value 1K -> 4K7
- renumbered R66 to R68, R67 to R69, R68 to R70, R69 to R71, R71 to R74, R72 to R75, R73 to R76, R74 to R77, R75 to R78, R76 to R79, R77 to R80, R78 to R81, R79 to R82, R80 to R83, R81 to R84, R82 to R85, R83 to R86, R84 to R87, R85 to R88, R86 to R89, R87 to R90, R88 to R91, R89 to R92, R90 to R93
Connections:
- net +3V3: now also R72.2
- net at R76.1, U1.A11 (MII2_RX_DV): now also R72.1
Other:
- note added: "Config: ------ MACIF_SEL: 0b00 => RMII MS_SEL2: 0b0 => Prefer Slave TX2P4: 0b0 => Enable 1.0V and 2.4V TX SWPD_ENB: 0b1 => Do not enter power down"

Commit message: Assigning Footprints
Parts:
- added C261: 8p2, Capacitor_SMD:C_0603_1608Metric, symbol Device:C
- added C262: 10p, Capacitor_SMD:C_0603_1608Metric, symbol Device:C
- D13: footprint (none) -> Diode_SMD:D_SOD-323
- D14, D15: footprint (none) -> UCLAMP3311P:SLP1006P2
- FB11: footprint Inductor_SMD:L_0805_2012Metric -> Inductor_SMD:L_1206_3216Metric
- H3: footprint (none) -> MountingHole:MountingHole_3.2mm_M3_Pad_Via
- J4: footprint (none) -> TerminalBlock_RND:TerminalBlock_RND_205-00288_1x03_P5.08mm_Horizontal
- L10, L11: footprint (none) -> ICI70CGI:ICI70CGI
- L9: footprint (none) -> PID75:PID75-251M
Connections:
- net GND: now also C262.2
- net at R83.2: now also C261.1; no longer U7.8 (XTAL_I/CLK_IN)
- new net: C261.2, C262.1, U7.8 (XTAL_I/CLK_IN)
Other:
- note added: "1Vp-p attenuation"
Changed lines of the file:
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@@
   (junction (at 175.26 62.23) (diameter 0) (color 0 0 0 0)
   )
+  (junction (at 57.15 102.87) (diameter 0) (color 0 0 0 0)
+  )
   (junction (at 151.13 78.74) (diameter 0) (color 0 0 0 0)
   )
@@
     (stroke (width 0) (type default) (color 0 0 0 0))
   )
-  (wire (pts (xy 69.85 83.82) (xy 69.85 106.68))
-    (stroke (width 0) (type default) (color 0 0 0 0))
-  )
   (wire (pts (xy 260.35 72.39) (xy 260.35 76.2))
     (stroke (width 0) (type default) (color 0 0 0 0))
@@
     (stroke (width 0) (type default) (color 0 0 0 0))
   )
-  (wire (pts (xy 50.8 83.82) (xy 69.85 83.82))
+  (wire (pts (xy 50.8 83.82) (xy 57.15 83.82))
+    (stroke (width 0) (type default) (color 0 0 0 0))
+  )
+  (wire (pts (xy 57.15 102.87) (xy 69.85 102.87))
     (stroke (width 0) (type default) (color 0 0 0 0))
   )
@@
     (stroke (width 0) (type default) (color 0 0 0 0))
   )
+  (wire (pts (xy 57.15 83.82) (xy 57.15 95.25))
+    (stroke (width 0) (type default) (color 0 0 0 0))
+  )
   (wire (pts (xy 256.54 97.79) (xy 256.54 100.33))
     (stroke (width 0) (type default) (color 0 0 0 0))
@@
   )
   (wire (pts (xy 156.21 132.08) (xy 171.45 132.08))
+    (stroke (width 0) (type default) (color 0 0 0 0))
+  )
+  (wire (pts (xy 69.85 102.87) (xy 69.85 106.68))
     (stroke (width 0) (type default) (color 0 0 0 0))
   )
@@
   )
   (text "DNP" (at 177.8 57.15 0)
+    (effects (font (size 1.27 1.27)) (justify left bottom))
+  )
+  (text "1Vp-p\nattenuation" (at 62.23 101.6 0)
     (effects (font (size 1.27 1.27)) (justify left bottom))
   )
@@
     (pin "2")
   )
+  (symbol (lib_id "Device:C") (at 57.15 106.68 0) (unit 1)
+    (in_bom yes) (on_board yes)
+    (property "Reference" "C262" (id 0) (at 57.785 104.14 0)
+      (effects (font (size 1.27 1.27)) (justify left))
+    )
+    (property "Value" "10p" (id 1) (at 57.785 109.22 0)
+      (effects (font (size 1.27 1.27)) (justify left))
+    )
+    (property "Footprint" "Capacitor_SMD:C_0603_1608Metric" (id 2) (at 58.1152 110.49 0)
+      (effects (font (size 1.27 1.27)) hide)
+    )
+    (property "Datasheet" "~" (id 3) (at 57.15 106.68 0)
+      (effects (font (size 1.27 1.27)) hide)
+    )
+    (pin "1")
+    (pin "2")
+  )
   (symbol (lib_id "Device:R") (at 156.21 63.5 90) (unit 1)
     (in_bom yes) (on_board yes)
@@
     (property "Reference" "L10" (id 0) (at 193.675 71.12 0))
     (property "Value" "ICI70CGI-222" (id 1) (at 180.34 71.12 90))
-    (property "Footprint" "" (id 2) (at 189.23 71.12 0)
-      (effects (font (size 1.27 1.27)) hide)
-    )
-    (property "Datasheet" "~" (id 3) (at 189.23 71.12 0)
+    (property "Footprint" "ICI70CGI:ICI70CGI" (id 2) (at 189.23 71.12 0)
+      (effects (font (size 1.27 1.27)) hide)
+    )
+    (property "Datasheet" "https://product.tdk.com/system/files/dam/doc/product/transformer/transformer/lan/data_sheet/30/ds/lan_mod/ici70cgi.pdf" (id 3) (at 189.23 71.12 0)
       (effects (font (size 1.27 1.27)) hide)
     )
@@
     (property "Reference" "L11" (id 0) (at 226.06 66.675 0))
     (property "Value" "RCM70CGI-471" (id 1) (at 226.06 77.47 0))
-    (property "Footprint" "" (id 2) (at 226.06 71.12 0)
-      (effects (font (size 1.27 1.27)) hide)
-    )
-    (property "Datasheet" "~" (id 3) (at 226.06 71.12 0)
+    (property "Footprint" "ICI70CGI:ICI70CGI" (id 2) (at 226.06 71.12 0)
+      (effects (font (size 1.27 1.27)) hide)
+    )
+    (property "Datasheet" "https://product.tdk.com/system/files/dam/doc/product/transformer/transformer/lan/data_sheet/30/ds/lan_mod/rcm70cgi.pdf" (id 3) (at 226.06 71.12 0)
       (effects (font (size 1.27 1.27)) hide)
     )
@@
     (property "Reference" "D15" (id 0) (at 170.18 93.98 0))
     (property "Value" "UCLAMP3311P" (id 1) (at 181.61 93.98 90))
-    (property "Footprint" "" (id 2) (at 172.72 93.98 0)
+    (property "Footprint" "UCLAMP3311P:SLP1006P2" (id 2) (at 172.72 93.98 0)
       (effects (font (size 1.27 1.27)) hide)
     )
@@
     (property "Reference" "H3" (id 0) (at 280.67 87.63 0))
     (property "Value" "CHASSIS_PE" (id 1) (at 278.765 87.63 0))
-    (property "Footprint" "" (id 2) (at 274.32 87.63 0)
+    (property "Footprint" "MountingHole:MountingHole_3.2mm_M3_Pad_Via" (id 2) (at 274.32 87.63 0)
       (effects (font (size 1.27 1.27)) hide)
     )
@@
     (property "Reference" "FB11" (id 0) (at 163.195 113.03 90))
     (property "Value" "FerriteBead" (id 1) (at 163.83 105.41 90))
-    (property "Footprint" "Inductor_SMD:L_0805_2012Metric" (id 2) (at 163.83 110.998 90)
+    (property "Footprint" "Inductor_SMD:L_1206_3216Metric" (id 2) (at 163.83 110.998 90)
       (effects (font (size 1.27 1.27)) hide)
     )
@@
     (property "Reference" "D14" (id 0) (at 165.1 93.98 0))
     (property "Value" "UCLAMP3311P" (id 1) (at 157.48 93.98 90))
-    (property "Footprint" "" (id 2) (at 167.64 93.98 0)
+    (property "Footprint" "UCLAMP3311P:SLP1006P2" (id 2) (at 167.64 93.98 0)
       (effects (font (size 1.27 1.27)) hide)
     )
@@
     (property "Reference" "L9" (id 0) (at 231.775 53.34 0))
     (property "Value" "PID75-251M" (id 1) (at 240.665 53.34 0))
-    (property "Footprint" "" (id 2) (at 236.22 53.34 0)
-      (effects (font (size 1.27 1.27)) hide)
-    )
-    (property "Datasheet" "~" (id 3) (at 236.22 53.34 0)
+    (property "Footprint" "PID75:PID75-251M" (id 2) (at 236.22 53.34 0)
+      (effects (font (size 1.27 1.27)) hide)
+    )
+    (property "Datasheet" "https://product.tdk.com/system/files/dam/doc/product/inductor/inductor/smd/data_sheet/30/db/ind_2008/pidx251m.pdf" (id 3) (at 236.22 53.34 0)
       (effects (font (size 1.27 1.27)) hide)
     )
@@
     (property "Reference" "D13" (id 0) (at 250.19 71.12 0))
     (property "Value" "CDSOD323-T36SC" (id 1) (at 252.73 63.5 90))
-    (property "Footprint" "" (id 2) (at 252.73 71.12 0)
+    (property "Footprint" "Diode_SMD:D_SOD-323" (id 2) (at 252.73 71.12 0)
       (effects (font (size 1.27 1.27)) hide)
     )
@@
     (property "Reference" "J4" (id 0) (at 269.24 67.31 0))
     (property "Value" "PHY2_MDI" (id 1) (at 269.24 77.47 0))
-    (property "Footprint" "" (id 2) (at 269.24 72.39 0)
+    (property "Footprint" "TerminalBlock_RND:TerminalBlock_RND_205-00288_1x03_P5.08mm_Horizontal" (id 2) (at 269.24 72.39 0)
       (effects (font (size 1.27 1.27)) hide)
     )
@@
     (pin "1")
   )
+  (symbol (lib_id "power:GND") (at 57.15 110.49 0) (unit 1)
+    (in_bom yes) (on_board yes)
+    (property "Reference" "#PWR0250" (id 0) (at 57.15 116.84 0)
+      (effects (font (size 1.27 1.27)) hide)
+    )
+    (property "Value" "GND" (id 1) (at 57.15 114.3 0))
+    (property "Footprint" "" (id 2) (at 57.15 110.49 0)
+      (effects (font (size 1.27 1.27)) hide)
+    )
+    (property "Datasheet" "" (id 3) (at 57.15 110.49 0)
+      (effects (font (size 1.27 1.27)) hide)
+    )
+    (pin "1")
+  )
+  (symbol (lib_id "Device:C") (at 57.15 99.06 0) (unit 1)
+    (in_bom yes) (on_board yes)
+    (property "Reference" "C261" (id 0) (at 57.785 96.52 0)
+      (effects (font (size 1.27 1.27)) (justify left))
+    )
+    (property "Value" "8p2" (id 1) (at 57.785 101.6 0)
+      (effects (font (size 1.27 1.27)) (justify left))
+    )
+    (property "Footprint" "Capacitor_SMD:C_0603_1608Metric" (id 2) (at 58.1152 102.87 0)
+      (effects (font (size 1.27 1.27)) hide)
+    )
+    (property "Datasheet" "~" (id 3) (at 57.15 99.06 0)
+      (effects (font (size 1.27 1.27)) hide)
+    )
+    (pin "1")
+    (pin "2")
+  )
   (symbol (lib_id "Device:R") (at 156.21 73.66 90) (unit 1)

Commit message: Fixing termination for T1L PHYs
Parts:
- removed R92, R93: 100, Resistor_SMD:R_0805_2012Metric, symbol Device:R
- C106, C107: value 10n -> 100p
- FB11: value FerriteBead -> 782763301
Connections:
- net GND: now also C106.2, C107.2
Changed lines of the file:
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@@
-    (stroke (width 0) (type default) (color 0 0 0 0))
-  )
-  (wire (pts (xy 247.65 87.63) (xy 247.65 91.44))
     (stroke (width 0) (type default) (color 0 0 0 0))
   )
@@
     (stroke (width 0) (type default) (color 0 0 0 0))
   )
-  (wire (pts (xy 247.65 99.06) (xy 247.65 100.33))
-    (stroke (width 0) (type default) (color 0 0 0 0))
-  )
   (wire (pts (xy 191.77 62.23) (xy 191.77 66.04))
     (stroke (width 0) (type default) (color 0 0 0 0))
@@
     (stroke (width 0) (type default) (color 0 0 0 0))
   )
-  (wire (pts (xy 238.76 87.63) (xy 238.76 91.44))
-    (stroke (width 0) (type default) (color 0 0 0 0))
-  )
   (polyline (pts (xy 135.89 49.53) (xy 165.1 49.53))
     (stroke (width 0) (type default) (color 0 0 0 0))
@@
   )
   (wire (pts (xy 156.21 120.65) (xy 156.21 109.22))
-    (stroke (width 0) (type default) (color 0 0 0 0))
-  )
-  (wire (pts (xy 238.76 99.06) (xy 238.76 100.33))
     (stroke (width 0) (type default) (color 0 0 0 0))
   )
@@
     (pin "2")
   )
-  (symbol (lib_id "power:GND") (at 238.76 100.33 0) (unit 1)
-    (in_bom yes) (on_board yes)
-    (property "Reference" "#PWR0113" (id 0) (at 238.76 106.68 0)
-      (effects (font (size 1.27 1.27)) hide)
-    )
-    (property "Value" "GND" (id 1) (at 238.76 104.14 0))
-    (property "Footprint" "" (id 2) (at 238.76 100.33 0)
-      (effects (font (size 1.27 1.27)) hide)
-    )
-    (property "Datasheet" "" (id 3) (at 238.76 100.33 0)
+  (symbol (lib_id "power:GND") (at 238.76 87.63 0) (unit 1)
+    (in_bom yes) (on_board yes)
+    (property "Reference" "#PWR0113" (id 0) (at 238.76 93.98 0)
+      (effects (font (size 1.27 1.27)) hide)
+    )
+    (property "Value" "GND" (id 1) (at 238.76 91.44 0))
+    (property "Footprint" "" (id 2) (at 238.76 87.63 0)
+      (effects (font (size 1.27 1.27)) hide)
+    )
+    (property "Datasheet" "" (id 3) (at 238.76 87.63 0)
       (effects (font (size 1.27 1.27)) hide)
     )
@@
     (pin "2")
   )
-  (symbol (lib_id "power:GND") (at 247.65 100.33 0) (unit 1)
-    (in_bom yes) (on_board yes)
-    (property "Reference" "#PWR0114" (id 0) (at 247.65 106.68 0)
-      (effects (font (size 1.27 1.27)) hide)
-    )
-    (property "Value" "GND" (id 1) (at 247.65 104.14 0))
-    (property "Footprint" "" (id 2) (at 247.65 100.33 0)
-      (effects (font (size 1.27 1.27)) hide)
-    )
-    (property "Datasheet" "" (id 3) (at 247.65 100.33 0)
+  (symbol (lib_id "power:GND") (at 247.65 87.63 0) (unit 1)
+    (in_bom yes) (on_board yes)
+    (property "Reference" "#PWR0114" (id 0) (at 247.65 93.98 0)
+      (effects (font (size 1.27 1.27)) hide)
+    )
+    (property "Value" "GND" (id 1) (at 247.65 91.44 0))
+    (property "Footprint" "" (id 2) (at 247.65 87.63 0)
+      (effects (font (size 1.27 1.27)) hide)
+    )
+    (property "Datasheet" "" (id 3) (at 247.65 87.63 0)
       (effects (font (size 1.27 1.27)) hide)
     )
@@
     (pin "9")
   )
-  (symbol (lib_id "Device:R") (at 238.76 95.25 180) (unit 1)
-    (in_bom yes) (on_board yes)
-    (property "Reference" "R92" (id 0) (at 236.728 95.25 90))
-    (property "Value" "100" (id 1) (at 238.76 95.25 90))
-    (property "Footprint" "Resistor_SMD:R_0805_2012Metric" (id 2) (at 240.538 95.25 90)
-      (effects (font (size 1.27 1.27)) hide)
-    )
-    (property "Datasheet" "~" (id 3) (at 238.76 95.25 0)
-      (effects (font (size 1.27 1.27)) hide)
-    )
-    (pin "1")
-    (pin "2")
-  )
   (symbol (lib_id "Device:D_TVS") (at 172.72 93.98 90) (unit 1)
     (in_bom yes) (on_board yes)
@@
     (in_bom yes) (on_board yes)
     (property "Reference" "FB11" (id 0) (at 163.195 113.03 90))
-    (property "Value" "FerriteBead" (id 1) (at 163.83 105.41 90))
+    (property "Value" "782763301" (id 1) (at 163.83 105.41 90))
     (property "Footprint" "Inductor_SMD:L_1206_3216Metric" (id 2) (at 163.83 110.998 90)
       (effects (font (size 1.27 1.27)) hide)
     )
     (property "Datasheet" "~" (id 3) (at 163.83 109.22 0)
-      (effects (font (size 1.27 1.27)) hide)
-    )
-    (pin "1")
-    (pin "2")
-  )
-  (symbol (lib_id "Device:R") (at 247.65 95.25 180) (unit 1)
-    (in_bom yes) (on_board yes)
-    (property "Reference" "R93" (id 0) (at 245.618 95.25 90))
-    (property "Value" "100" (id 1) (at 247.65 95.25 90))
-    (property "Footprint" "Resistor_SMD:R_0805_2012Metric" (id 2) (at 249.428 95.25 90)
-      (effects (font (size 1.27 1.27)) hide)
-    )
-    (property "Datasheet" "~" (id 3) (at 247.65 95.25 0)
       (effects (font (size 1.27 1.27)) hide)
     )
@@
       (effects (font (size 1.27 1.27)) (justify left))
     )
-    (property "Value" "10n" (id 1) (at 239.395 86.36 0)
+    (property "Value" "100p" (id 1) (at 239.395 86.36 0)
       (effects (font (size 1.27 1.27)) (justify left))
     )
@@
       (effects (font (size 1.27 1.27)) (justify left))
     )
-    (property "Value" "10n" (id 1) (at 248.285 86.36 0)
-      (effects (font (size 1.27 1.27)) (justify left))
-    )
+    (property "Value" "100p" (id 1) (at 248.285 86.36 0)
+      (effects (font (size 1.27 1.27)) (justify left))
+    )
