File: 10Base-T1L-PHY6.kicad_sch (KiCad schematic)
At the start: 53 parts, among them J8 PHY6_MDI, U11 ADIN1100, U2 SJA1105Q

Commit message: Minor corrections
Parts:
- added R178: 4K7, Resistor_SMD:R_0603_1608Metric, symbol Device:R
- R179: renamed from R172; value 1K -> 4K7
- R180: renamed from R173; value 1K -> 4K7
- renumbered R168 to R174, R169 to R175, R170 to R176, R171 to R177, R174 to R181, R175 to R182, R176 to R183, R177 to R184, R178 to R185, R179 to R186, R180 to R187, R181 to R188, R182 to R189, R183 to R190, R184 to R191, R185 to R192, R186 to R193, R187 to R194, R188 to R195, R189 to R196, R190 to R197, R191 to R198, R192 to R199, R193 to R200
Connections:
- net +3V3: now also R178.2
- net at R183.1, U2.G14 (MII3_RX_DV): now also R178.1
Other:
- note added: "Config: ------ MACIF_SEL: 0b00 => RMII MS_SEL2: 0b0 => Prefer Slave TX2P4: 0b0 => Enable 1.0V and 2.4V TX SWPD_ENB: 0b1 => Do not enter power down"

Commit message: Assigning Footprints
Parts:
- added C269: 8p2, Capacitor_SMD:C_0603_1608Metric, symbol Device:C
- added C270: 10p, Capacitor_SMD:C_0603_1608Metric, symbol Device:C
- D33: footprint (none) -> Diode_SMD:D_SOD-323
- D34, D35: footprint (none) -> UCLAMP3311P:SLP1006P2
- FB15: footprint Inductor_SMD:L_0805_2012Metric -> Inductor_SMD:L_1206_3216Metric
- H7: footprint (none) -> MountingHole:MountingHole_3.2mm_M3_Pad_Via
- J8: footprint (none) -> TerminalBlock_RND:TerminalBlock_RND_205-00288_1x03_P5.08mm_Horizontal
- L21: footprint (none) -> PID75:PID75-251M
- L22, L23: footprint (none) -> ICI70CGI:ICI70CGI
Connections:
- net GND: now also C270.2
- net at U11.8 (XTAL_I/CLK_IN): now also C269.2, C270.1; no longer R190.2
- new net: C269.1, R190.2
Other:
- note added: "1Vp-p attenuation"
Changed lines of the file:
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@@
   (junction (at 232.41 76.2) (diameter 0) (color 0 0 0 0)
   )
+  (junction (at 55.88 102.87) (diameter 0) (color 0 0 0 0)
+  )
   (junction (at 170.18 104.14) (diameter 0) (color 0 0 0 0)
   )
@@
     (stroke (width 0) (type default) (color 0 0 0 0))
   )
+  (wire (pts (xy 55.88 83.82) (xy 55.88 95.25))
+    (stroke (width 0) (type default) (color 0 0 0 0))
+  )
   (wire (pts (xy 119.38 104.14) (xy 170.18 104.14))
     (stroke (width 0) (type default) (color 0 0 0 0))
@@
     (stroke (width 0) (type default) (color 0 0 0 0))
   )
+  (wire (pts (xy 68.58 102.87) (xy 68.58 106.68))
+    (stroke (width 0) (type default) (color 0 0 0 0))
+  )
   (wire (pts (xy 140.97 83.82) (xy 139.7 83.82))
     (stroke (width 0) (type default) (color 0 0 0 0))
@@
     (stroke (width 0) (type default) (color 0 0 0 0))
   )
+  (wire (pts (xy 55.88 102.87) (xy 68.58 102.87))
+    (stroke (width 0) (type default) (color 0 0 0 0))
+  )
   (wire (pts (xy 246.38 87.63) (xy 246.38 91.44))
     (stroke (width 0) (type default) (color 0 0 0 0))
@@
     (stroke (width 0) (type default) (color 0 0 0 0))
   )
-  (wire (pts (xy 49.53 83.82) (xy 68.58 83.82))
+  (wire (pts (xy 49.53 83.82) (xy 55.88 83.82))
     (stroke (width 0) (type default) (color 0 0 0 0))
   )
@@
   )
   (wire (pts (xy 213.36 62.23) (xy 213.36 68.58))
-    (stroke (width 0) (type default) (color 0 0 0 0))
-  )
-  (wire (pts (xy 68.58 83.82) (xy 68.58 106.68))
     (stroke (width 0) (type default) (color 0 0 0 0))
   )
@@
   (text "Generic 1206 Footprints.\nPopulate according \nto EMC needs."
     (at 254 113.03 0)
+    (effects (font (size 1.27 1.27)) (justify left bottom))
+  )
+  (text "1Vp-p\nattenuation" (at 60.96 101.6 0)
     (effects (font (size 1.27 1.27)) (justify left bottom))
   )
@@
     (pin "1")
   )
+  (symbol (lib_id "power:GND") (at 55.88 110.49 0) (unit 1)
+    (in_bom yes) (on_board yes)
+    (property "Reference" "#PWR0254" (id 0) (at 55.88 116.84 0)
+      (effects (font (size 1.27 1.27)) hide)
+    )
+    (property "Value" "GND" (id 1) (at 55.88 114.3 0))
+    (property "Footprint" "" (id 2) (at 55.88 110.49 0)
+      (effects (font (size 1.27 1.27)) hide)
+    )
+    (property "Datasheet" "" (id 3) (at 55.88 110.49 0)
+      (effects (font (size 1.27 1.27)) hide)
+    )
+    (pin "1")
+  )
+  (symbol (lib_id "Device:C") (at 55.88 106.68 0) (unit 1)
+    (in_bom yes) (on_board yes)
+    (property "Reference" "C270" (id 0) (at 56.515 104.14 0)
+      (effects (font (size 1.27 1.27)) (justify left))
+    )
+    (property "Value" "10p" (id 1) (at 56.515 109.22 0)
+      (effects (font (size 1.27 1.27)) (justify left))
+    )
+    (property "Footprint" "Capacitor_SMD:C_0603_1608Metric" (id 2) (at 56.8452 110.49 0)
+      (effects (font (size 1.27 1.27)) hide)
+    )
+    (property "Datasheet" "~" (id 3) (at 55.88 106.68 0)
+      (effects (font (size 1.27 1.27)) hide)
+    )
+    (pin "1")
+    (pin "2")
+  )
   (symbol (lib_id "Device:R") (at 179.07 53.34 90) (unit 1)
     (in_bom yes) (on_board yes)
@@
     (property "Reference" "D35" (id 0) (at 168.91 93.98 0))
     (property "Value" "UCLAMP3311P" (id 1) (at 180.34 93.98 90))
-    (property "Footprint" "" (id 2) (at 171.45 93.98 0)
+    (property "Footprint" "UCLAMP3311P:SLP1006P2" (id 2) (at 171.45 93.98 0)
       (effects (font (size 1.27 1.27)) hide)
     )
@@
     (property "Reference" "L23" (id 0) (at 224.79 66.675 0))
     (property "Value" "RCM70CGI-471" (id 1) (at 224.79 77.47 0))
-    (property "Footprint" "" (id 2) (at 224.79 71.12 0)
-      (effects (font (size 1.27 1.27)) hide)
-    )
-    (property "Datasheet" "~" (id 3) (at 224.79 71.12 0)
+    (property "Footprint" "ICI70CGI:ICI70CGI" (id 2) (at 224.79 71.12 0)
+      (effects (font (size 1.27 1.27)) hide)
+    )
+    (property "Datasheet" "https://product.tdk.com/system/files/dam/doc/product/transformer/transformer/lan/data_sheet/30/ds/lan_mod/rcm70cgi.pdf" (id 3) (at 224.79 71.12 0)
       (effects (font (size 1.27 1.27)) hide)
     )
@@
     (property "Reference" "L22" (id 0) (at 192.405 71.12 0))
     (property "Value" "ICI70CGI-222" (id 1) (at 179.07 71.12 90))
-    (property "Footprint" "" (id 2) (at 187.96 71.12 0)
-      (effects (font (size 1.27 1.27)) hide)
-    )
-    (property "Datasheet" "~" (id 3) (at 187.96 71.12 0)
+    (property "Footprint" "ICI70CGI:ICI70CGI" (id 2) (at 187.96 71.12 0)
+      (effects (font (size 1.27 1.27)) hide)
+    )
+    (property "Datasheet" "https://product.tdk.com/system/files/dam/doc/product/transformer/transformer/lan/data_sheet/30/ds/lan_mod/ici70cgi.pdf" (id 3) (at 187.96 71.12 0)
       (effects (font (size 1.27 1.27)) hide)
     )
@@
     (property "Reference" "L21" (id 0) (at 230.505 53.34 0))
     (property "Value" "PID75-251M" (id 1) (at 239.395 53.34 0))
-    (property "Footprint" "" (id 2) (at 234.95 53.34 0)
-      (effects (font (size 1.27 1.27)) hide)
-    )
-    (property "Datasheet" "~" (id 3) (at 234.95 53.34 0)
+    (property "Footprint" "PID75:PID75-251M" (id 2) (at 234.95 53.34 0)
+      (effects (font (size 1.27 1.27)) hide)
+    )
+    (property "Datasheet" "https://product.tdk.com/system/files/dam/doc/product/inductor/inductor/smd/data_sheet/30/db/ind_2008/pidx251m.pdf" (id 3) (at 234.95 53.34 0)
       (effects (font (size 1.27 1.27)) hide)
     )
@@
     (property "Reference" "H7" (id 0) (at 279.4 87.63 0))
     (property "Value" "CHASSIS_PE" (id 1) (at 277.495 87.63 0))
-    (property "Footprint" "" (id 2) (at 273.05 87.63 0)
+    (property "Footprint" "MountingHole:MountingHole_3.2mm_M3_Pad_Via" (id 2) (at 273.05 87.63 0)
       (effects (font (size 1.27 1.27)) hide)
     )
@@
     )
     (pin "1")
+  )
+  (symbol (lib_id "Device:C") (at 55.88 99.06 0) (unit 1)
+    (in_bom yes) (on_board yes)
+    (property "Reference" "C269" (id 0) (at 56.515 96.52 0)
+      (effects (font (size 1.27 1.27)) (justify left))
+    )
+    (property "Value" "8p2" (id 1) (at 56.515 101.6 0)
+      (effects (font (size 1.27 1.27)) (justify left))
+    )
+    (property "Footprint" "Capacitor_SMD:C_0603_1608Metric" (id 2) (at 56.8452 102.87 0)
+      (effects (font (size 1.27 1.27)) hide)
+    )
+    (property "Datasheet" "~" (id 3) (at 55.88 99.06 0)
+      (effects (font (size 1.27 1.27)) hide)
+    )
+    (pin "1")
+    (pin "2")
   )
   (symbol (lib_id "Device:R") (at 154.94 63.5 90) (unit 1)
@@
     (property "Reference" "D34" (id 0) (at 163.83 93.98 0))
     (property "Value" "UCLAMP3311P" (id 1) (at 156.21 93.98 90))
-    (property "Footprint" "" (id 2) (at 166.37 93.98 0)
+    (property "Footprint" "UCLAMP3311P:SLP1006P2" (id 2) (at 166.37 93.98 0)
       (effects (font (size 1.27 1.27)) hide)
     )
@@
     (property "Reference" "J8" (id 0) (at 267.97 67.31 0))
     (property "Value" "PHY6_MDI" (id 1) (at 267.97 77.47 0))
-    (property "Footprint" "" (id 2) (at 267.97 72.39 0)
+    (property "Footprint" "TerminalBlock_RND:TerminalBlock_RND_205-00288_1x03_P5.08mm_Horizontal" (id 2) (at 267.97 72.39 0)
       (effects (font (size 1.27 1.27)) hide)
     )
@@
     (property "Reference" "D33" (id 0) (at 248.92 71.12 0))
     (property "Value" "CDSOD323-T36SC" (id 1) (at 251.46 63.5 90))
-    (property "Footprint" "" (id 2) (at 251.46 71.12 0)
+    (property "Footprint" "Diode_SMD:D_SOD-323" (id 2) (at 251.46 71.12 0)
       (effects (font (size 1.27 1.27)) hide)
     )
@@
     (property "Reference" "FB15" (id 0) (at 161.925 113.03 90))
     (property "Value" "FerriteBead" (id 1) (at 162.56 105.41 90))
-    (property "Footprint" "Inductor_SMD:L_0805_2012Metric" (id 2) (at 162.56 110.998 90)
-      (effects (font (size 1.27 1.27)) hide)
-    )
+    (property "Footprint" "Inductor_SMD:L_1206_3216Metric" (id 2) (at 162.56 110.998 90)
+      (effects (font (size 1.27 1.27)) hide)
+    )

Commit message: Fixing termination for T1L PHYs
Parts:
- removed R199, R200: 100, Resistor_SMD:R_0805_2012Metric, symbol Device:R
- C162, C163: value 10n -> 100p
- FB15: value FerriteBead -> 782763301
Connections:
- net GND: now also C162.2, C163.2
Changed lines of the file:
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@@
-    (stroke (width 0) (type default) (color 0 0 0 0))
-  )
-  (wire (pts (xy 246.38 87.63) (xy 246.38 91.44))
     (stroke (width 0) (type default) (color 0 0 0 0))
   )
@@
     (stroke (width 0) (type default) (color 0 0 0 0))
   )
-  (wire (pts (xy 237.49 99.06) (xy 237.49 100.33))
-    (stroke (width 0) (type default) (color 0 0 0 0))
-  )
   (wire (pts (xy 237.49 45.72) (xy 243.84 45.72))
     (stroke (width 0) (type default) (color 0 0 0 0))
@@
     (stroke (width 0) (type default) (color 0 0 0 0))
   )
-  (wire (pts (xy 237.49 87.63) (xy 237.49 91.44))
-    (stroke (width 0) (type default) (color 0 0 0 0))
-  )
   (wire (pts (xy 49.53 88.9) (xy 77.47 88.9))
     (stroke (width 0) (type default) (color 0 0 0 0))
@@
   )
   (wire (pts (xy 149.86 58.42) (xy 149.86 63.5))
-    (stroke (width 0) (type default) (color 0 0 0 0))
-  )
-  (wire (pts (xy 246.38 99.06) (xy 246.38 100.33))
     (stroke (width 0) (type default) (color 0 0 0 0))
   )
@@
       (effects (font (size 1.27 1.27)) (justify left))
     )
-    (property "Value" "10n" (id 1) (at 247.015 86.36 0)
+    (property "Value" "100p" (id 1) (at 247.015 86.36 0)
       (effects (font (size 1.27 1.27)) (justify left))
     )
@@
     (pin "2")
   )
-  (symbol (lib_id "Device:R") (at 237.49 95.25 180) (unit 1)
-    (in_bom yes) (on_board yes)
-    (property "Reference" "R199" (id 0) (at 235.458 95.25 90))
-    (property "Value" "100" (id 1) (at 237.49 95.25 90))
-    (property "Footprint" "Resistor_SMD:R_0805_2012Metric" (id 2) (at 239.268 95.25 90)
-      (effects (font (size 1.27 1.27)) hide)
-    )
-    (property "Datasheet" "~" (id 3) (at 237.49 95.25 0)
-      (effects (font (size 1.27 1.27)) hide)
-    )
-    (pin "1")
-    (pin "2")
-  )
-  (symbol (lib_id "power:GND") (at 237.49 100.33 0) (unit 1)
-    (in_bom yes) (on_board yes)
-    (property "Reference" "#PWR0161" (id 0) (at 237.49 106.68 0)
-      (effects (font (size 1.27 1.27)) hide)
-    )
-    (property "Value" "GND" (id 1) (at 237.49 104.14 0))
-    (property "Footprint" "" (id 2) (at 237.49 100.33 0)
-      (effects (font (size 1.27 1.27)) hide)
-    )
-    (property "Datasheet" "" (id 3) (at 237.49 100.33 0)
+  (symbol (lib_id "power:GND") (at 237.49 87.63 0) (unit 1)
+    (in_bom yes) (on_board yes)
+    (property "Reference" "#PWR0161" (id 0) (at 237.49 93.98 0)
+      (effects (font (size 1.27 1.27)) hide)
+    )
+    (property "Value" "GND" (id 1) (at 237.49 91.44 0))
+    (property "Footprint" "" (id 2) (at 237.49 87.63 0)
+      (effects (font (size 1.27 1.27)) hide)
+    )
+    (property "Datasheet" "" (id 3) (at 237.49 87.63 0)
       (effects (font (size 1.27 1.27)) hide)
     )
@@
     (pin "2")
   )
-  (symbol (lib_id "power:GND") (at 246.38 100.33 0) (unit 1)
-    (in_bom yes) (on_board yes)
-    (property "Reference" "#PWR0162" (id 0) (at 246.38 106.68 0)
-      (effects (font (size 1.27 1.27)) hide)
-    )
-    (property "Value" "GND" (id 1) (at 246.38 104.14 0))
-    (property "Footprint" "" (id 2) (at 246.38 100.33 0)
-      (effects (font (size 1.27 1.27)) hide)
-    )
-    (property "Datasheet" "" (id 3) (at 246.38 100.33 0)
+  (symbol (lib_id "power:GND") (at 246.38 87.63 0) (unit 1)
+    (in_bom yes) (on_board yes)
+    (property "Reference" "#PWR0162" (id 0) (at 246.38 93.98 0)
+      (effects (font (size 1.27 1.27)) hide)
+    )
+    (property "Value" "GND" (id 1) (at 246.38 91.44 0))
+    (property "Footprint" "" (id 2) (at 246.38 87.63 0)
+      (effects (font (size 1.27 1.27)) hide)
+    )
+    (property "Datasheet" "" (id 3) (at 246.38 87.63 0)
       (effects (font (size 1.27 1.27)) hide)
     )
@@
       (effects (font (size 1.27 1.27)) (justify left))
     )
-    (property "Value" "10n" (id 1) (at 238.125 86.36 0)
+    (property "Value" "100p" (id 1) (at 238.125 86.36 0)
       (effects (font (size 1.27 1.27)) (justify left))
     )
@@
     (pin "2")
   )
-  (symbol (lib_id "Device:R") (at 246.38 95.25 180) (unit 1)
-    (in_bom yes) (on_board yes)
-    (property "Reference" "R200" (id 0) (at 244.348 95.25 90))
-    (property "Value" "100" (id 1) (at 246.38 95.25 90))
-    (property "Footprint" "Resistor_SMD:R_0805_2012Metric" (id 2) (at 248.158 95.25 90)
-      (effects (font (size 1.27 1.27)) hide)
-    )
-    (property "Datasheet" "~" (id 3) (at 246.38 95.25 0)
-      (effects (font (size 1.27 1.27)) hide)
-    )
-    (pin "1")
-    (pin "2")
-  )
   (symbol (lib_id "power:GNDPWR") (at 269.24 100.33 0) (unit 1)
     (in_bom yes) (on_board yes)
@@
     (in_bom yes) (on_board yes)
     (property "Reference" "FB15" (id 0) (at 161.925 113.03 90))
-    (property "Value" "FerriteBead" (id 1) (at 162.56 105.41 90))
+    (property "Value" "782763301" (id 1) (at 162.56 105.41 90))
     (property "Footprint" "Inductor_SMD:L_1206_3216Metric" (id 2) (at 162.56 110.998 90)
       (effects (font (size 1.27 1.27)) hide)
