File: Power_Supply.kicad_sch (KiCad schematic)
At the start: 34 parts, among them J13 PWR IN, Q45 SiA449DJ, U18 LM22678TJ-ADJ

Commit message: Minor corrections
Parts:
- renumbered R307 to R314, R308 to R315, R309 to R316, R310 to R317, R311 to R318, R312 to R319, R313 to R320
Changed lines of the file:
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@@
   (symbol (lib_id "Device:R") (at 246.38 90.17 0) (unit 1)
     (in_bom yes) (on_board yes)
-    (property "Reference" "R310" (id 0) (at 248.412 90.17 90))
+    (property "Reference" "R317" (id 0) (at 248.412 90.17 90))
     (property "Value" "4K7" (id 1) (at 246.38 90.17 90))
     (property "Footprint" "Resistor_SMD:R_0603_1608Metric" (id 2) (at 244.602 90.17 90)
@@
   (symbol (lib_id "Device:R") (at 246.38 100.33 0) (unit 1)
     (in_bom yes) (on_board yes)
-    (property "Reference" "R311" (id 0) (at 248.412 100.33 90))
+    (property "Reference" "R318" (id 0) (at 248.412 100.33 90))
     (property "Value" "3K" (id 1) (at 246.38 100.33 90))
     (property "Footprint" "Resistor_SMD:R_0603_1608Metric" (id 2) (at 244.602 100.33 90)
@@
   (symbol (lib_id "power:GND") (at 162.56 110.49 0) (unit 1)
     (in_bom yes) (on_board yes)
-    (property "Reference" "#PWR0244" (id 0) (at 162.56 116.84 0)
+    (property "Reference" "#PWR0245" (id 0) (at 162.56 116.84 0)
       (effects (font (size 1.27 1.27)) hide)
     )
@@
   (symbol (lib_id "Device:R") (at 256.54 85.09 0) (unit 1)
     (in_bom yes) (on_board yes)
-    (property "Reference" "R307" (id 0) (at 258.572 85.09 90))
+    (property "Reference" "R314" (id 0) (at 258.572 85.09 90))
     (property "Value" "1R0" (id 1) (at 256.54 85.09 90))
     (property "Footprint" "Resistor_SMD:R_0805_2012Metric" (id 2) (at 254.762 85.09 90)
@@
   (symbol (lib_id "power:+24V") (at 162.56 83.82 0) (unit 1)
     (in_bom yes) (on_board yes)
-    (property "Reference" "#PWR0243" (id 0) (at 162.56 87.63 0)
+    (property "Reference" "#PWR0244" (id 0) (at 162.56 87.63 0)
       (effects (font (size 1.27 1.27)) hide)
     )
@@
   (symbol (lib_id "Device:R") (at 144.78 102.87 0) (unit 1)
     (in_bom yes) (on_board yes)
-    (property "Reference" "R312" (id 0) (at 146.812 102.87 90))
+    (property "Reference" "R319" (id 0) (at 146.812 102.87 90))
     (property "Value" "10K" (id 1) (at 144.78 102.87 90))
     (property "Footprint" "" (id 2) (at 143.002 102.87 90)
@@
   (symbol (lib_id "Device:R") (at 274.32 85.09 0) (unit 1)
     (in_bom yes) (on_board yes)
-    (property "Reference" "R309" (id 0) (at 276.352 85.09 90))
+    (property "Reference" "R316" (id 0) (at 276.352 85.09 90))
     (property "Value" "1R0" (id 1) (at 274.32 85.09 90))
     (property "Footprint" "Resistor_SMD:R_0805_2012Metric" (id 2) (at 272.542 85.09 90)
@@
   (symbol (lib_id "power:GND") (at 63.5 133.35 0) (unit 1)
     (in_bom yes) (on_board yes)
-    (property "Reference" "#PWR0246" (id 0) (at 63.5 139.7 0)
+    (property "Reference" "#PWR0247" (id 0) (at 63.5 139.7 0)
       (effects (font (size 1.27 1.27)) hide)
     )
@@
   (symbol (lib_id "Device:R") (at 265.43 85.09 0) (unit 1)
     (in_bom yes) (on_board yes)
-    (property "Reference" "R308" (id 0) (at 267.462 85.09 90))
+    (property "Reference" "R315" (id 0) (at 267.462 85.09 90))
     (property "Value" "1R0" (id 1) (at 265.43 85.09 90))
     (property "Footprint" "Resistor_SMD:R_0805_2012Metric" (id 2) (at 263.652 85.09 90)
@@
   (symbol (lib_id "Device:R") (at 53.34 119.38 90) (unit 1)
     (in_bom yes) (on_board yes)
-    (property "Reference" "R313" (id 0) (at 53.34 117.348 90))
+    (property "Reference" "R320" (id 0) (at 53.34 117.348 90))
     (property "Value" "4M7" (id 1) (at 53.34 119.38 90))
     (property "Footprint" "Resistor_SMD:R_1206_3216Metric" (id 2) (at 53.34 121.158 90)
@@
   (symbol (lib_id "power:+3V3") (at 274.32 76.2 0) (unit 1)
     (in_bom yes) (on_board yes)
-    (property "Reference" "#PWR0242" (id 0) (at 274.32 80.01 0)
+    (property "Reference" "#PWR0243" (id 0) (at 274.32 80.01 0)
       (effects (font (size 1.27 1.27)) hide)
     )
@@
   (symbol (lib_id "power:GNDPWR") (at 43.18 133.35 0) (unit 1)
     (in_bom yes) (on_board yes)
-    (property "Reference" "#PWR0245" (id 0) (at 43.18 138.43 0)
-      (effects (font (size 1.27 1.27)) hide)
-    )
+    (property "Reference" "#PWR0246" (id 0) (at 43.18 138.43 0)
+      (effects (font (size 1.27 1.27)) hide)
+    )

Commit message: Assigning Footprints
Parts:
- C242: footprint (none) -> Capacitor_SMD:C_0603_1608Metric
- D58: value D_Zener -> BZT52C10; footprint (none) -> Diode_SMD:D_SOD-123
- F1: value 5A -> RUEF500; footprint (none) -> Fuse:Fuse_Bourns_MF-RG500
- H10: footprint (none) -> MountingHole:MountingHole_3.2mm_M3_Pad_Via
- J13: footprint (none) -> TerminalBlock_RND:TerminalBlock_RND_205-00287_1x02_P5.08mm_Horizontal
- L25, L26, L27: footprint (none) -> MSS1583:MSS1583
- L28: footprint (none) -> Inductor_SMD:L_Bourns_SRF1260
- R319: footprint (none) -> Resistor_SMD:R_0603_1608Metric
- RV1: footprint (none) -> Varistor:RV_Disc_D12mm_W3.9mm_P7.5mm
Other:
- moved on the sheet: C256, H10, R320

Commit message: Fixing termination for T1L PHYs
Parts:
- U18: MPN (none) -> LM22678TJ-ADJ/NOPB
Changed lines of the file:
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@@
+      (effects (font (size 1.27 1.27)) hide)
+    )
+    (property "MPN" "LM22678TJ-ADJ/NOPB" (id 4) (at 205.74 90.17 0)
       (effects (font (size 1.27 1.27)) hide)
     )
