File: SJA1105Q_Switch.kicad_sch (KiCad schematic)
At the start: 23 parts, among them J1 Conn_ARM_JTAG_SWD_10, U1 SJA1105Q, U2 SJA1105Q, X1 ASE-25.000MHz

Commit message: Fixing termination for T1L PHYs
Parts:
- X1: MPN (none) -> ASE-25.000MHZ-L-C-T; ON_FARNELL (none) -> 2308704
Changed lines of the file:
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@@
       (effects (font (size 1.27 1.27)) hide)
     )
-    (property "Datasheet" "~" (id 3) (at 64.77 104.14 0)
+    (property "Datasheet" "https://abracon.com/Oscillators/ASEseries.pdf" (id 3) (at 64.77 104.14 0)
       (effects (font (size 1.27 1.27)) hide)
     )
+    (property "MPN" "ASE-25.000MHZ-L-C-T" (id 4) (at 67.31 104.14 0)
+      (effects (font (size 1.27 1.27)) hide)
+    )
+    (property "ON_FARNELL" "2308704" (id 5) (at 67.31 104.14 0)
+      (effects (font (size 1.27 1.27)) hide)
+    )
