File: kicad/10Base-T1L-PHY0.kicad_sch (KiCad schematic)
At the start: 52 parts, among them J2 PHY0_MDI, U1 SJA1105Q, U5 ADIN1100

Commit message: Initial Placement and Hierarchical Schematic
Parts:
- removed C75: 220n, Capacitor_SMD:C_0805_2012Metric, symbol Device:C
- removed L3: PID75-251M, PID75:PID75-251M, symbol L_differential_1324:L_Coupled_1324
- removed L4: ICI70CGI-222, ICI70CGI:ICI70CGI, symbol Device:L_Coupled_1423
- removed L5: RCM70CGI-471, ICI70CGI:ICI70CGI, symbol Device:L_Coupled_1324
- added C402: 220n, Capacitor_SMD:C_0805_2012Metric, symbol Device:C
- added L401: PID75-251M, PID75:PID75-251M, symbol L_differential_1324:L_Coupled_1324
- added L402: ICI70CGI-222, ICI70CGI:ICI70CGI, symbol Device:L_Coupled_1423
- added L403: RCM70CGI-471, ICI70CGI:ICI70CGI, symbol Device:L_Coupled_1243
- J401: renamed from J2; footprint TerminalBlock_RND:TerminalBlock_RND_205-00288_1x03_P5.08mm_Horizontal -> Connector_Wago:Wago_734-163_1x03_P3.50mm_Horizontal
- renumbered C74 to C401, C76 to C403, C77 to C404, C78 to C405, C79 to C406, C80 to C407, C257 to C408, C258 to C409, C81 to C410, C82 to C411, C83 to C412, C84 to C413, C85 to C414, C86 to C415, C87 to C416, D1 to D401, D2 to D402, D3 to D403, D4 to D404, D5 to D405, FB9 to FB401, H1 to H401, R17 to R401, R18 to R402, R19 to R403, R20 to R404, R21 to R405, R22 to R406, R23 to R407, R24 to R408, R25 to R409, R26 to R410, R27 to R411, R28 to R412, R29 to R413, R30 to R414, R31 to R415, R32 to R416, R33 to R417, R34 to R418, R35 to R419, R36 to R420, R37 to R421, R38 to R422, R39 to R423, U1 to U201, U5 to U401
Connections:
- net MDI_PoDL_N_0: now also L401.2
- net MDI_PoDL_P_0: now also L401.3
- net at R402.1: now also C402.1, L402.1
- net at R402.2: now also C402.2, L403.4
- net at C403.2, R418.2: now also L402.3
- net at C404.2, R419.2: now also L403.1
- net at C406.1, D403.2 (A2), J401.1 (Pin_1): now also L401.4, L403.3
- net at C405.1, D403.1 (A1), J401.2 (Pin_2): now also L401.1, L403.2
- net at C401.2, R401.2: now also L402.2
- net at C404.1, R419.1: now also L402.4
