File: kicad/10Base-T1L-PHY1.kicad_sch (KiCad schematic)
At the start: 53 parts, among them J3 PHY1_MDI, U1 SJA1105Q, U6 ADIN1100

Commit message: Initial Placement and Hierarchical Schematic
Parts:
- removed C89: 220n, Capacitor_SMD:C_0805_2012Metric, symbol Device:C
- removed L6: PID75-251M, PID75:PID75-251M, symbol L_differential_1324:L_Coupled_1324
- removed L7: ICI70CGI-222, ICI70CGI:ICI70CGI, symbol Device:L_Coupled_1423
- removed L8: RCM70CGI-471, ICI70CGI:ICI70CGI, symbol Device:L_Coupled_1324
- added C502: 220n, Capacitor_SMD:C_0805_2012Metric, symbol Device:C
- added L501: PID75-251M, PID75:PID75-251M, symbol L_differential_1324:L_Coupled_1324
- added L502: ICI70CGI-222, ICI70CGI:ICI70CGI, symbol Device:L_Coupled_1423
- added L503: RCM70CGI-471, ICI70CGI:ICI70CGI, symbol Device:L_Coupled_1243
- J501: renamed from J3; footprint TerminalBlock_RND:TerminalBlock_RND_205-00288_1x03_P5.08mm_Horizontal -> Connector_Wago:Wago_734-163_1x03_P3.50mm_Horizontal
- renumbered C88 to C501, C90 to C503, C91 to C504, C92 to C505, C93 to C506, C94 to C507, C259 to C508, C260 to C509, C95 to C510, C96 to C511, C97 to C512, C98 to C513, C99 to C514, C100 to C515, C101 to C516, D6 to D501, D7 to D502, D8 to D503, D9 to D504, D10 to D505, FB10 to FB501, H2 to H501, R42 to R501, R43 to R502, R44 to R503, R45 to R504, R46 to R505, R47 to R506, R48 to R507, R49 to R508, R50 to R509, R51 to R510, R52 to R511, R53 to R512, R54 to R513, R55 to R514, R56 to R515, R57 to R516, R58 to R517, R59 to R518, R60 to R519, R61 to R520, R62 to R521, R63 to R522, R64 to R523, R65 to R524, U1 to U201, U6 to U501
Connections:
- net MDI_PoDL_N_1: now also L501.2
- net MDI_PoDL_P_1: now also L501.3
- net at C506.1, D503.2 (A2), J501.1 (Pin_1): now also L501.4, L503.3
- net at C505.1, D503.1 (A1), J501.2 (Pin_2): now also L501.1, L503.2
- net at C504.1, R520.1: now also L502.4
- net at C504.2, R520.2: now also L503.1
- net at R502.1: now also C502.1, L502.1
- net at R502.2: now also C502.2, L503.4
- net at C501.2, R501.2: now also L502.2
- net at C503.2, R519.2: now also L502.3
