File: kicad/10Base-T1L-PHY2.kicad_sch (KiCad schematic)
At the start: 53 parts, among them J4 PHY2_MDI, U1 SJA1105Q, U7 ADIN1100

Commit message: Initial Placement and Hierarchical Schematic
Parts:
- removed C103: 220n, Capacitor_SMD:C_0805_2012Metric, symbol Device:C
- removed L10: ICI70CGI-222, ICI70CGI:ICI70CGI, symbol Device:L_Coupled_1423
- removed L11: RCM70CGI-471, ICI70CGI:ICI70CGI, symbol Device:L_Coupled_1324
- removed L9: PID75-251M, PID75:PID75-251M, symbol L_differential_1324:L_Coupled_1324
- added C602: 220n, Capacitor_SMD:C_0805_2012Metric, symbol Device:C
- added L601: PID75-251M, PID75:PID75-251M, symbol L_differential_1324:L_Coupled_1324
- added L602: ICI70CGI-222, ICI70CGI:ICI70CGI, symbol Device:L_Coupled_1423
- added L603: RCM70CGI-471, ICI70CGI:ICI70CGI, symbol Device:L_Coupled_1243
- J601: renamed from J4; footprint TerminalBlock_RND:TerminalBlock_RND_205-00288_1x03_P5.08mm_Horizontal -> Connector_Wago:Wago_734-163_1x03_P3.50mm_Horizontal
- renumbered C102 to C601, C104 to C603, C105 to C604, C106 to C605, C107 to C606, C108 to C607, C261 to C608, C262 to C609, C109 to C610, C110 to C611, C111 to C612, C112 to C613, C113 to C614, C114 to C615, C115 to C616, D11 to D601, D12 to D602, D13 to D603, D14 to D604, D15 to D605, FB11 to FB601, H3 to H601, R68 to R601, R69 to R602, R70 to R603, R71 to R604, R72 to R605, R73 to R606, R74 to R607, R75 to R608, R76 to R609, R77 to R610, R78 to R611, R79 to R612, R80 to R613, R81 to R614, R82 to R615, R83 to R616, R84 to R617, R85 to R618, R86 to R619, R87 to R620, R88 to R621, R89 to R622, R90 to R623, R91 to R624, U1 to U201, U7 to U601
Connections:
- net MDI_PoDL_N_2: now also L601.2
- net MDI_PoDL_P_2: now also L601.3
- net at C603.2, R619.2: now also L602.3
- net at R602.1: now also C602.1, L602.1
- net at R602.2: now also C602.2, L603.4
- net at C601.2, R601.2: now also L602.2
- net at C604.1, R620.1: now also L602.4
- net at C604.2, R620.2: now also L603.1
- net at C606.1, D603.2 (A2), J601.1 (Pin_1): now also L601.4, L603.3
- net at C605.1, D603.1 (A1), J601.2 (Pin_2): now also L601.1, L603.2
