File: kicad/10Base-T1L-PHY3.kicad_sch (KiCad schematic)
At the start: 54 parts, among them J5 PHY3_MDI, U1 SJA1105Q, U8 ADIN1100

Commit message: Initial Placement and Hierarchical Schematic
Parts:
- J701: renamed from J5; footprint TerminalBlock_RND:TerminalBlock_RND_205-00288_1x03_P5.08mm_Horizontal -> Connector_Wago:Wago_734-163_1x03_P3.50mm_Horizontal
- L703: renamed from L14; symbol Device:L_Coupled_1324 -> Device:L_Coupled_1243
- renumbered C116 to C701, C117 to C702, C118 to C703, C119 to C704, C120 to C705, C121 to C706, C122 to C707, C263 to C708, C264 to C709, C123 to C710, C124 to C711, C125 to C712, C126 to C713, C127 to C714, C128 to C715, C129 to C716, D16 to D701, D17 to D702, D18 to D703, D19 to D704, D20 to D705, FB12 to FB701, H4 to H701, L12 to L701, L13 to L702, R94 to R701, R95 to R702, R96 to R703, R97 to R704, R98 to R705, R99 to R706, R100 to R707, R101 to R708, R102 to R709, R103 to R710, R104 to R711, R105 to R712, R106 to R713, R107 to R714, R108 to R715, R109 to R716, R110 to R717, R111 to R718, R112 to R719, R113 to R720, R114 to R721, R115 to R722, R116 to R723, R117 to R724, R118 to R725, U1 to U201, U8 to U701
Connections:
- net at C702.2, R702.2: now also L703.4; no longer L703.1
- net at C704.2, R721.2: now also L703.1; no longer L703.2
- net at C705.1, D703.1 (A1), J701.2 (Pin_2)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: now also L703.2; no longer L703.4
