File: kicad/10Base-T1L-PHY4.kicad_sch (KiCad schematic)
At the start: 53 parts, among them J6 PHY4_MDI, U2 SJA1105Q, U9 ADIN1100

Commit message: Initial Placement and Hierarchical Schematic
Parts:
- removed C131: 220n, Capacitor_SMD:C_0805_2012Metric, symbol Device:C
- removed L15: PID75-251M, PID75:PID75-251M, symbol L_differential_1324:L_Coupled_1324
- removed L16: ICI70CGI-222, ICI70CGI:ICI70CGI, symbol Device:L_Coupled_1423
- removed L17: RCM70CGI-471, ICI70CGI:ICI70CGI, symbol Device:L_Coupled_1324
- added C802: 220n, Capacitor_SMD:C_0805_2012Metric, symbol Device:C
- added L801: PID75-251M, PID75:PID75-251M, symbol L_differential_1324:L_Coupled_1324
- added L802: ICI70CGI-222, ICI70CGI:ICI70CGI, symbol Device:L_Coupled_1423
- added L803: RCM70CGI-471, ICI70CGI:ICI70CGI, symbol Device:L_Coupled_1243
- J801: renamed from J6; footprint TerminalBlock_RND:TerminalBlock_RND_205-00288_1x03_P5.08mm_Horizontal -> Connector_Wago:Wago_734-163_1x03_P3.50mm_Horizontal
- renumbered C130 to C801, C132 to C803, C133 to C804, C134 to C805, C135 to C806, C136 to C807, C265 to C808, C266 to C809, C137 to C810, C138 to C811, C139 to C812, C140 to C813, C141 to C814, C142 to C815, C143 to C816, D21 to D801, D22 to D802, D23 to D803, D24 to D804, D25 to D805, FB13 to FB801, H5 to H801, R121 to R801, R122 to R802, R123 to R803, R124 to R804, R125 to R805, R126 to R806, R127 to R807, R128 to R808, R129 to R809, R130 to R810, R131 to R811, R132 to R812, R133 to R813, R134 to R814, R135 to R815, R136 to R816, R137 to R817, R138 to R818, R139 to R819, R140 to R820, R141 to R821, R142 to R822, R143 to R823, R144 to R824, U2 to U202, U9 to U801
Connections:
- net MDI_PoDL_N_4: now also L801.2
- net MDI_PoDL_P_4: now also L801.3
- net at C801.2, R801.2: now also L802.2
- net at C804.1, R820.1: now also L802.4
- net at C804.2, R820.2: now also L803.1
- net at R802.2: now also C802.2, L803.4
- net at C806.1, D803.2 (A2), J801.1 (Pin_1): now also L801.4, L803.3
- net at C805.1, D803.1 (A1), J801.2 (Pin_2): now also L801.1, L803.2
- net at R802.1: now also C802.1, L802.1
- net at C803.2, R819.2: now also L802.3
