File: kicad/10Base-T1L-PHY5.kicad_sch (KiCad schematic)
At the start: 54 parts, among them J7 PHY5_MDI, U10 ADIN1100, U2 SJA1105Q

Commit message: Initial Placement and Hierarchical Schematic
Parts:
- removed C145: 220n, Capacitor_SMD:C_0805_2012Metric, symbol Device:C
- removed L18: PID75-251M, PID75:PID75-251M, symbol L_differential_1324:L_Coupled_1324
- removed L19: ICI70CGI-222, ICI70CGI:ICI70CGI, symbol Device:L_Coupled_1423
- removed L20: RCM70CGI-471, ICI70CGI:ICI70CGI, symbol Device:L_Coupled_1324
- added C902: 220n, Capacitor_SMD:C_0805_2012Metric, symbol Device:C
- added L901: PID75-251M, PID75:PID75-251M, symbol L_differential_1324:L_Coupled_1324
- added L902: ICI70CGI-222, ICI70CGI:ICI70CGI, symbol Device:L_Coupled_1423
- added L903: RCM70CGI-471, ICI70CGI:ICI70CGI, symbol Device:L_Coupled_1243
- J901: renamed from J7; footprint TerminalBlock_RND:TerminalBlock_RND_205-00288_1x03_P5.08mm_Horizontal -> Connector_Wago:Wago_734-163_1x03_P3.50mm_Horizontal
- renumbered C144 to C901, C146 to C903, C147 to C904, C148 to C905, C149 to C906, C150 to C907, C267 to C908, C268 to C909, C151 to C910, C152 to C911, C153 to C912, C154 to C913, C155 to C914, C156 to C915, C157 to C916, D26 to D901, D27 to D902, D28 to D903, D29 to D904, D30 to D905, FB14 to FB901, H6 to H901, R147 to R901, R148 to R902, R149 to R903, R150 to R904, R151 to R905, R152 to R906, R153 to R907, R154 to R908, R155 to R909, R156 to R910, R157 to R911, R158 to R912, R159 to R913, R160 to R914, R161 to R915, R162 to R916, R163 to R917, R164 to R918, R165 to R919, R166 to R920, R167 to R921, R168 to R922, R169 to R923, R170 to R924, R171 to R925, U2 to U202, U10 to U901
Connections:
- net MDI_PoDL_N_5: now also L901.2
- net MDI_PoDL_P_5: now also L901.3
- net at C906.1, D903.2 (A2), J901.1 (Pin_1): now also L901.4, L903.3
- net at C904.1, R921.1: now also L902.4
- net at C904.2, R921.2: now also L903.1
- net at C903.2, R920.2: now also L902.3
- net at R902.1: now also C902.1, L902.1
- net at R902.2: now also C902.2, L903.4
- net at C905.1, D903.1 (A1), J901.2 (Pin_2): now also L901.1, L903.2
- net at C901.2, R901.2: now also L902.2
