File: kicad/10Base-T1L-PHY6.kicad_sch (KiCad schematic)
At the start: 54 parts, among them J8 PHY6_MDI, U11 ADIN1100, U2 SJA1105Q

Commit message: Initial Placement and Hierarchical Schematic
Parts:
- removed C159: 220n, Capacitor_SMD:C_0805_2012Metric, symbol Device:C
- removed L21: PID75-251M, PID75:PID75-251M, symbol L_differential_1324:L_Coupled_1324
- removed L22: ICI70CGI-222, ICI70CGI:ICI70CGI, symbol Device:L_Coupled_1423
- removed L23: RCM70CGI-471, ICI70CGI:ICI70CGI, symbol Device:L_Coupled_1324
- added C1002: 220n, Capacitor_SMD:C_0805_2012Metric, symbol Device:C
- added L1001: PID75-251M, PID75:PID75-251M, symbol L_differential_1324:L_Coupled_1324
- added L1002: ICI70CGI-222, ICI70CGI:ICI70CGI, symbol Device:L_Coupled_1423
- added L1003: RCM70CGI-471, ICI70CGI:ICI70CGI, symbol Device:L_Coupled_1243
- J1001: renamed from J8; footprint TerminalBlock_RND:TerminalBlock_RND_205-00288_1x03_P5.08mm_Horizontal -> Connector_Wago:Wago_734-163_1x03_P3.50mm_Horizontal
- renumbered C158 to C1001, C160 to C1003, C161 to C1004, C162 to C1005, C163 to C1006, C164 to C1007, C269 to C1008, C270 to C1009, C165 to C1010, C166 to C1011, C167 to C1012, C168 to C1013, C169 to C1014, C170 to C1015, C171 to C1016, D31 to D1001, D32 to D1002, D33 to D1003, D34 to D1004, D35 to D1005, FB15 to FB1001, H7 to H1001, R174 to R1001, R175 to R1002, R176 to R1003, R177 to R1004, R178 to R1005, R179 to R1006, R180 to R1007, R181 to R1008, R182 to R1009, R183 to R1010, R184 to R1011, R185 to R1012, R186 to R1013, R187 to R1014, R188 to R1015, R189 to R1016, R190 to R1017, R191 to R1018, R192 to R1019, R193 to R1020, R194 to R1021, R195 to R1022, R196 to R1023, R197 to R1024, R198 to R1025, U11 to U1001, U2 to U202
Connections:
- net MDI_PoDL_N_6: now also L1001.2
- net MDI_PoDL_P_6: now also L1001.3
- net at C1003.2, R1020.2: now also L1002.3
- net at R1002.1: now also C1002.1, L1002.1
- net at R1002.2: now also C1002.2, L1003.4
- net at C1004.1, R1021.1: now also L1002.4
- net at C1004.2, R1021.2: now also L1003.1
- net at C1001.2, R1001.2: now also L1002.2
- net at C1006.1, D1003.2 (A2), J1001.1 (Pin_1): now also L1001.4, L1003.3
- net at C1005.1, D1003.1 (A1), J1001.2 (Pin_2): now also L1001.1, L1003.2
