File: kicad/PoDL_PHY0-1.kicad_sch (KiCad schematic)
At the start: 45 parts, among them Q1 DMG3414U, Q10 DMG3414U, Q11 DMG3414U, Q12 MMBT3904, Q2 MMBTA06, Q3 MMBT3904, Q4 DMG3414U, Q5 DMG3414U, Q6 MMBT3904, Q7 DMG3414U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

Commit message: Initial Placement and Hierarchical Schematic
Parts:
- renumbered C192 to C1201, C193 to C1202, C194 to C1203, C195 to C1204, C196 to C1205, C197 to C1206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
