File: kicad/PoDL_PHY2-3.kicad_sch (KiCad schematic)
At the start: 45 parts, among them Q13 DMG3414U, Q14 MMBTA06, Q15 MMBT3904, Q16 DMG3414U, Q17 DMG3414U, Q18 MMBT3904, Q19 DMG3414U, Q20 MMBTA06, Q21 MMBT3904, Q22 DMG3414U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

Commit message: Initial Placement and Hierarchical Schematic
Parts:
- renumbered C200 to C1301, C201 to C1302, C202 to C1303, C203 to C1304, C204 to C1305, C205 to C1306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
