File: kicad/PoDL_PHY4_REG0.kicad_sch (KiCad schematic)
At the start: 29 parts, among them Q25 DMG3414U, Q26 MMBTA06, Q27 MMBT3904, Q28 DMG3414U, Q29 DMG3414U, Q30 MMBT3904, Q31 SiS412DN, U14 LTC4296-1

Commit message: Initial Placement and Hierarchical Schematic
Parts:
- removed C208: 2u2, Capacitor_SMD:C_0603_1608Metric, symbol Device:C
- removed C209: 100n, Capacitor_SMD:C_0603_1608Metric, symbol Device:C
- removed C210, C211: 2n2, Capacitor_SMD:C_0603_1608Metric, symbol Device:C
- removed D48: S1B-13-F, Diode_SMD:D_SMB, symbol Device:D
- removed D49: BAT54, BAT54:SOT-23-DIODE, symbol Device:D_Schottky
- removed D50: MMBD914LT1G, MMBD914L:SOT-23-DIODE, symbol Device:D
- removed Q25, Q28, Q29: DMG3414U, Package_TO_SOT_SMD:SOT-23, symbol Device:Q_NMOS_GSD
- removed Q26: MMBTA06, Package_TO_SOT_SMD:SOT-23, symbol Device:Q_NPN_BEC
- removed Q27, Q30: MMBT3904, Package_TO_SOT_SMD:SOT-23, symbol Device:Q_NPN_BEC
- removed R260: 0R24, Resistor_SMD:R_1206_3216Metric, symbol Device:R
- removed R261: 50K, Resistor_SMD:R_0603_1608Metric, symbol Device:R
- removed R262: 20, Resistor_SMD:R_1206_3216Metric, symbol Device:R
- removed R263: 50, Resistor_SMD:R_1206_3216Metric, symbol Device:R
- removed R264: 5K, Resistor_SMD:R_0603_1608Metric, symbol Device:R
- removed R265, R267: 5, Resistor_SMD:R_1206_3216Metric, symbol Device:R
- removed R266: 10K, Resistor_SMD:R_0603_1608Metric, symbol Device:R
- removed R268: 0R062, Resistor_SMD:R_1206_3216Metric, symbol Device:R
- removed unit 5 of U14
- renumbered C212 to C1405, C213 to C1406, C214 to C1407, Q31 to Q1407, R269 to R1410, R270 to R1411, U14 to U1401
Other:
- note removed: "CLASS 12"
- note removed: "Class 12 24V / 632mA"
- note removed: "Design following LTC4296-1 datasheet closely!"
- moved on the sheet: C1405, C1406, C1407, Q1407, R1410, R1411, U1401F
