File: kicad/PoDL_PHY5-6.kicad_sch (KiCad schematic)
At the start: 45 parts, among them Q32 DMG3414U, Q33 MMBTA06, Q34 MMBT3904, Q35 DMG3414U, Q36 DMG3414U, Q37 MMBT3904, Q38 DMG3414U, Q39 MMBTA06, Q40 MMBT3904, Q41 DMG3414U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

Commit message: Initial Placement and Hierarchical Schematic
Parts:
- renumbered C215 to C1501, C216 to C1502, C217 to C1503, C218 to C1504, C219 to C1505, C220 to C1506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
