File: kicad/PoDL_REG1.kicad_sch (KiCad schematic)
At the start: 7 parts, among them Q44 SiS412DN, U15 LTC4296-1

Commit message: Initial Placement and Hierarchical Schematic
Parts:
- renumbered C223 to C1601, C224 to C1602, C225 to C1603, Q44 to Q1601, R289 to R1601, R290 to R1602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
Other:
- moved on the sheet: C1601, C1602, C1603, Q1601, R1601, R1602, U1601F
