File: kicad/Power_Supply.kicad_sch (KiCad schematic)
At the start: 34 parts, among them J13 PWR IN, Q45 SiA449DJ, U18 LM22678TJ-ADJ

Commit message: Initial Placement and Hierarchical Schematic
Parts:
- removed H10: CHASSIS_PE, MountingHole:MountingHole_3.2mm_M3_Pad_Via, symbol Mechanical:MountingHole_Pad
- J1501: renamed from J13; footprint TerminalBlock_RND:TerminalBlock_RND_205-00287_1x02_P5.08mm_Horizontal -> TerminalBlock_RND:TerminalBlock_RND_205-00001_1x02_P5.00mm_Horizontal
- renumbered C242 to C1501, C243 to C1502, C244 to C1503, C245 to C1504, C246 to C1505, C247 to C1506, C248 to C1507, C249 to C1508, C250 to C1509, C251 to C1510, C252 to C1511, C253 to C1512, C254 to C1513, C255 to C1514, C256 to C1515, D58 to D1501, D59 to D1502, F1 to F1501, L25 to L1501, L26 to L1502, L27 to L1503, L28 to L1504, Q45 to Q1501, R314 to R1501, R315 to R1502, R316 to R1503, R317 to R1504, R318 to R1505, R319 to R1506, R320 to R1507, RV1 to RV1501, U18 to U1501
Connections:
- net GND: now also L1504.3; no longer L1504.4
- net at C1505.1, L1502.1: now also L1504.4; no longer L1504.3
- net at C1504.1, F1501.2, RV1501.1: now also L1504.2; no longer L1504.1
- net at C1512.2, J1501.2 (Pin_2), RV1501.2: now also L1504.1; no longer L1504.2
