File: kicad/SJA1105Q_Power.kicad_sch (KiCad schematic)
At the start: 84 parts, among them U1 SJA1105Q, U2 SJA1105Q, U3 SC4626C, U4 SC4626C

Commit message: Initial Placement and Hierarchical Schematic
Parts:
- renumbered C4 to C1101, C5 to C1102, C6 to C1103, C7 to C1104, C8 to C1105, C9 to C1106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
