File: kicad/SJA1105Q_Switch.kicad_sch (KiCad schematic)
At the start: 23 parts, among them J1 Conn_ARM_JTAG_SWD_10, U1 SJA1105Q, U2 SJA1105Q, X1 ASE-25.000MHz

Commit message: Initial Placement and Hierarchical Schematic
Parts:
- removed R11: 22, Resistor_SMD:R_0603_1608Metric, symbol Device:R
- renumbered C1 to C201, C2 to C202, C3 to C203, J1 to J201, R1 to R201, R2 to R202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
Connections:
- net at R212.1: now also X201.3 (OUT)
