File: kicad/100Base-TX-PHY7.kicad_sch (KiCad schematic)
At the start: 54 parts, among them J9 JK0654219, U12 KSZ9131RNX, U13 SC4626C, U2 SJA1105Q

Commit message: Initial Placement and Hierarchical Schematic
Parts:
- removed H8: CHASSIS_PE, MountingHole:MountingHole_3.2mm_M3_Pad_Via, symbol Mechanical:MountingHole_Pad
- renumbered C172 to C1001, C173 to C1002, C174 to C1003, C175 to C1004, C176 to C1005, C177 to C1006, C178 to C1007, C179 to C1008, C180 to C1009, C181 to C1010, C182 to C1011, C183 to C1012, C184 to C1013, C185 to C1014, C186 to C1015, C187 to C1016, C188 to C1017, C189 to C1018, C190 to C1019, C191 to C1020, FB16 to FB1001, FB17 to FB1002, FB18 to FB1003, J9 to J1001, L24 to L1001, R201 to R1001, R202 to R1002, R203 to R1003, R204 to R1004, R205 to R1005, R206 to R1006, R207 to R1007, R321 to R1008, R208 to R1009, R209 to R1010, R210 to R1011, R211 to R1012, R212 to R1013, R213 to R1014, R214 to R1015, R215 to R1016, R216 to R1017, R217 to R1018, R218 to R1019, R219 to R1020, R220 to R1021, R322 to R1022, R221 to R1023, R222 to R1024, R223 to R1025, U12 to U1001, U13 to U1002, U2 to U202
Connections:
- net ETH7_PD+: now reaches J1001.8 (MX4+), U1001.10 (TXRXP_D)
- net ETH7_PD-: now reaches J1001.9 (MX4-), U1001.11 (TXRXM_D)
- net ETH7_PA+: now reaches J1001.11 (MX1+), U1001.2 (TXRXP_A)
- net ETH7_PA-: now reaches J1001.10 (MX1-), U1001.3 (TXRXM_A)
- net ETH7_PB+: now reaches J1001.4 (MX2+), U1001.5 (TXRXP_B)
- net ETH7_PB-: now reaches J1001.5 (MX2-), U1001.6 (TXRXM_B)
- net ETH7_PC+: now reaches J1001.3 (MX3+), U1001.7 (TXRXP_C)
- net ETH7_PC-: now reaches J1001.2 (MX3-), U1001.8 (TXRXM_C)

Commit message: Smaller Cicruit Corrections
Parts:
- added R1026, R1027, R1028: 3K3, Resistor_SMD:R_0603_1608Metric, symbol Device:R
Connections:
- net +3V3: now also R1027.1
- net GND: now also R1026.2, R1028.2
- net at U1001.38 (INT_N/PME_N2/ALLPHYAD): now also R1027.2, R1028.1
- net at U1001.48 (ISET): now also R1026.1
Other:
- note added: "DNP"
Changed lines of the file:
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@@
   (junction (at 194.31 132.08) (diameter 0) (color 0 0 0 0)
   )
+  (junction (at 95.25 118.11) (diameter 0) (color 0 0 0 0)
+  )
   (junction (at 186.69 132.08) (diameter 0) (color 0 0 0 0)
   )
@@
   (junction (at 186.69 68.58) (diameter 0) (color 0 0 0 0)
   )
+  (junction (at 114.3 172.72) (diameter 0) (color 0 0 0 0)
+  )
   (junction (at 207.01 38.1) (diameter 0) (color 0 0 0 0)
   )
@@
   (junction (at 179.07 121.92) (diameter 0) (color 0 0 0 0)
   )
+  (junction (at 101.6 144.78) (diameter 0) (color 0 0 0 0)
+  )
   (wire (pts (xy 220.98 86.36) (xy 207.01 86.36))
     (stroke (width 0) (type default) (color 0 0 0 0))
@@
     (stroke (width 0) (type default) (color 0 0 0 0))
   )
+  (wire (pts (xy 118.11 160.02) (xy 114.3 160.02))
+    (stroke (width 0) (type default) (color 0 0 0 0))
+  )
   (wire (pts (xy 200.66 48.26) (xy 220.98 48.26))
     (stroke (width 0) (type default) (color 0 0 0 0))
   )
+  (wire (pts (xy 101.6 162.56) (xy 101.6 144.78))
+    (stroke (width 0) (type default) (color 0 0 0 0))
+  )
   (wire (pts (xy 163.83 142.24) (xy 163.83 144.78))
     (stroke (width 0) (type default) (color 0 0 0 0))
@@
     (stroke (width 0) (type default) (color 0 0 0 0))
   )
+  (wire (pts (xy 101.6 128.27) (xy 101.6 144.78))
+    (stroke (width 0) (type default) (color 0 0 0 0))
+  )
   (wire (pts (xy 237.49 149.86) (xy 237.49 152.4))
     (stroke (width 0) (type default) (color 0 0 0 0))
@@
     (stroke (width 0) (type default) (color 0 0 0 0))
   )
+  (wire (pts (xy 101.6 170.18) (xy 101.6 172.72))
+    (stroke (width 0) (type default) (color 0 0 0 0))
+  )
   (wire (pts (xy 161.29 129.54) (xy 163.83 129.54))
     (stroke (width 0) (type default) (color 0 0 0 0))
@@
     (stroke (width 0) (type default) (color 0 0 0 0))
   )
-  (wire (pts (xy 171.45 160.02) (xy 171.45 163.83))
+  (wire (pts (xy 171.45 160.02) (xy 171.45 170.18))
+    (stroke (width 0) (type default) (color 0 0 0 0))
+  )
+  (wire (pts (xy 114.3 172.72) (xy 114.3 170.18))
     (stroke (width 0) (type default) (color 0 0 0 0))
   )
@@
     (stroke (width 0) (type default) (color 0 0 0 0))
   )
+  (wire (pts (xy 101.6 172.72) (xy 114.3 172.72))
+    (stroke (width 0) (type default) (color 0 0 0 0))
+  )
   (wire (pts (xy 201.93 106.68) (xy 201.93 104.14))
     (stroke (width 0) (type default) (color 0 0 0 0))
@@
     (stroke (width 0) (type default) (color 0 0 0 0))
   )
+  (wire (pts (xy 114.3 160.02) (xy 114.3 162.56))
+    (stroke (width 0) (type default) (color 0 0 0 0))
+  )
   (wire (pts (xy 67.31 48.26) (xy 90.17 48.26))
     (stroke (width 0) (type default) (color 0 0 0 0))
   )
+  (wire (pts (xy 101.6 144.78) (xy 118.11 144.78))
+    (stroke (width 0) (type default) (color 0 0 0 0))
+  )
   (wire (pts (xy 114.3 55.88) (xy 118.11 55.88))
     (stroke (width 0) (type default) (color 0 0 0 0))
@@
     (stroke (width 0) (type default) (color 0 0 0 0))
   )
+  (wire (pts (xy 95.25 118.11) (xy 101.6 118.11))
+    (stroke (width 0) (type default) (color 0 0 0 0))
+  )
   (wire (pts (xy 194.31 147.32) (xy 201.93 147.32))
     (stroke (width 0) (type default) (color 0 0 0 0))
@@
     (stroke (width 0) (type default) (color 0 0 0 0))
   )
+  (wire (pts (xy 101.6 118.11) (xy 101.6 120.65))
+    (stroke (width 0) (type default) (color 0 0 0 0))
+  )
   (wire (pts (xy 200.66 88.9) (xy 220.98 88.9))
     (stroke (width 0) (type default) (color 0 0 0 0))
@@
   )
   (wire (pts (xy 237.49 139.7) (xy 243.84 139.7))
+    (stroke (width 0) (type default) (color 0 0 0 0))
+  )
+  (wire (pts (xy 114.3 173.99) (xy 114.3 172.72))
     (stroke (width 0) (type default) (color 0 0 0 0))
   )
@@
   (text "Generic 1206 Footprints.\nPopulate according \nto EMC needs."
     (at 250.19 114.3 0)
+    (effects (font (size 1.27 1.27)) (justify left bottom))
+  )
+  (text "DNP" (at 100.33 167.64 90)
     (effects (font (size 1.27 1.27)) (justify left bottom))
   )
@@
     (pin "2")
   )
+  (symbol (lib_id "Device:R") (at 101.6 166.37 0) (unit 1)
+    (in_bom yes) (on_board yes)
+    (property "Reference" "R1028" (id 0) (at 103.632 166.37 90))
+    (property "Value" "3K3" (id 1) (at 101.6 166.37 90))
+    (property "Footprint" "Resistor_SMD:R_0603_1608Metric" (id 2) (at 99.822 166.37 90)
+      (effects (font (size 1.27 1.27)) hide)
+    )
+    (property "Datasheet" "~" (id 3) (at 101.6 166.37 0)
+      (effects (font (size 1.27 1.27)) hide)
+    )
+    (pin "1")
+    (pin "2")
+  )
   (symbol (lib_id "Device:C") (at 194.31 153.67 0) (unit 1)
     (in_bom yes) (on_board yes)
@@
     (pin "2")
   )
+  (symbol (lib_id "Device:R") (at 101.6 124.46 0) (unit 1)
+    (in_bom yes) (on_board yes)
+    (property "Reference" "R1027" (id 0) (at 103.632 124.46 90))
+    (property "Value" "3K3" (id 1) (at 101.6 124.46 90))
+    (property "Footprint" "Resistor_SMD:R_0603_1608Metric" (id 2) (at 99.822 124.46 90)
+      (effects (font (size 1.27 1.27)) hide)
+    )
+    (property "Datasheet" "~" (id 3) (at 101.6 124.46 0)
+      (effects (font (size 1.27 1.27)) hide)
+    )
+    (pin "1")
+    (pin "2")
+  )
   (symbol (lib_id "Device:C") (at 196.85 68.58 90) (unit 1)
     (in_bom yes) (on_board yes)
@@
     )
     (pin "1")
+  )
+  (symbol (lib_id "Device:R") (at 114.3 166.37 0) (unit 1)
+    (in_bom yes) (on_board yes)
+    (property "Reference" "R1026" (id 0) (at 116.332 166.37 90))
+    (property "Value" "3K3" (id 1) (at 114.3 166.37 90))
+    (property "Footprint" "Resistor_SMD:R_0603_1608Metric" (id 2) (at 112.522 166.37 90)
+      (effects (font (size 1.27 1.27)) hide)
+    )
+    (property "Datasheet" "~" (id 3) (at 114.3 166.37 0)
+      (effects (font (size 1.27 1.27)) hide)
+    )
+    (pin "1")
+    (pin "2")
   )
   (symbol (lib_id "power:+3V3") (at 220.98 144.78 0) (unit 1)
@@
     (pin "2")
   )
-  (symbol (lib_id "power:GND") (at 171.45 163.83 0) (unit 1)
-    (in_bom yes) (on_board yes)
-    (property "Reference" "#PWR01018" (id 0) (at 171.45 170.18 0)
-      (effects (font (size 1.27 1.27)) hide)
-    )
-    (property "Value" "GND" (id 1) (at 171.45 167.64 0))
-    (property "Footprint" "" (id 2) (at 171.45 163.83 0)
-      (effects (font (size 1.27 1.27)) hide)
-    )
-    (property "Datasheet" "" (id 3) (at 171.45 163.83 0)
+  (symbol (lib_id "power:GND") (at 171.45 170.18 0) (unit 1)
+    (in_bom yes) (on_board yes)
+    (property "Reference" "#PWR01018" (id 0) (at 171.45 176.53 0)
+      (effects (font (size 1.27 1.27)) hide)
+    )
+    (property "Value" "GND" (id 1) (at 171.45 173.99 0))
+    (property "Footprint" "" (id 2) (at 171.45 170.18 0)
+      (effects (font (size 1.27 1.27)) hide)
+    )
+    (property "Datasheet" "" (id 3) (at 171.45 170.18 0)
       (effects (font (size 1.27 1.27)) hide)
     )
@@
       (effects (font (size 1.27 1.27)) hide)
     )
+    (pin "1")
+  )
+  (symbol (lib_id "power:GND") (at 114.3 173.99 0) (unit 1)
+    (in_bom yes) (on_board yes)
+    (property "Reference" "#PWR0101" (id 0) (at 114.3 180.34 0)
+      (effects (font (size 1.27 1.27)) hide)
+    )
+    (property "Value" "GND" (id 1) (at 114.3 177.8 0))
+    (property "Footprint" "" (id 2) (at 114.3 173.99 0)
+      (effects (font (size 1.27 1.27)) hide)
+    )
+    (property "Datasheet" "" (id 3) (at 114.3 173.99 0)
+      (effects (font (size 1.27 1.27)) hide)
+    )
