File: kicad/Open_10Base-T1L_Switch.kicad_sch (KiCad schematic)
At the start: 0 parts

Commit message: Initial Placement and Hierarchical Schematic
Other:
- sheet PoDL PHY4 REG0 renamed PoDL_REG0
- removed sheet PoDL PHY 0-1
- removed sheet PoDL PHY 2-3
- removed sheet PoDL PHY 5-6
- removed sheet PoDL REG1
- added sheet PoDL_REG1 (PoDL_REG.kicad_sch)
- added sheet UnusedUnits (UnusedUnits.kicad_sch)
- sheet 10Base-T1L-PHY0: file 10Base-T1L-PHY0.kicad_sch -> 10Base-T1L-PHY.kicad_sch
- sheet 10Base-T1L-PHY0 ports: added REG_LSNS, SCCPI, SCCPO; removed none
- sheet 10Base-T1L-PHY1: file 10Base-T1L-PHY1.kicad_sch -> 10Base-T1L-PHY.kicad_sch
- sheet 10Base-T1L-PHY1 ports: added REG_LSNS, SCCPI, SCCPO; removed none
- sheet 10Base-T1L-PHY2: file 10Base-T1L-PHY2.kicad_sch -> 10Base-T1L-PHY.kicad_sch
- sheet 10Base-T1L-PHY2 ports: added REG_LSNS, SCCPI, SCCPO; removed none
- sheet 10Base-T1L-PHY3: file 10Base-T1L-PHY3.kicad_sch -> 10Base-T1L-PHY.kicad_sch
- sheet 10Base-T1L-PHY3 ports: added REG_LSNS, SCCPI, SCCPO; removed none
- sheet 10Base-T1L-PHY4: file 10Base-T1L-PHY4.kicad_sch -> 10Base-T1L-PHY.kicad_sch
- sheet 10Base-T1L-PHY4 ports: added REG_LSNS, SCCPI, SCCPO; removed none
- sheet 10Base-T1L-PHY5: file 10Base-T1L-PHY5.kicad_sch -> 10Base-T1L-PHY.kicad_sch
- sheet 10Base-T1L-PHY5 ports: added REG_LSNS, SCCPI, SCCPO; removed none
- sheet 10Base-T1L-PHY6: file 10Base-T1L-PHY6.kicad_sch -> 10Base-T1L-PHY.kicad_sch
- sheet 10Base-T1L-PHY6 ports: added REG_LSNS, SCCPI, SCCPO; removed none
- sheet PoDL_REG0: file PoDL_PHY4_REG0.kicad_sch -> PoDL_REG.kicad_sch
- sheet PoDL_REG0 ports: added LSNS0, LSNS12, LSNS34, SPI_SS; removed none
- note added: "7 PHYs 10Base-T1L ADIN1100 PHY PoDL circuitry"
- note removed: "7 PHYs 10Base-T1L ADIN1100 PHY"
