File: kicad/System_Controller.kicad_sch (KiCad schematic)
At the start: 49 parts, among them J10 CONSOLE, J11 USB_ISP, J12 Conn_ARM_JTAG_SWD_10, SW1 USB_PGM, SW2 USB_PGM, U16 RP2040, U17 IS25LP128F-JBLE, Y1 12MHz

Commit message: Initial Placement and Hierarchical Schematic
Parts:
- removed C240: 1u, Capacitor_SMD:C_1206_3216Metric, symbol Device:C
- removed H9: CHASSIS_PE, MountingHole:MountingHole_3.2mm_M3_Pad_Via, symbol Mechanical:MountingHole_Pad
- removed R305: 4M7, Resistor_SMD:R_1206_3216Metric, symbol Device:R
- renumbered C226 to C1401, C227 to C1402, C228 to C1403, C229 to C1404, C230 to C1405, C231 to C1406, C232 to C1407, C233 to C1408, C234 to C1409, C235 to C1410, C236 to C1411, C237 to C1412, C238 to C1413, C239 to C1414, C241 to C1416, D57 to D1401, J10 to J1401, J11 to J1402, J12 to J1403, R291 to R1401, R292 to R1402, R293 to R1403, R294 to R1404, R295 to R1405, R296 to R1406, R297 to R1407, R298 to R1408, R299 to R1409, R300 to R1410, R301 to R1411, R302 to R1412, R303 to R1413, R304 to R1414, R306 to R1416, R307 to R1417, R308 to R1418, R309 to R1419, R310 to R1420, R311 to R1421, R312 to R1422, R313 to R1423, SW1 to SW1401, SW2 to SW1402, U16 to U1401, U17 to U1402, Y1 to Y1401
Connections:
- net GNDPWR is gone; now on net GND: J1402.6 (Shield)
Other:
- note removed: "Generic 1206 Footprints. Populate according to EMC needs."
